File: kicad/memory.kicad_sch (KiCad schematic)
At the start: 12 parts, among them J8 Molex 87715-9106, U11 ATF22V10C-7PX, U12 ATF22V10C-7PX, U25 CD74ACT273E, U31 AS7C256C-15PCN, U32 AS7C256C-15PCN

Commit message: Tidy every schematic sheet: spread parts, straight runs, buses kept, horizontal tabs
Shared port, expansion and cartridge sheets laid out by hand; buses from
other sheets get a bus label at each chip, busy control nets a label at
each pin; some PLD and connector symbols reordered so wires run straight;
sideways power symbols read across. 0 netlist problems, no overlaps.

Co-Authored-By: Claude Opus 5.5 (1M context) <noreply@anthropic.com>
Claude-Session: https://claude.ai/code/session_01L9AkLuEg13EebxDmgXsaEp
Other:
- moved on the sheet: C31, C32, J8, U31, U32

Commit message: Number parts from 1 for each kind; US zigzag resistor symbols
Main board R1-R54, RN1-RN2, D1-D5, JP1-JP2, F1, NT1, non-decoupling
capacitors C41-C46 (decaps keep Cn = Un); keyboard keys 1-63 row by row
(SWn, Dn, Rn per key). Resistors use R_US / R_Network08_US. --check now
fails on gaps or hundreds in the numbering. PDFs regenerated.

Co-Authored-By: Claude Opus 5.5 (1M context) <noreply@anthropic.com>
Claude-Session: https://claude.ai/code/session_01L9AkLuEg13EebxDmgXsaEp
Parts:
- removed R701: 10k, Resistor_THT:R_Axial_DIN0207_L6.3mm_D2.5mm_P10.16mm_Horizontal, symbol placard_std:R
- added R13: 10k, Resistor_THT:R_Axial_DIN0207_L6.3mm_D2.5mm_P10.16mm_Horizontal, symbol placard_std:R_US
Connections:
- net +5V: now also R13.1
- net at J8.B10 (/CART): now also R13.2
Changed lines of the file:
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@@
   (wire (pts (xy 271.78 128.27) (xy 271.78 125.73)) (stroke (width 0) (type default)))
   (symbol (lib_id "power:+5V") (at 271.78 125.73 0) (unit 1) (in_bom yes) (on_board yes) (dnp no) (property "Reference" "#PWR0723" (at 271.78 125.73 0) (effects (font (size 1.27 1.27)) hide)) (property "Value" "+5V" (at 271.78 119.38 0) (effects (font (size 2 2)))) (property "Footprint" "" (at 271.78 125.73 0) (effects (font (size 1.27 1.27)) hide)) (property "Datasheet" "" (at 271.78 125.73 0) (effects (font (size 1.27 1.27)) hide)) (pin "1") (instances (project "placard" (path "/e3450542-4ffc-59d4-a4a7-45636233928a/be6ca3b6-de05-5292-a0bc-3d79896ebd7e" (reference "#PWR0723") (unit 1)))))
-  (symbol (lib_id "placard_std:R") (at 271.78 132.08 0) (unit 1) (in_bom yes) (on_board yes) (dnp no) (property "Reference" "R701" (at 273.78 131.58 0) (effects (font (size 2.54 2.54) bold) (justify left bottom))) (property "Value" "10k" (at 273.78 134.68 0) (effects (font (size 2 2)) (justify left top))) (property "Footprint" "Resistor_THT:R_Axial_DIN0207_L6.3mm_D2.5mm_P10.16mm_Horizontal" (at 271.78 132.08 0) (effects (font (size 1.27 1.27)) hide)) (property "Datasheet" "~" (at 271.78 132.08 0) (effects (font (size 1.27 1.27)) hide)) (pin "1") (pin "2") (instances (project "placard" (path "/e3450542-4ffc-59d4-a4a7-45636233928a/be6ca3b6-de05-5292-a0bc-3d79896ebd7e" (reference "R701") (unit 1)))))
+  (symbol (lib_id "placard_std:R_US") (at 271.78 132.08 0) (unit 1) (in_bom yes) (on_board yes) (dnp no) (property "Reference" "R13" (at 273.78 131.58 0) (effects (font (size 2.54 2.54) bold) (justify left bottom))) (property "Value" "10k" (at 273.78 134.68 0) (effects (font (size 2 2)) (justify left top))) (property "Footprint" "Resistor_THT:R_Axial_DIN0207_L6.3mm_D2.5mm_P10.16mm_Horizontal" (at 271.78 132.08 0) (effects (font (size 1.27 1.27)) hide)) (property "Datasheet" "~" (at 271.78 132.08 0) (effects (font (size 1.27 1.27)) hide)) (pin "1") (pin "2") (instances (project "placard" (path "/e3450542-4ffc-59d4-a4a7-45636233928a/be6ca3b6-de05-5292-a0bc-3d79896ebd7e" (reference "R13") (unit 1)))))
   (text "Lower 32K: /CE = A15 (RAM U31, cartridge /CE_LO); upper: /CE_HI from U12." (at 20 258 0) (effects (font (size 2.2 2.2)) (justify left bottom)))
   (text "RUN low (cartridge loading): /ROM_OE held off, map register clear (all ROM)." (at 20 261.52 0) (effects (font (size 2.2 2.2)) (justify left bottom)))

Commit message: Bill of materials for the main board, cartridge and keyboard
Manufacturer and MPN fields on every schematic part (empty where none is
chosen), set from an MPN table in gen_kicad_schematic.py; net tie, cartridge
edge fingers and solder jumper excluded from the BOM.  gen_bom.py groups the
parts by part number into docs/BOM.md and docs/BOM.csv, adding sockets,
shunts, keyboard LEDs, keycaps, stabilizers and the keyboard ribbon cable.

Co-Authored-By: Claude Opus 5.5 (1M context) <noreply@anthropic.com>
Claude-Session: https://claude.ai/code/session_018iEnPngycbxX6Tt4Wzp3zN
Parts:
- J8: MPN (none) -> 87715-9106; Manufacturer (none) -> Molex
- U11, U12: MPN (none) -> ATF22V10C-7PX; Manufacturer (none) -> Microchip
- U25: MPN (none) -> CD74ACT273E; Manufacturer (none) -> Texas Instruments
- U31, U32: MPN (none) -> AS7C256C-15PCN; Manufacturer (none) -> Alliance Memory

Commit message: Main board layout: 290 x 140 mm outline, dimensions, connectors and slots placed
gen_kicad_pcb.py places the outline, dimensions, mounting holes, back-edge
I/O (USB-C, audio, VGA, PS/2), left-side SW1/SW2/SD, right-side SNES ports,
cartridge slot J8, expansion slots J9-J12 and keyboard header J1, linked to
the schematic symbols, and draws docs/placard_board_layout.png.
gen_kicad_connectors.py writes preliminary footprints for the parts KiCad
has none for; the schematic generator now assigns all connector footprints.

Co-Authored-By: Claude Opus 5.5 (1M context) <noreply@anthropic.com>
Claude-Session: https://claude.ai/code/session_013qXQudFqhMaBbYKyavQCXN
Parts:
- J8: footprint (none) -> placard:Molex_87715-9106_PCIe_x4_Vertical
Changed lines of the file:
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@@
   (wire (pts (xy 320.04 143.51) (xy 320.04 146.05)) (stroke (width 0) (type default)))
   (symbol (lib_id "power:GND") (at 320.04 146.05 0) (unit 1) (in_bom yes) (on_board yes) (dnp no) (property "Reference" "#PWR0722" (at 320.04 146.05 0) (effects (font (size 1.27 1.27)) hide)) (property "Value" "GND" (at 320.04 152.4 0) (effects (font (size 2 2)) hide)) (property "Footprint" "" (at 320.04 146.05 0) (effects (font (size 1.27 1.27)) hide)) (property "Datasheet" "" (at 320.04 146.05 0) (effects (font (size 1.27 1.27)) hide)) (pin "1") (instances (project "placard" (path "/e3450542-4ffc-59d4-a4a7-45636233928a/be6ca3b6-de05-5292-a0bc-3d79896ebd7e" (reference "#PWR0722") (unit 1)))))
-  (symbol (lib_id "placard_parts:Cartridge_Slot") (at 320.04 95.25 0) (unit 1) (in_bom yes) (on_board yes) (dnp no) (property "Reference" "J8" (at 304.8 44 0) (effects (font (size 2.54 2.54) bold) (justify left bottom))) (property "Value" "Molex 87715-9106" (at 304.8 150 0) (effects (font (size 2 2)) (justify left top))) (property "Footprint" "" (at 320.04 95.25 0) (effects (font (size 1.27 1.27)) hide)) (property "Datasheet" "~" (at 320.04 95.25 0) (effects (font (size 1.27 1.27)) hide)) (property "Manufacturer" "Molex" (at 320.04 95.25 0) (effects (font (size 1.27 1.27)) hide)) (property "MPN" "87715-9106" (at 320.04 95.25 0) (effects (font (size 1.27 1.27)) hide)) (pin "A3") (pin "B3") (pin "A4") (pin "B4") (pin "A5") (pin "B5") (pin "A6") (pin "B6") (pin "A7") (pin "B7") (pin "A8") (pin "B8") (pin "A9") (pin "B9") (pin "A10") (pin "A16") (pin "B16") (pin "A17") (pin "B10") (pin "A22") (pin "A23") (pin "A24") (pin "A25") (pin "A26") (pin "A27") (pin "A28") (pin "A29") (pin "A30") (pin "A32") (pin "B20") (pin "A12") (pin "B12") (pin "A13") (pin "B13") (pin "A14") (pin "B14") (pin "A15") (pin "B15") (pin "A20") (pin "A18") (pin "B19") (pin "B17") (pin "B18") (pin "A19") (pin "B22") (pin "B23") (pin "B24") (pin "B25") (pin "B26") (pin "B27") (pin "B28") (pin "B29") (pin "B30") (pin "B32") (pin "A2") (pin "B2") (pin "A1") (pin "B1") (pin "A11") (pin "B11") (pin "A21") (pin "B21") (pin "A31") (pin "B31") (instances (project "placard" (path "/e3450542-4ffc-59d4-a4a7-45636233928a/be6ca3b6-de05-5292-a0bc-3d79896ebd7e" (reference "J8") (unit 1)))))
+  (symbol (lib_id "placard_parts:Cartridge_Slot") (at 320.04 95.25 0) (unit 1) (in_bom yes) (on_board yes) (dnp no) (property "Reference" "J8" (at 304.8 44 0) (effects (font (size 2.54 2.54) bold) (justify left bottom))) (property "Value" "Molex 87715-9106" (at 304.8 150 0) (effects (font (size 2 2)) (justify left top))) (property "Footprint" "placard:Molex_87715-9106_PCIe_x4_Vertical" (at 320.04 95.25 0) (effects (font (size 1.27 1.27)) hide)) (property "Datasheet" "~" (at 320.04 95.25 0) (effects (font (size 1.27 1.27)) hide)) (property "Manufacturer" "Molex" (at 320.04 95.25 0) (effects (font (size 1.27 1.27)) hide)) (property "MPN" "87715-9106" (at 320.04 95.25 0) (effects (font (size 1.27 1.27)) hide)) (pin "A3") (pin "B3") (pin "A4") (pin "B4") (pin "A5") (pin "B5") (pin "A6") (pin "B6") (pin "A7") (pin "B7") (pin "A8") (pin "B8") (pin "A9") (pin "B9") (pin "A10") (pin "A16") (pin "B16") (pin "A17") (pin "B10") (pin "A22") (pin "A23") (pin "A24") (pin "A25") (pin "A26") (pin "A27") (pin "A28") (pin "A29") (pin "A30") (pin "A32") (pin "B20") (pin "A12") (pin "B12") (pin "A13") (pin "B13") (pin "A14") (pin "B14") (pin "A15") (pin "B15") (pin "A20") (pin "A18") (pin "B19") (pin "B17") (pin "B18") (pin "A19") (pin "B22") (pin "B23") (pin "B24") (pin "B25") (pin "B26") (pin "B27") (pin "B28") (pin "B29") (pin "B30") (pin "B32") (pin "A2") (pin "B2") (pin "A1") (pin "B1") (pin "A11") (pin "B11") (pin "A21") (pin "B21") (pin "A31") (pin "B31") (instances (project "placard" (path "/e3450542-4ffc-59d4-a4a7-45636233928a/be6ca3b6-de05-5292-a0bc-3d79896ebd7e" (reference "J8") (unit 1)))))
   (wire (pts (xy 177.8 76.2) (xy 208.28 76.2)) (stroke (width 0) (type default)))
   (wire (pts (xy 208.28 76.2) (xy 208.28 246.38)) (stroke (width 0) (type default)))

Commit message: Part numbers for the remaining parts; J6 Tensility 54-00174; optional J1 and J9-J12
Every schematic part gets Manufacturer/MPN: Yageo MFR-25 resistors by value,
Bourns 4609X networks, KEMET/TDK ceramics, Panasonic FR electrolytics, ECS
oscillator, Assmann VGA, Sullins headers, Wurth box header, Cherry switches.
Sockets get On Shore numbers (0.3" 24/28-pin are ED241DT/ED281DT; ED28DT is
0.6"). J6 becomes the Tensility 54-00174 TRRS jack with a footprint drawn
from its datasheet. Digi-Key prices from Justin for the oscillator, VGA and
audio jack. The expansion slot sockets and the keyboard header are optional,
with a BOM total without them.

Co-Authored-By: Claude Opus 5.5 (1M context) <noreply@anthropic.com>
Claude-Session: https://claude.ai/code/session_01L9AkLuEg13EebxDmgXsaEp
Parts:
- C11, C12, C25, C31, C32: MPN (none) -> C320C104K5R5TA; Manufacturer (none) -> KEMET
- R13: MPN (none) -> MFR-25FBF52-10K; Manufacturer (none) -> Yageo
