File: kicad/expansion.kicad_sch (KiCad schematic)
At the start: 8 parts, among them J10 Slot 2, J11 Slot 3, J12 Slot 4, J9 Slot 1

Commit message: Tidy every schematic sheet: spread parts, straight runs, buses kept, horizontal tabs
Shared port, expansion and cartridge sheets laid out by hand; buses from
other sheets get a bus label at each chip, busy control nets a label at
each pin; some PLD and connector symbols reordered so wires run straight;
sideways power symbols read across. 0 netlist problems, no overlaps.

Co-Authored-By: Claude Opus 5.5 (1M context) <noreply@anthropic.com>
Claude-Session: https://claude.ai/code/session_01L9AkLuEg13EebxDmgXsaEp
Connections:
- net SEL1: no longer names the net of J9.B17 (SEL), R1101.1
- net SEL2: no longer names the net of J10.B17 (SEL), R1102.1
- net SEL3: no longer names the net of J11.B17 (SEL), R1103.1
- net SEL4: no longer names the net of J12.B17 (SEL), R1104.1
Other:
- moved on the sheet: R1101

Commit message: Number parts from 1 for each kind; US zigzag resistor symbols
Main board R1-R54, RN1-RN2, D1-D5, JP1-JP2, F1, NT1, non-decoupling
capacitors C41-C46 (decaps keep Cn = Un); keyboard keys 1-63 row by row
(SWn, Dn, Rn per key). Resistors use R_US / R_Network08_US. --check now
fails on gaps or hundreds in the numbering. PDFs regenerated.

Co-Authored-By: Claude Opus 5.5 (1M context) <noreply@anthropic.com>
Claude-Session: https://claude.ai/code/session_01L9AkLuEg13EebxDmgXsaEp
Parts:
- removed R1101, R1102, R1103, R1104: 1k, Resistor_THT:R_Axial_DIN0207_L6.3mm_D2.5mm_P10.16mm_Horizontal, symbol placard_std:R
- added R51, R52, R53, R54: 1k, Resistor_THT:R_Axial_DIN0207_L6.3mm_D2.5mm_P10.16mm_Horizontal, symbol placard_std:R_US
Connections:
- net +5V: now also R53.2, R54.2
- net GND: now also R51.2, R52.2
- net at J12.B17 (SEL): now also R54.1
- net at J10.B17 (SEL): now also R52.1
- net at J11.B17 (SEL): now also R53.1
- net at J9.B17 (SEL): now also R51.1
Changed lines of the file:
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@@
   (wire (pts (xy 88.9 133.35) (xy 91.44 133.35)) (stroke (width 0) (type default)))
   (symbol (lib_id "power:GND") (at 91.44 133.35 90) (unit 1) (in_bom yes) (on_board yes) (dnp no) (property "Reference" "#PWR1103" (at 91.44 133.35 0) (effects (font (size 1.27 1.27)) hide)) (property "Value" "GND" (at 99.79 133.35 90) (effects (font (size 2 2)) hide)) (property "Footprint" "" (at 91.44 133.35 0) (effects (font (size 1.27 1.27)) hide)) (property "Datasheet" "" (at 91.44 133.35 0) (effects (font (size 1.27 1.27)) hide)) (pin "1") (instances (project "placard" (path "/e3450542-4ffc-59d4-a4a7-45636233928a/bfc0f6be-8446-560f-84eb-4facad0d0e51" (reference "#PWR1103") (unit 1)))))
-  (symbol (lib_id "placard_std:R") (at 85.09 133.35 90) (unit 1) (in_bom yes) (on_board yes) (dnp no) (property "Reference" "R1101" (at 80.47 138.85 90) (effects (font (size 2.54 2.54) bold) (justify right top))) (property "Value" "1k" (at 80.47 139.55 90) (effects (font (size 2 2)) (justify right bottom))) (property "Footprint" "Resistor_THT:R_Axial_DIN0207_L6.3mm_D2.5mm_P10.16mm_Horizontal" (at 85.09 133.35 0) (effects (font (size 1.27 1.27)) hide)) (property "Datasheet" "~" (at 85.09 133.35 0) (effects (font (size 1.27 1.27)) hide)) (pin "1") (pin "2") (instances (project "placard" (path "/e3450542-4ffc-59d4-a4a7-45636233928a/bfc0f6be-8446-560f-84eb-4facad0d0e51" (reference "R1101") (unit 1)))))
+  (symbol (lib_id "placard_std:R_US") (at 85.09 133.35 90) (unit 1) (in_bom yes) (on_board yes) (dnp no) (property "Reference" "R51" (at 80.47 138.85 90) (effects (font (size 2.54 2.54) bold) (justify right top))) (property "Value" "1k" (at 80.47 139.55 90) (effects (font (size 2 2)) (justify right bottom))) (property "Footprint" "Resistor_THT:R_Axial_DIN0207_L6.3mm_D2.5mm_P10.16mm_Horizontal" (at 85.09 133.35 0) (effects (font (size 1.27 1.27)) hide)) (property "Datasheet" "~" (at 85.09 133.35 0) (effects (font (size 1.27 1.27)) hide)) (pin "1") (pin "2") (instances (project "placard" (path "/e3450542-4ffc-59d4-a4a7-45636233928a/bfc0f6be-8446-560f-84eb-4facad0d0e51" (reference "R51") (unit 1)))))
   (wire (pts (xy 77.47 133.35) (xy 81.28 133.35)) (stroke (width 0) (type default)))
   (wire (pts (xy 154.94 80.01) (xy 154.94 77.47)) (stroke (width 0) (type default)))
@@
   (wire (pts (xy 184.15 133.35) (xy 186.69 133.35)) (stroke (width 0) (type default)))
   (symbol (lib_id "power:GND") (at 186.69 133.35 90) (unit 1) (in_bom yes) (on_board yes) (dnp no) (property "Reference" "#PWR1106" (at 186.69 133.35 0) (effects (font (size 1.27 1.27)) hide)) (property "Value" "GND" (at 195.04 133.35 90) (effects (font (size 2 2)) hide)) (property "Footprint" "" (at 186.69 133.35 0) (effects (font (size 1.27 1.27)) hide)) (property "Datasheet" "" (at 186.69 133.35 0) (effects (font (size 1.27 1.27)) hide)) (pin "1") (instances (project "placard" (path "/e3450542-4ffc-59d4-a4a7-45636233928a/bfc0f6be-8446-560f-84eb-4facad0d0e51" (reference "#PWR1106") (unit 1)))))
-  (symbol (lib_id "placard_std:R") (at 180.34 133.35 90) (unit 1) (in_bom yes) (on_board yes) (dnp no) (property "Reference" "R1102" (at 175.72 138.85 90) (effects (font (size 2.54 2.54) bold) (justify right top))) (property "Value" "1k" (at 175.72 139.55 90) (effects (font (size 2 2)) (justify right bottom))) (property "Footprint" "Resistor_THT:R_Axial_DIN0207_L6.3mm_D2.5mm_P10.16mm_Horizontal" (at 180.34 133.35 0) (effects (font (size 1.27 1.27)) hide)) (property "Datasheet" "~" (at 180.34 133.35 0) (effects (font (size 1.27 1.27)) hide)) (pin "1") (pin "2") (instances (project "placard" (path "/e3450542-4ffc-59d4-a4a7-45636233928a/bfc0f6be-8446-560f-84eb-4facad0d0e51" (reference "R1102") (unit 1)))))
+  (symbol (lib_id "placard_std:R_US") (at 180.34 133.35 90) (unit 1) (in_bom yes) (on_board yes) (dnp no) (property "Reference" "R52" (at 175.72 138.85 90) (effects (font (size 2.54 2.54) bold) (justify right top))) (property "Value" "1k" (at 175.72 139.55 90) (effects (font (size 2 2)) (justify right bottom))) (property "Footprint" "Resistor_THT:R_Axial_DIN0207_L6.3mm_D2.5mm_P10.16mm_Horizontal" (at 180.34 133.35 0) (effects (font (size 1.27 1.27)) hide)) (property "Datasheet" "~" (at 180.34 133.35 0) (effects (font (size 1.27 1.27)) hide)) (pin "1") (pin "2") (instances (project "placard" (path "/e3450542-4ffc-59d4-a4a7-45636233928a/bfc0f6be-8446-560f-84eb-4facad0d0e51" (reference "R52") (unit 1)))))
   (wire (pts (xy 172.72 133.35) (xy 176.53 133.35)) (stroke (width 0) (type default)))
   (wire (pts (xy 250.19 80.01) (xy 250.19 77.47)) (stroke (width 0) (type default)))
@@
   (wire (pts (xy 279.4 133.35) (xy 281.94 133.35)) (stroke (width 0) (type default)))
   (symbol (lib_id "power:+5V") (at 281.94 133.35 270) (unit 1) (in_bom yes) (on_board yes) (dnp no) (property "Reference" "#PWR1109" (at 281.94 133.35 0) (effects (font (size 1.27 1.27)) hide)) (property "Value" "+5V" (at 290.29 133.35 90) (effects (font (size 2 2)))) (property "Footprint" "" (at 281.94 133.35 0) (effects (font (size 1.27 1.27)) hide)) (property "Datasheet" "" (at 281.94 133.35 0) (effects (font (size 1.27 1.27)) hide)) (pin "1") (instances (project "placard" (path "/e3450542-4ffc-59d4-a4a7-45636233928a/bfc0f6be-8446-560f-84eb-4facad0d0e51" (reference "#PWR1109") (unit 1)))))
-  (symbol (lib_id "placard_std:R") (at 275.59 133.35 90) (unit 1) (in_bom yes) (on_board yes) (dnp no) (property "Reference" "R1103" (at 270.97 138.85 90) (effects (font (size 2.54 2.54) bold) (justify right top))) (property "Value" "1k" (at 270.97 139.55 90) (effects (font (size 2 2)) (justify right bottom))) (property "Footprint" "Resistor_THT:R_Axial_DIN0207_L6.3mm_D2.5mm_P10.16mm_Horizontal" (at 275.59 133.35 0) (effects (font (size 1.27 1.27)) hide)) (property "Datasheet" "~" (at 275.59 133.35 0) (effects (font (size 1.27 1.27)) hide)) (pin "1") (pin "2") (instances (project "placard" (path "/e3450542-4ffc-59d4-a4a7-45636233928a/bfc0f6be-8446-560f-84eb-4facad0d0e51" (reference "R1103") (unit 1)))))
+  (symbol (lib_id "placard_std:R_US") (at 275.59 133.35 90) (unit 1) (in_bom yes) (on_board yes) (dnp no) (property "Reference" "R53" (at 270.97 138.85 90) (effects (font (size 2.54 2.54) bold) (justify right top))) (property "Value" "1k" (at 270.97 139.55 90) (effects (font (size 2 2)) (justify right bottom))) (property "Footprint" "Resistor_THT:R_Axial_DIN0207_L6.3mm_D2.5mm_P10.16mm_Horizontal" (at 275.59 133.35 0) (effects (font (size 1.27 1.27)) hide)) (property "Datasheet" "~" (at 275.59 133.35 0) (effects (font (size 1.27 1.27)) hide)) (pin "1") (pin "2") (instances (project "placard" (path "/e3450542-4ffc-59d4-a4a7-45636233928a/bfc0f6be-8446-560f-84eb-4facad0d0e51" (reference "R53") (unit 1)))))
   (wire (pts (xy 267.97 133.35) (xy 271.78 133.35)) (stroke (width 0) (type default)))
   (wire (pts (xy 345.44 80.01) (xy 345.44 77.47)) (stroke (width 0) (type default)))
@@
   (wire (pts (xy 374.65 133.35) (xy 377.19 133.35)) (stroke (width 0) (type default)))
   (symbol (lib_id "power:+5V") (at 377.19 133.35 270) (unit 1) (in_bom yes) (on_board yes) (dnp no) (property "Reference" "#PWR1112" (at 377.19 133.35 0) (effects (font (size 1.27 1.27)) hide)) (property "Value" "+5V" (at 385.54 133.35 90) (effects (font (size 2 2)))) (property "Footprint" "" (at 377.19 133.35 0) (effects (font (size 1.27 1.27)) hide)) (property "Datasheet" "" (at 377.19 133.35 0) (effects (font (size 1.27 1.27)) hide)) (pin "1") (instances (project "placard" (path "/e3450542-4ffc-59d4-a4a7-45636233928a/bfc0f6be-8446-560f-84eb-4facad0d0e51" (reference "#PWR1112") (unit 1)))))
-  (symbol (lib_id "placard_std:R") (at 370.84 133.35 90) (unit 1) (in_bom yes) (on_board yes) (dnp no) (property "Reference" "R1104" (at 366.22 138.85 90) (effects (font (size 2.54 2.54) bold) (justify right top))) (property "Value" "1k" (at 366.22 139.55 90) (effects (font (size 2 2)) (justify right bottom))) (property "Footprint" "Resistor_THT:R_Axial_DIN0207_L6.3mm_D2.5mm_P10.16mm_Horizontal" (at 370.84 133.35 0) (effects (font (size 1.27 1.27)) hide)) (property "Datasheet" "~" (at 370.84 133.35 0) (effects (font (size 1.27 1.27)) hide)) (pin "1") (pin "2") (instances (project "placard" (path "/e3450542-4ffc-59d4-a4a7-45636233928a/bfc0f6be-8446-560f-84eb-4facad0d0e51" (reference "R1104") (unit 1)))))
+  (symbol (lib_id "placard_std:R_US") (at 370.84 133.35 90) (unit 1) (in_bom yes) (on_board yes) (dnp no) (property "Reference" "R54" (at 366.22 138.85 90) (effects (font (size 2.54 2.54) bold) (justify right top))) (property "Value" "1k" (at 366.22 139.55 90) (effects (font (size 2 2)) (justify right bottom))) (property "Footprint" "Resistor_THT:R_Axial_DIN0207_L6.3mm_D2.5mm_P10.16mm_Horizontal" (at 370.84 133.35 0) (effects (font (size 1.27 1.27)) hide)) (property "Datasheet" "~" (at 370.84 133.35 0) (effects (font (size 1.27 1.27)) hide)) (pin "1") (pin "2") (instances (project "placard" (path "/e3450542-4ffc-59d4-a4a7-45636233928a/bfc0f6be-8446-560f-84eb-4facad0d0e51" (reference "R54") (unit 1)))))
   (wire (pts (xy 363.22 133.35) (xy 367.03 133.35)) (stroke (width 0) (type default)))
   (text "SEL: GND on slots 1 and 2, +5 V on slots 3 and 4 (through 1k): the A7 half the card answers." (at 30 205 0) (effects (font (size 2.5 2.5)) (justify left bottom)))

Commit message: Main board layout: 290 x 140 mm outline, dimensions, connectors and slots placed
gen_kicad_pcb.py places the outline, dimensions, mounting holes, back-edge
I/O (USB-C, audio, VGA, PS/2), left-side SW1/SW2/SD, right-side SNES ports,
cartridge slot J8, expansion slots J9-J12 and keyboard header J1, linked to
the schematic symbols, and draws docs/placard_board_layout.png.
gen_kicad_connectors.py writes preliminary footprints for the parts KiCad
has none for; the schematic generator now assigns all connector footprints.

Co-Authored-By: Claude Opus 5.5 (1M context) <noreply@anthropic.com>
Claude-Session: https://claude.ai/code/session_013qXQudFqhMaBbYKyavQCXN
Parts:
- J10, J11, J12, J9: footprint (none) -> placard:CardEdge_2x20_P2.54mm_Vertical

Commit message: Part numbers for the remaining parts; J6 Tensility 54-00174; optional J1 and J9-J12
Every schematic part gets Manufacturer/MPN: Yageo MFR-25 resistors by value,
Bourns 4609X networks, KEMET/TDK ceramics, Panasonic FR electrolytics, ECS
oscillator, Assmann VGA, Sullins headers, Wurth box header, Cherry switches.
Sockets get On Shore numbers (0.3" 24/28-pin are ED241DT/ED281DT; ED28DT is
0.6"). J6 becomes the Tensility 54-00174 TRRS jack with a footprint drawn
from its datasheet. Digi-Key prices from Justin for the oscillator, VGA and
audio jack. The expansion slot sockets and the keyboard header are optional,
with a BOM total without them.

Co-Authored-By: Claude Opus 5.5 (1M context) <noreply@anthropic.com>
Claude-Session: https://claude.ai/code/session_01L9AkLuEg13EebxDmgXsaEp
Parts:
- J10, J11, J12, J9: MPN (none) -> EBC20DCAN; Manufacturer (none) -> Sullins
- R51, R52, R53, R54: MPN (none) -> MFR-25FBF52-1K; Manufacturer (none) -> Yageo

Commit message: Kit footprints: DIP sockets with puller room and part number, resistors with value
Justin: put the chip-puller room in the socket footprints (User.Eco1,
2.5 mm past each end) and the part number in silkscreen between the pin
rows; resistors get their value in silkscreen on the body. New
gen_kicad_kit_footprints.py derives them from KiCad's stock footprints;
schematic, symbols, BOM and PDFs now name them. The board file is left
as is (Justin is editing it): Update PCB from Schematic swaps them in.

Co-Authored-By: Claude Opus 5.5 (1M context) <noreply@anthropic.com>
Claude-Session: https://claude.ai/code/session_01JnVuvUvdWezUUU6Sgmg16H
Parts:
- R51, R52, R53, R54: footprint Resistor_THT:R_Axial_DIN0207_L6.3mm_D2.5mm_P10.16mm_Horizontal -> placard:R_Axial_DIN0207_L6.3mm_D2.5mm_P10.16mm_Horizontal_Value
