File: kicad/expansion.kicad_sch (KiCad schematic)
At the start: 8 parts, among them J10 Slot 2, J11 Slot 3, J12 Slot 4, J9 Slot 1

Commit message: Schematic: expansion slot contacts A8-B11 become BT1-BT8 (slot-1 boot)
Cards latch D7:D0, so the slots no longer carry SRC7:SRC0.  Slot 1's
BT1-BT5 carry STALL_IN, STALL_OUT, PC_ENABLE, PIXEL_ENABLE and /CART;
BT6-BT8 and slots 2-4's boot contacts are not connected
(EXPANSION.md, "Booting from slot 1").  Slots respaced to keep the labels
on the page.

Co-Authored-By: Claude Opus 5.5 (1M context) <noreply@anthropic.com>
Claude-Session: https://claude.ai/code/session_016q7L8WUy2bLsrwHss8WZwY
Connections:
- removed net SRC0: J10.A8 (SD0), J11.A8 (SD0), J12.A8 (SD0), J9.A8 (SD0)
- removed net SRC1: J10.B8 (SD1), J11.B8 (SD1), J12.B8 (SD1), J9.B8 (SD1)
- removed net SRC2: J10.A9 (SD2), J11.A9 (SD2), J12.A9 (SD2), J9.A9 (SD2)
- removed net SRC3: J10.B9 (SD3), J11.B9 (SD3), J12.B9 (SD3), J9.B9 (SD3)
- removed net SRC4: J10.A10 (SD4), J11.A10 (SD4), J12.A10 (SD4), J9.A10 (SD4)
- removed net SRC5: J10.B10 (SD5), J11.B10 (SD5), J12.B10 (SD5), J9.B10 (SD5)
- removed net SRC6: J10.A11 (SD6), J11.A11 (SD6), J12.A11 (SD6), J9.A11 (SD6)
- removed net SRC7: J10.B11 (SD7), J11.B11 (SD7), J12.B11 (SD7), J9.B11 (SD7)
- new net PC_ENABLE: J9.A9 (BT3)
- new net PIXEL_ENABLE: J9.B9 (BT4)
- new net STALL_IN: J9.A8 (BT1)
- new net STALL_OUT: J9.B8 (BT2)
- new net ~{CART}: J9.A10 (BT5)
- no-connect marks 0 -> 27
Other:
- note added: "BT1-BT8 (boot contacts): slot 1 only, STALL_IN, STALL_OUT, PC_ENABLE, PIXEL_ENABLE, /CART; cards latch D7:D0."
- note removed: "SD7:SD0 = SRC7:SRC0, the source drivers' side of the series resistors (the write data)."
- moved on the sheet: J10, J11, J12, J9, R51, R52, R53, R54

Commit message: Schematic: rename buses to ADDR / DATABUS / D, wire the shared port outputs
- Address bus A15:A0 is now ADDR15:ADDR0, the data bus D7:D0 is DATABUS7:DATABUS0
  and the D register's outputs DR7:DR0 are D7:D0 (main board and both cartridges).
- Shared port sheet: U38's outputs P_SCK, P_MOSI, P_CS, P_PS2D and K0 are wired
  to the SNES pads, the SD dividers and the PS/2 hold diodes (K0 -> D6 ->
  keyboard CLK).  J3 now sits level with U38's SCK/MOSI pins, J2 above it.
- Parts moved so the longer labels fit: U3/U4 and the PC bus, U18, U22, U11,
  U31, U32, RN1, R5-R12; expansion slots in two rows.
- SCHEMATIC_PLAN.md: the bus names.

Co-Authored-By: Claude Opus 5.5 <noreply@anthropic.com>
Claude-Session: https://claude.ai/code/session_01DnW5SUv7E4nz9tGtPvD1qV
Connections:
- net A0 renamed ADDR0
- net A1 renamed ADDR1
- net A2 renamed ADDR2
- net A3 renamed ADDR3
- net A4 renamed ADDR4
- net A5 renamed ADDR5
- net A6 renamed ADDR6
- net A7 renamed ADDR7
- net D0 renamed DATABUS0
- net D1 renamed DATABUS1
- net D2 renamed DATABUS2
- net D3 renamed DATABUS3
- net D4 renamed DATABUS4
- net D5 renamed DATABUS5
- net D6 renamed DATABUS6
- net D7 renamed DATABUS7
Other:
- note added: "BT1-BT8 (boot contacts): slot 1 only, STALL_IN, STALL_OUT, PC_ENABLE, PIXEL_ENABLE, /CART; cards latch DATABUS7:0."
- note removed: "BT1-BT8 (boot contacts): slot 1 only, STALL_IN, STALL_OUT, PC_ENABLE, PIXEL_ENABLE, /CART; cards latch D7:D0."
- moved on the sheet: J10, J11, J12, J9, R51, R52, R53, R54
