File: kicad/video_timing.kicad_sch (KiCad schematic)
At the start: 10 parts, among them U13 ATF22V10C-10PU, U14 ATF22V10C-10PU, U15 ATF22V10C-7PX, U29 SN74F541N, U35 ATF22V10C-10PU

Commit message: Tidy every schematic sheet: spread parts, straight runs, buses kept, horizontal tabs
Shared port, expansion and cartridge sheets laid out by hand; buses from
other sheets get a bus label at each chip, busy control nets a label at
each pin; some PLD and connector symbols reordered so wires run straight;
sideways power symbols read across. 0 netlist problems, no overlaps.

Co-Authored-By: Claude Opus 5.5 (1M context) <noreply@anthropic.com>
Claude-Session: https://claude.ai/code/session_01L9AkLuEg13EebxDmgXsaEp
Other:
- moved on the sheet: C13, C14, U13, U14

Commit message: Bill of materials for the main board, cartridge and keyboard
Manufacturer and MPN fields on every schematic part (empty where none is
chosen), set from an MPN table in gen_kicad_schematic.py; net tie, cartridge
edge fingers and solder jumper excluded from the BOM.  gen_bom.py groups the
parts by part number into docs/BOM.md and docs/BOM.csv, adding sockets,
shunts, keyboard LEDs, keycaps, stabilizers and the keyboard ribbon cable.

Co-Authored-By: Claude Opus 5.5 (1M context) <noreply@anthropic.com>
Claude-Session: https://claude.ai/code/session_018iEnPngycbxX6Tt4Wzp3zN
Parts:
- U13, U14, U35: MPN (none) -> ATF22V10C-10PU; Manufacturer (none) -> Microchip
- U15: MPN (none) -> ATF22V10C-7PX; Manufacturer (none) -> Microchip
- U29: MPN (none) -> SN74F541N; Manufacturer (none) -> Texas Instruments

Commit message: Part numbers for the remaining parts; J6 Tensility 54-00174; optional J1 and J9-J12
Every schematic part gets Manufacturer/MPN: Yageo MFR-25 resistors by value,
Bourns 4609X networks, KEMET/TDK ceramics, Panasonic FR electrolytics, ECS
oscillator, Assmann VGA, Sullins headers, Wurth box header, Cherry switches.
Sockets get On Shore numbers (0.3" 24/28-pin are ED241DT/ED281DT; ED28DT is
0.6"). J6 becomes the Tensility 54-00174 TRRS jack with a footprint drawn
from its datasheet. Digi-Key prices from Justin for the oscillator, VGA and
audio jack. The expansion slot sockets and the keyboard header are optional,
with a BOM total without them.

Co-Authored-By: Claude Opus 5.5 (1M context) <noreply@anthropic.com>
Claude-Session: https://claude.ai/code/session_01L9AkLuEg13EebxDmgXsaEp
Parts:
- C13, C14, C15, C29, C35: MPN (none) -> C320C104K5R5TA; Manufacturer (none) -> KEMET

Commit message: Schematic: row tint and blank line
Video out sheet: U23 is a 74HCT377; Q6:Q4 drive the row tint (R56-R58
910 ohm, two 1N4148 per channel into VGA_R/G/B, BAT85 D27-D29 from each
node to VIDEN).  Video timing sheet: U23 Q7 (LC7) to H counter pin 6.
New Device:D symbol in placard_std; H counter symbol has LC7.  The
regenerated symbol library also brings the memory control /WE pin type
up to date.  BOM not regenerated yet.

Co-Authored-By: Claude Opus 5.5 (1M context) <noreply@anthropic.com>
Claude-Session: https://claude.ai/code/session_01AyS52y3xy4qvxwvt915gG3
Connections:
- net LC7: now reaches U13.6 (LC7)
Other:
- note added: "LC7 (mode byte bit 7, U23 Q7) blanks the line."

Commit message: Every PLD is an ATF22V10C-7PX (one part number)
Justin: switch the seven main-board -10PU PLDs (Branch, PC x2, H, V,
color decoder, audio slot) and the cartridge loader to the -7PX, for one
part number to buy, program and kit (.52 more per main board). Symbols,
schematics, PDFs, BOM, docs and PLD comments updated; CHIPS.md keeps the
grade each PLD could use.

Co-Authored-By: Claude Opus 5.5 (1M context) <noreply@anthropic.com>
Claude-Session: https://claude.ai/code/session_01JnVuvUvdWezUUU6Sgmg16H
Parts:
- U13, U14, U35: value ATF22V10C-10PU -> ATF22V10C-7PX; MPN ATF22V10C-10PU -> ATF22V10C-7PX

Commit message: Kit footprints: DIP sockets with puller room and part number, resistors with value
Justin: put the chip-puller room in the socket footprints (User.Eco1,
2.5 mm past each end) and the part number in silkscreen between the pin
rows; resistors get their value in silkscreen on the body. New
gen_kicad_kit_footprints.py derives them from KiCad's stock footprints;
schematic, symbols, BOM and PDFs now name them. The board file is left
as is (Justin is editing it): Update PCB from Schematic swaps them in.

Co-Authored-By: Claude Opus 5.5 (1M context) <noreply@anthropic.com>
Claude-Session: https://claude.ai/code/session_01JnVuvUvdWezUUU6Sgmg16H
Parts:
- U13, U14, U15, U35: footprint Package_DIP:DIP-24_W7.62mm -> placard:DIP-24_W7.62mm_Socket_Puller
- U29: footprint Package_DIP:DIP-20_W7.62mm -> placard:DIP-20_W7.62mm_Socket_Puller
