File: kicad/video_timing.kicad_sch (KiCad schematic)
At the start: 10 parts, among them U13 ATF22V10C-7PX, U14 ATF22V10C-7PX, U15 ATF22V10C-7PX, U29 SN74F541N, U35 ATF22V10C-7PX

Commit message: Name the vertical sync /VSYNC like /HSYNC
Sync PLD rev 09 declares pin 18 active low (PIN 18 = !VSYNC) with the
equation written as logical true, the same way the H counter declares
!HSYNC.  The pin output is unchanged (low during counts 532-533) and the
equation drops from 6 product terms to 1.  Schematic net, symbol pin,
VHDL comments, bring-up labels and docs follow; main schematic PDF
regenerated.

Co-Authored-By: Claude Opus 5.5 (1M context) <noreply@anthropic.com>
Claude-Session: https://claude.ai/code/session_013veaZZUxC2KxHUx8e17FHP
Connections:
- net VSYNC renamed ~{VSYNC}
Changed lines of the file:
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@@
   (global_label "PIXEL_ENABLE" (shape output) (at 275.59 93.98 0) (fields_autoplaced) (effects (font (size 2 2)) (justify left)) (property "Intersheetrefs" "${INTERSHEET_REFS}" (at 275.59 93.98 0) (effects (font (size 2 2)) (justify left) hide)))
   (wire (pts (xy 264.16 99.06) (xy 275.59 99.06)) (stroke (width 0) (type default)))
-  (global_label "VSYNC" (shape output) (at 275.59 99.06 0) (fields_autoplaced) (effects (font (size 2 2)) (justify left)) (property "Intersheetrefs" "${INTERSHEET_REFS}" (at 275.59 99.06 0) (effects (font (size 2 2)) (justify left) hide)))
+  (global_label "~{VSYNC}" (shape output) (at 275.59 99.06 0) (fields_autoplaced) (effects (font (size 2 2)) (justify left)) (property "Intersheetrefs" "${INTERSHEET_REFS}" (at 275.59 99.06 0) (effects (font (size 2 2)) (justify left) hide)))
   (wire (pts (xy 264.16 111.76) (xy 275.59 111.76)) (stroke (width 0) (type default)))
   (global_label "ADDR_SEL" (shape output) (at 275.59 111.76 0) (fields_autoplaced) (effects (font (size 2 2)) (justify left)) (property "Intersheetrefs" "${INTERSHEET_REFS}" (at 275.59 111.76 0) (effects (font (size 2 2)) (justify left) hide)))

Commit message: VGA syncs: 47 ohm series resistors R61/R62 at the PLD pins
/HSYNC (U13 pin 21) and /VSYNC (U15 pin 18) now reach J7 through R61 and
R62 (47 ohm, Yageo MFR-25FBF52-47R, sharing R5-R12's BOM line); nets after
them are /VGA_HSYNC and /VGA_VSYNC.  Symbol uuids kept; board file untouched
(pull in with Update PCB from Schematic).  R60 22k gets its MPN.

Co-Authored-By: Claude Opus 5.5 (1M context) <noreply@anthropic.com>
Claude-Session: https://claude.ai/code/session_01B4M15KLwAcnVuRUejEFj2o
Parts:
- added R61, R62: 47, placard:R_Axial_DIN0207_L6.3mm_D2.5mm_P10.16mm_Horizontal_Value, symbol placard_std:R_US
Connections:
- net ~{HSYNC}: no longer names the net of U13.21 (/HSYNC)
- net ~{HSYNC}: now also R61.1
- net ~{VSYNC}: no longer names the net of U15.18 (/VSYNC)
- net ~{VSYNC}: now also R62.1
- new net ~{VGA_HSYNC}: R61.2
- new net ~{VGA_VSYNC}: R62.2
Changed lines of the file:
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@@
   (symbol (lib_id "power:GND") (at 254 64.77 0) (unit 1) (in_bom yes) (on_board yes) (dnp no) (property "Reference" "#PWR0813" (at 254 64.77 0) (effects (font (size 1.27 1.27)) hide)) (property "Value" "GND" (at 254 71.12 0) (effects (font (size 2 2)) hide)) (property "Footprint" "" (at 254 64.77 0) (effects (font (size 1.27 1.27)) hide)) (property "Datasheet" "" (at 254 64.77 0) (effects (font (size 1.27 1.27)) hide)) (pin "1") (instances (project "placard" (path "/e3450542-4ffc-59d4-a4a7-45636233928a/222c409e-e9c7-5ee1-806a-ff3848ff76be" (reference "#PWR0813") (unit 1)))))
   (symbol (lib_id "placard_std:C") (at 254 60.96 0) (unit 1) (in_bom yes) (on_board yes) (dnp no) (property "Reference" "C15" (at 256 60.46 0) (effects (font (size 2.54 2.54) bold) (justify left bottom))) (property "Value" "100n" (at 256 63.56 0) (effects (font (size 2 2)) (justify left top))) (property "Footprint" "Capacitor_THT:C_Disc_D5.0mm_W2.5mm_P5.00mm" (at 254 60.96 0) (effects (font (size 1.27 1.27)) hide)) (property "Datasheet" "~" (at 254 60.96 0) (effects (font (size 1.27 1.27)) hide)) (property "Manufacturer" "KEMET" (at 254 60.96 0) (effects (font (size 1.27 1.27)) hide)) (property "MPN" "C320C104K5R5TA" (at 254 60.96 0) (effects (font (size 1.27 1.27)) hide)) (pin "1") (pin "2") (instances (project "placard" (path "/e3450542-4ffc-59d4-a4a7-45636233928a/222c409e-e9c7-5ee1-806a-ff3848ff76be" (reference "C15") (unit 1)))))
+  (symbol (lib_id "placard_std:R_US") (at 119.38 96.52 90) (unit 1) (in_bom yes) (on_board yes) (dnp no) (property "Reference" "R61" (at 114.88 93.12 90) (effects (font (size 2.54 2.54) bold) (justify right top))) (property "Value" "47" (at 123.38 93.12 90) (effects (font (size 2 2)) (justify right bottom))) (property "Footprint" "placard:R_Axial_DIN0207_L6.3mm_D2.5mm_P10.16mm_Horizontal_Value" (at 119.38 96.52 0) (effects (font (size 1.27 1.27)) hide)) (property "Datasheet" "~" (at 119.38 96.52 0) (effects (font (size 1.27 1.27)) hide)) (property "Manufacturer" "Yageo" (at 119.38 96.52 0) (effects (font (size 1.27 1.27)) hide)) (property "MPN" "MFR-25FBF52-47R" (at 119.38 96.52 0) (effects (font (size 1.27 1.27)) hide)) (pin "1") (pin "2") (instances (project "placard" (path "/e3450542-4ffc-59d4-a4a7-45636233928a/222c409e-e9c7-5ee1-806a-ff3848ff76be" (reference "R61") (unit 1)))))
+  (wire (pts (xy 99.06 96.52) (xy 115.57 96.52)) (stroke (width 0) (type default)))
+  (wire (pts (xy 123.19 96.52) (xy 130.81 96.52)) (stroke (width 0) (type default)))
+  (symbol (lib_id "placard_std:R_US") (at 312.42 99.06 90) (unit 1) (in_bom yes) (on_board yes) (dnp no) (property "Reference" "R62" (at 307.92 95.66 90) (effects (font (size 2.54 2.54) bold) (justify right top))) (property "Value" "47" (at 316.42 95.66 90) (effects (font (size 2 2)) (justify right bottom))) (property "Footprint" "placard:R_Axial_DIN0207_L6.3mm_D2.5mm_P10.16mm_Horizontal_Value" (at 312.42 99.06 0) (effects (font (size 1.27 1.27)) hide)) (property "Datasheet" "~" (at 312.42 99.06 0) (effects (font (size 1.27 1.27)) hide)) (property "Manufacturer" "Yageo" (at 312.42 99.06 0) (effects (font (size 1.27 1.27)) hide)) (property "MPN" "MFR-25FBF52-47R" (at 312.42 99.06 0) (effects (font (size 1.27 1.27)) hide)) (pin "1") (pin "2") (instances (project "placard" (path "/e3450542-4ffc-59d4-a4a7-45636233928a/222c409e-e9c7-5ee1-806a-ff3848ff76be" (reference "R62") (unit 1)))))
+  (wire (pts (xy 264.16 99.06) (xy 308.61 99.06)) (stroke (width 0) (type default)))
+  (wire (pts (xy 316.23 99.06) (xy 323.85 99.06)) (stroke (width 0) (type default)))
   (wire (pts (xy 233.68 177.8) (xy 233.68 175.26)) (stroke (width 0) (type default)))
   (symbol (lib_id "power:+5V") (at 233.68 175.26 0) (unit 1) (in_bom yes) (on_board yes) (dnp no) (property "Reference" "#PWR0814" (at 233.68 175.26 0) (effects (font (size 1.27 1.27)) hide)) (property "Value" "+5V" (at 233.68 168.91 0) (effects (font (size 2 2)))) (property "Footprint" "" (at 233.68 175.26 0) (effects (font (size 1.27 1.27)) hide)) (property "Datasheet" "" (at 233.68 175.26 0) (effects (font (size 1.27 1.27)) hide)) (pin "1") (instances (project "placard" (path "/e3450542-4ffc-59d4-a4a7-45636233928a/222c409e-e9c7-5ee1-806a-ff3848ff76be" (reference "#PWR0814") (unit 1)))))
@@
   (bus (pts (xy 107.95 85.09) (xy 107.95 87.63)) (stroke (width 0) (type default)))
   (bus (pts (xy 107.95 87.63) (xy 107.95 90.17)) (stroke (width 0) (type default)))
-  (wire (pts (xy 99.06 96.52) (xy 110.49 96.52)) (stroke (width 0) (type default)))
-  (global_label "~{HSYNC}" (shape output) (at 110.49 96.52 0) (fields_autoplaced) (effects (font (size 2 2)) (justify left)) (property "Intersheetrefs" "${INTERSHEET_REFS}" (at 110.49 96.52 0) (effects (font (size 2 2)) (justify left) hide)))
   (wire (pts (xy 99.06 101.6) (xy 109.22 101.6)) (stroke (width 0) (type default)))
   (wire (pts (xy 109.22 101.6) (xy 110.49 101.6)) (stroke (width 0) (type default)))
@@
   (wire (pts (xy 264.16 93.98) (xy 275.59 93.98)) (stroke (width 0) (type default)))
   (global_label "PIXEL_ENABLE" (shape output) (at 275.59 93.98 0) (fields_autoplaced) (effects (font (size 2 2)) (justify left)) (property "Intersheetrefs" "${INTERSHEET_REFS}" (at 275.59 93.98 0) (effects (font (size 2 2)) (justify left) hide)))
-  (wire (pts (xy 264.16 99.06) (xy 275.59 99.06)) (stroke (width 0) (type default)))
-  (global_label "~{VSYNC}" (shape output) (at 275.59 99.06 0) (fields_autoplaced) (effects (font (size 2 2)) (justify left)) (property "Intersheetrefs" "${INTERSHEET_REFS}" (at 275.59 99.06 0) (effects (font (size 2 2)) (justify left) hide)))
   (wire (pts (xy 264.16 111.76) (xy 275.59 111.76)) (stroke (width 0) (type default)))
   (global_label "ADDR_SEL" (shape output) (at 275.59 111.76 0) (fields_autoplaced) (effects (font (size 2 2)) (justify left)) (property "Intersheetrefs" "${INTERSHEET_REFS}" (at 275.59 111.76 0) (effects (font (size 2 2)) (justify left) hide)))
@@
   (bus (pts (xy 367.03 153.67) (xy 367.03 156.21)) (stroke (width 0) (type default)))
   (bus (pts (xy 367.03 156.21) (xy 367.03 158.75)) (stroke (width 0) (type default)))
+  (global_label "~{VGA_HSYNC}" (shape passive) (at 130.81 96.52 0) (fields_autoplaced) (effects (font (size 2 2)) (justify left)) (property "Intersheetrefs" "${INTERSHEET_REFS}" (at 130.81 96.52 0) (effects (font (size 2 2)) (justify left) hide)))
+  (global_label "~{VGA_VSYNC}" (shape passive) (at 323.85 99.06 0) (fields_autoplaced) (effects (font (size 2 2)) (justify left)) (property "Intersheetrefs" "${INTERSHEET_REFS}" (at 323.85 99.06 0) (effects (font (size 2 2)) (justify left) hide)))
   (bus (pts (xy 44.45 74.93) (xy 44.45 67.31)) (stroke (width 0) (type default)))
   (bus (pts (xy 44.45 67.31) (xy 40.64 67.31)) (stroke (width 0) (type default)))

Commit message: BOM/schematic: stocked substitutes from the first parts order
D18 Kingbright WP7113ID (LTL2R3KRD-EM out of stock), 100n TDK
FG28X7R1H104KNT00 (KEMET C320C104 $0.66 at Mouser), C45 TDK
FG24C0G1H153JNT06 (KEMET non-stocked), Vishay BAT85S-TAP and
1N4148-TAP, MF-RG300-0, USB4125-GF-A-0190; Mouser prices re-checked.

Co-Authored-By: Claude Opus 5.5 (1M context) <noreply@anthropic.com>
Claude-Session: https://claude.ai/code/session_017y5UgjExE8oeP7QrfvhCzb
Parts:
- C13, C14, C15, C29, C35: MPN C320C104K5R5TA -> FG28X7R1H104KNT00; Manufacturer KEMET -> TDK

Commit message: Put every symbol, footprint and 3D model in the project library
- gen_kicad_stock_footprints.py: copies of the KiCad 9.0.6 footprints the
  boards use (C_Disc, CP_Radial, DO-15/DO-35, LED, pin header, oscillator,
  TO-92, SIP9, mounting holes, net tie) into placard.pretty, and KiCad's
  STEP models for them and for the DIP socket / resistor kit footprints
  into placard.3dshapes
- model paths use the PLACARD_LIB text variable (main board
  ${KIPRJMOD}/lib, cartridges ${KIPRJMOD}/../lib) so the shared footprints
  find their models in all three projects
- placard_std gains the 28C256 EEPROM and the power symbols; symbol
  Footprint defaults name placard footprints (relay, SIP9, oscillator,
  TO-92, EEPROM socket)
- schematics regenerated with placard_std power/EEPROM symbols and
  placard: footprints; BOM CSVs and PDFs regenerated
- cartridge .kicad_pro files take in Justin's local KiCad 9 settings

Co-Authored-By: Claude Opus 5.5 <noreply@anthropic.com>
Claude-Session: https://claude.ai/code/session_017okF1JiLRNFTfH7Az85hff
Parts:
- C13, C14, C15, C29, C35: footprint Capacitor_THT:C_Disc_D5.0mm_W2.5mm_P5.00mm -> placard:C_Disc_D5.0mm_W2.5mm_P5.00mm
