File: kicad/power.kicad_sch (KiCad schematic)
At the start: 20 parts, among them J13 USB4125-GF-A, K1 G5LE-1 DC5, SW1 ANT11TFHQE, SW2 PTS645VL58-2 LFS, U40 MCP1700-3302E/TO, X1 25.175 MHz

Commit message: Add 3D models for the connectors, switches and polyfuse
Every connector/switch footprint in kicad/lib/placard.pretty now names a
STEP model in kicad/lib/placard.3dshapes via ${KIPRJMOD}, so the board shows
them in any KiCad version without a 3D library path.

- gen_kicad_3d_models.py (CadQuery) generates models at typical dimensions
  for J8 cart slot, J9-J12 expansion slots, J5 stacked PS/2, J6 audio jack,
  SW1 toggle, J4 SD socket, F1 polyfuse and J2/J3 SNES ports; leads are put
  on the footprint pads. KiCad's own models are copied for SW2, J7, J13.
- gen_kicad_connectors.py adds the model to its footprints and makes
  project copies of KiCad's SD, MF-RG300, PTS645 and DSUB-15-HD footprints
  (same pads) pointing at the project models; removes a duplicated block.
- Schematic, BOM and gen_kicad_pcb.py use the placard: copies for J4, J7,
  F1, SW2. kicad/placard.kicad_pcb is not touched.
- docs/connector_3d_models.png: KiCad STEP export of the footprints.

Co-Authored-By: Claude Opus 5.5 (1M context) <noreply@anthropic.com>
Claude-Session: https://claude.ai/code/session_011CYV6fCf1RGSdDoH9HuCKo
Parts:
- F1: footprint Fuse:Fuse_Bourns_MF-RG300 -> placard:Fuse_Bourns_MF-RG300
- SW2: footprint Button_Switch_THT:SW_Tactile_SPST_Angled_PTS645Vx58-2LFS -> placard:SW_Tactile_SPST_Angled_PTS645Vx58-2LFS
Changed lines of the file:
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@@
   (junction (at 71.12 96.52) (diameter 0) (color 0 0 0 0))
   (symbol (lib_id "power:GND") (at 71.12 101.6 0) (unit 1) (in_bom yes) (on_board yes) (dnp no) (property "Reference" "#PWR0201" (at 71.12 101.6 0) (effects (font (size 1.27 1.27)) hide)) (property "Value" "GND" (at 71.12 107.95 0) (effects (font (size 2 2)) hide)) (property "Footprint" "" (at 71.12 101.6 0) (effects (font (size 1.27 1.27)) hide)) (property "Datasheet" "" (at 71.12 101.6 0) (effects (font (size 1.27 1.27)) hide)) (pin "1") (instances (project "placard" (path "/e3450542-4ffc-59d4-a4a7-45636233928a/f2696644-57a6-5352-a354-a3e1bf43cc65" (reference "#PWR0201") (unit 1)))))
-  (symbol (lib_id "placard_std:Polyfuse") (at 91.44 81.28 90) (unit 1) (in_bom yes) (on_board yes) (dnp no) (property "Reference" "F1" (at 86.4 79.28 90) (effects (font (size 2.54 2.54) bold) (justify right top))) (property "Value" "3 A hold" (at 86.4 83.28 90) (effects (font (size 2 2)) (justify right bottom))) (property "Footprint" "Fuse:Fuse_Bourns_MF-RG300" (at 91.44 81.28 0) (effects (font (size 1.27 1.27)) hide)) (property "Datasheet" "~" (at 91.44 81.28 0) (effects (font (size 1.27 1.27)) hide)) (property "Manufacturer" "Bourns" (at 91.44 81.28 0) (effects (font (size 1.27 1.27)) hide)) (property "MPN" "MF-RG300" (at 91.44 81.28 0) (effects (font (size 1.27 1.27)) hide)) (pin "1") (pin "2") (instances (project "placard" (path "/e3450542-4ffc-59d4-a4a7-45636233928a/f2696644-57a6-5352-a354-a3e1bf43cc65" (reference "F1") (unit 1)))))
+  (symbol (lib_id "placard_std:Polyfuse") (at 91.44 81.28 90) (unit 1) (in_bom yes) (on_board yes) (dnp no) (property "Reference" "F1" (at 86.4 79.28 90) (effects (font (size 2.54 2.54) bold) (justify right top))) (property "Value" "3 A hold" (at 86.4 83.28 90) (effects (font (size 2 2)) (justify right bottom))) (property "Footprint" "placard:Fuse_Bourns_MF-RG300" (at 91.44 81.28 0) (effects (font (size 1.27 1.27)) hide)) (property "Datasheet" "~" (at 91.44 81.28 0) (effects (font (size 1.27 1.27)) hide)) (property "Manufacturer" "Bourns" (at 91.44 81.28 0) (effects (font (size 1.27 1.27)) hide)) (property "MPN" "MF-RG300" (at 91.44 81.28 0) (effects (font (size 1.27 1.27)) hide)) (pin "1") (pin "2") (instances (project "placard" (path "/e3450542-4ffc-59d4-a4a7-45636233928a/f2696644-57a6-5352-a354-a3e1bf43cc65" (reference "F1") (unit 1)))))
   (wire (pts (xy 68.58 81.28) (xy 87.63 81.28)) (stroke (width 0) (type default)))
   (symbol (lib_id "placard_std:SW_SPST") (at 124.46 81.28 0) (unit 1) (in_bom yes) (on_board yes) (dnp no) (property "Reference" "SW1" (at 119.8 76.68 0) (effects (font (size 2.54 2.54) bold) (justify left bottom))) (property "Value" "ANT11TFHQE" (at 118.5 83.88 0) (effects (font (size 2 2)) (justify left top))) (property "Footprint" "placard:SW_Toggle_CIT_ANT11TFHQE" (at 124.46 81.28 0) (effects (font (size 1.27 1.27)) hide)) (property "Datasheet" "~" (at 124.46 81.28 0) (effects (font (size 1.27 1.27)) hide)) (property "Manufacturer" "CIT Relay and Switch" (at 124.46 81.28 0) (effects (font (size 1.27 1.27)) hide)) (property "MPN" "ANT11TFHQE" (at 124.46 81.28 0) (effects (font (size 1.27 1.27)) hide)) (property "Description" "Power on/off: SPDT on-on toggle, 5 A 28 V DC, right-angle PCB, 1/4-40 bushing" (at 124.46 81.28 0) (effects (font (size 1.27 1.27)) hide)) (pin "1") (pin "2") (instances (project "placard" (path "/e3450542-4ffc-59d4-a4a7-45636233928a/f2696644-57a6-5352-a354-a3e1bf43cc65" (reference "SW1") (unit 1)))))
@@
   (no_connect (at 177.8 86.36))
   (symbol (lib_id "placard_std:G5LE-1") (at 170.18 78.74 270) (unit 1) (in_bom yes) (on_board yes) (dnp no) (property "Reference" "K1" (at 167.68 89.78 90) (effects (font (size 2.54 2.54) bold) (justify left bottom))) (property "Value" "G5LE-1 DC5" (at 167.68 92.28 90) (effects (font (size 2 2)) (justify left top))) (property "Footprint" "Relay_THT:Relay_SPDT_Omron-G5LE-1" (at 170.18 78.74 0) (effects (font (size 1.27 1.27)) hide)) (property "Datasheet" "http://www.omron.com/ecb/products/pdf/en-g5le.pdf" (at 170.18 78.74 0) (effects (font (size 1.27 1.27)) hide)) (property "Manufacturer" "Omron" (at 170.18 78.74 0) (effects (font (size 1.27 1.27)) hide)) (property "MPN" "G5LE-1 DC5" (at 170.18 78.74 0) (effects (font (size 1.27 1.27)) hide)) (pin "1") (pin "2") (pin "3") (pin "4") (pin "5") (instances (project "placard" (path "/e3450542-4ffc-59d4-a4a7-45636233928a/f2696644-57a6-5352-a354-a3e1bf43cc65" (reference "K1") (unit 1)))))
-  (symbol (lib_id "placard_std:SW_Push") (at 157.48 73.66 0) (unit 1) (in_bom yes) (on_board yes) (dnp no) (property "Reference" "SW2" (at 154.9 68.68 0) (effects (font (size 2.54 2.54) bold) (justify left bottom))) (property "Value" "PTS645VL58-2 LFS" (at 144.4 54.78 0) (effects (font (size 2 2)) (justify left top))) (property "Footprint" "Button_Switch_THT:SW_Tactile_SPST_Angled_PTS645Vx58-2LFS" (at 157.48 73.66 0) (effects (font (size 1.27 1.27)) hide)) (property "Datasheet" "~" (at 157.48 73.66 0) (effects (font (size 1.27 1.27)) hide)) (property "Manufacturer" "C&K" (at 157.48 73.66 0) (effects (font (size 1.27 1.27)) hide)) (property "MPN" "PTS645VL58-2 LFS" (at 157.48 73.66 0) (effects (font (size 1.27 1.27)) hide)) (pin "1") (pin "2") (instances (project "placard" (path "/e3450542-4ffc-59d4-a4a7-45636233928a/f2696644-57a6-5352-a354-a3e1bf43cc65" (reference "SW2") (unit 1)))))
+  (symbol (lib_id "placard_std:SW_Push") (at 157.48 73.66 0) (unit 1) (in_bom yes) (on_board yes) (dnp no) (property "Reference" "SW2" (at 154.9 68.68 0) (effects (font (size 2.54 2.54) bold) (justify left bottom))) (property "Value" "PTS645VL58-2 LFS" (at 144.4 54.78 0) (effects (font (size 2 2)) (justify left top))) (property "Footprint" "placard:SW_Tactile_SPST_Angled_PTS645Vx58-2LFS" (at 157.48 73.66 0) (effects (font (size 1.27 1.27)) hide)) (property "Datasheet" "~" (at 157.48 73.66 0) (effects (font (size 1.27 1.27)) hide)) (property "Manufacturer" "C&K" (at 157.48 73.66 0) (effects (font (size 1.27 1.27)) hide)) (property "MPN" "PTS645VL58-2 LFS" (at 157.48 73.66 0) (effects (font (size 1.27 1.27)) hide)) (pin "1") (pin "2") (instances (project "placard" (path "/e3450542-4ffc-59d4-a4a7-45636233928a/f2696644-57a6-5352-a354-a3e1bf43cc65" (reference "SW2") (unit 1)))))
   (symbol (lib_id "placard_std:D_Schottky") (at 170.18 63.5 0) (unit 1) (in_bom yes) (on_board yes) (dnp no) (property "Reference" "D8" (at 163.18 60.3 0) (effects (font (size 2.54 2.54) bold) (justify left bottom))) (property "Value" "BAT85" (at 171.18 60.3 0) (effects (font (size 2 2)) (justify left top))) (property "Footprint" "Diode_THT:D_DO-35_SOD27_P7.62mm_Horizontal" (at 170.18 63.5 0) (effects (font (size 1.27 1.27)) hide)) (property "Datasheet" "~" (at 170.18 63.5 0) (effects (font (size 1.27 1.27)) hide)) (property "Manufacturer" "Vishay" (at 170.18 63.5 0) (effects (font (size 1.27 1.27)) hide)) (property "MPN" "BAT85" (at 170.18 63.5 0) (effects (font (size 1.27 1.27)) hide)) (pin "1") (pin "2") (instances (project "placard" (path "/e3450542-4ffc-59d4-a4a7-45636233928a/f2696644-57a6-5352-a354-a3e1bf43cc65" (reference "D8") (unit 1)))))
   (wire (pts (xy 142.24 88.9) (xy 142.24 91.44)) (stroke (width 0) (type default)))
