File: kicad/power.kicad_sch (KiCad schematic)
At the start: 20 parts, among them J13 USB4125-GF-A, K1 G5LE-1 DC5, SW1 ANT11TFHQE, SW2 PTS645VL58-2 LFS, U40 MCP1700-3302E/TO, X1 25.175 MHz

Commit message: Add power LED D18 + R59 on +5V after the reset relay
Green 3 mm Lite-On LTL-4231N with a 1k resistor (about 3 mA) on the
power sheet, so it goes dark while the reset button holds K1 in.
Adds Device:LED to placard_std, the part to the BOM, and the LED to
BRINGUP.md step 1 and SCHEMATIC_PLAN.md.

Co-Authored-By: Claude Opus 5.5 (1M context) <noreply@anthropic.com>
Claude-Session: https://claude.ai/code/session_01NLo1PnnNYQvqfKJdgiTTV9
Parts:
- added D18: LTL-4231N, LED_THT:LED_D3.0mm, symbol placard_std:LED
- added R59: 1k, placard:R_Axial_DIN0207_L6.3mm_D2.5mm_P10.16mm_Horizontal_Value, symbol placard_std:R_US
Connections:
- net +5V: now also R59.1
- net GND: now also D18.1 (K)
- new net: D18.2 (A), R59.2
Other:
- note added: "D18 power LED (green, 3 mm) on +5V,"
- note added: "R59 1k: about 3 mA."
- note added: "after K1: dark while reset is held."

Commit message: Power LED D18: Lite-On LTL2R3KRD-EM, red 5 mm
Justin wants a larger LED. Footprint LED_THT:LED_D5.0mm; R59 stays 1k
(about 3 mA at 1.9 V). BOM, BRINGUP.md, SCHEMATIC_PLAN.md and the PDFs
follow.

Co-Authored-By: Claude Opus 5.5 (1M context) <noreply@anthropic.com>
Claude-Session: https://claude.ai/code/session_01NLo1PnnNYQvqfKJdgiTTV9
Parts:
- D18: value LTL-4231N -> LTL2R3KRD-EM; footprint LED_THT:LED_D3.0mm -> LED_THT:LED_D5.0mm; MPN LTL-4231N -> LTL2R3KRD-EM
Other:
- note added: "D18 power LED (red, 5 mm) on +5V,"
- note removed: "D18 power LED (green, 3 mm) on +5V,"
Changed lines of the file:
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@@
 (kicad_sch (version 20230121) (generator eeschema)
   (paper "A3")
-  (title_block (title "Placard: Power and clock") (date "2026-10-24") (rev "1") (company "Placard computer") (comment 1 "Generated by src/scripts/gen_kicad_schematic.py; plan in docs/SCHEMATIC_PLAN.md") (comment 2 "Chip numbers U1-U40 = docs/CHIPS.md; decoupling Cn goes with Un"))
+  (title_block (title "Placard: Power and clock") (date "2026-10-25") (rev "1") (company "Placard computer") (comment 1 "Generated by src/scripts/gen_kicad_schematic.py; plan in docs/SCHEMATIC_PLAN.md") (comment 2 "Chip numbers U1-U40 = docs/CHIPS.md; decoupling Cn goes with Un"))
   (text "Power and clock" (at 15 22 0) (effects (font (size 6 6) bold) (justify left bottom)))
   (text "USB-C 5 V in, 3.3 V for the SD card, 25.175 MHz oscillator (CLK), cartridge STALL and RUN" (at 15 30 0) (effects (font (size 3 3)) (justify left bottom)))
@@
   (symbol (lib_id "power:+5V") (at 304.8 78.74 0) (unit 1) (in_bom yes) (on_board yes) (dnp no) (property "Reference" "#PWR0214" (at 304.8 78.74 0) (effects (font (size 1.27 1.27)) hide)) (property "Value" "+5V" (at 304.8 72.39 0) (effects (font (size 2 2)))) (property "Footprint" "" (at 304.8 78.74 0) (effects (font (size 1.27 1.27)) hide)) (property "Datasheet" "" (at 304.8 78.74 0) (effects (font (size 1.27 1.27)) hide)) (pin "1") (instances (project "placard" (path "/e3450542-4ffc-59d4-a4a7-45636233928a/f2696644-57a6-5352-a354-a3e1bf43cc65" (reference "#PWR0214") (unit 1)))))
   (symbol (lib_id "placard_std:R_US") (at 304.8 88.9 0) (unit 1) (in_bom yes) (on_board yes) (dnp no) (property "Reference" "R59" (at 306.8 88.4 0) (effects (font (size 2.54 2.54) bold) (justify left bottom))) (property "Value" "1k" (at 306.8 91.5 0) (effects (font (size 2 2)) (justify left top))) (property "Footprint" "placard:R_Axial_DIN0207_L6.3mm_D2.5mm_P10.16mm_Horizontal_Value" (at 304.8 88.9 0) (effects (font (size 1.27 1.27)) hide)) (property "Datasheet" "~" (at 304.8 88.9 0) (effects (font (size 1.27 1.27)) hide)) (property "Manufacturer" "Yageo" (at 304.8 88.9 0) (effects (font (size 1.27 1.27)) hide)) (property "MPN" "MFR-25FBF52-1K" (at 304.8 88.9 0) (effects (font (size 1.27 1.27)) hide)) (pin "1") (pin "2") (instances (project "placard" (path "/e3450542-4ffc-59d4-a4a7-45636233928a/f2696644-57a6-5352-a354-a3e1bf43cc65" (reference "R59") (unit 1)))))
-  (symbol (lib_id "placard_std:LED") (at 304.8 104.14 90) (unit 1) (in_bom yes) (on_board yes) (dnp no) (property "Reference" "D18" (at 307.8 103.58 90) (effects (font (size 2.54 2.54) bold) (justify right top))) (property "Value" "LTL-4231N" (at 307.8 106.68 90) (effects (font (size 2 2)) (justify right bottom))) (property "Footprint" "LED_THT:LED_D3.0mm" (at 304.8 104.14 0) (effects (font (size 1.27 1.27)) hide)) (property "Datasheet" "~" (at 304.8 104.14 0) (effects (font (size 1.27 1.27)) hide)) (property "Manufacturer" "Lite-On" (at 304.8 104.14 0) (effects (font (size 1.27 1.27)) hide)) (property "MPN" "LTL-4231N" (at 304.8 104.14 0) (effects (font (size 1.27 1.27)) hide)) (pin "1") (pin "2") (instances (project "placard" (path "/e3450542-4ffc-59d4-a4a7-45636233928a/f2696644-57a6-5352-a354-a3e1bf43cc65" (reference "D18") (unit 1)))))
+  (symbol (lib_id "placard_std:LED") (at 304.8 104.14 90) (unit 1) (in_bom yes) (on_board yes) (dnp no) (property "Reference" "D18" (at 307.8 103.58 90) (effects (font (size 2.54 2.54) bold) (justify right top))) (property "Value" "LTL2R3KRD-EM" (at 307.8 106.68 90) (effects (font (size 2 2)) (justify right bottom))) (property "Footprint" "LED_THT:LED_D5.0mm" (at 304.8 104.14 0) (effects (font (size 1.27 1.27)) hide)) (property "Datasheet" "~" (at 304.8 104.14 0) (effects (font (size 1.27 1.27)) hide)) (property "Manufacturer" "Lite-On" (at 304.8 104.14 0) (effects (font (size 1.27 1.27)) hide)) (property "MPN" "LTL2R3KRD-EM" (at 304.8 104.14 0) (effects (font (size 1.27 1.27)) hide)) (pin "1") (pin "2") (instances (project "placard" (path "/e3450542-4ffc-59d4-a4a7-45636233928a/f2696644-57a6-5352-a354-a3e1bf43cc65" (reference "D18") (unit 1)))))
   (wire (pts (xy 304.8 78.74) (xy 304.8 85.09)) (stroke (width 0) (type default)))
   (wire (pts (xy 304.8 92.71) (xy 304.8 100.33)) (stroke (width 0) (type default)))
   (wire (pts (xy 304.8 107.95) (xy 304.8 110.49)) (stroke (width 0) (type default)))
   (symbol (lib_id "power:GND") (at 304.8 110.49 0) (unit 1) (in_bom yes) (on_board yes) (dnp no) (property "Reference" "#PWR0215" (at 304.8 110.49 0) (effects (font (size 1.27 1.27)) hide)) (property "Value" "GND" (at 304.8 116.84 0) (effects (font (size 2 2)) hide)) (property "Footprint" "" (at 304.8 110.49 0) (effects (font (size 1.27 1.27)) hide)) (property "Datasheet" "" (at 304.8 110.49 0) (effects (font (size 1.27 1.27)) hide)) (pin "1") (instances (project "placard" (path "/e3450542-4ffc-59d4-a4a7-45636233928a/f2696644-57a6-5352-a354-a3e1bf43cc65" (reference "#PWR0215") (unit 1)))))
-  (text "D18 power LED (green, 3 mm) on +5V," (at 282 124 0) (effects (font (size 2.5 2.5)) (justify left bottom)))
+  (text "D18 power LED (red, 5 mm) on +5V," (at 282 124 0) (effects (font (size 2.5 2.5)) (justify left bottom)))
   (text "after K1: dark while reset is held." (at 282 128 0) (effects (font (size 2.5 2.5)) (justify left bottom)))
   (text "R59 1k: about 3 mA." (at 282 132 0) (effects (font (size 2.5 2.5)) (justify left bottom)))

Commit message: Carry the PS/2 receiver PLD and the dropped matrix keyboard through the design
The matrix keyboard (U37, U39, J1, RN2, the keyboard board) is gone and the
PS/2 receiver PLD U42 (ATF22V10_PS2.pld rev 02) is added everywhere except
the hand-edited board layout:

- Drivers: receiver-based kbd_scan / mouse_poll / ps2_poll, PS2_LSN listened
  device, ps2_pause waits for a half-received mouse byte and holds the line
  at least 100 us; pad_read frees the mouse clock only briefly.
- Simulator: PS/2 keyboard and mouse models with abort/resend; tests pass.
- Bring-up ROM polls the PS/2 keyboard; BRINGUP.md step 18 rewritten.
- FPGA: port_pld rev 04, new ps2_pld, basys_top wired to both, matrix gone.
- Schematic: shared port sheet redrawn (U38, U42, D1/D4/D5/D19, R60),
  keyboard project, key switch footprints and header removed, C42 -> C47,
  PDFs and I/O PNG regenerated (netlist and ERC clean).
- BOM: keyboard board removed, U42 and C42 added; main board $184.77.
- Docs: IO, CHIPS, PLD_USAGE, LIBRARY, MENU, SCHEMATIC_PLAN, KITTING,
  EXPANSION, ROM, README, kicad README; dated notes in KIT_PRICING and CASE
  (keyboard kit and keyboard bay are moot, re-cost and case rethink pending).
- Block diagram regenerated (33 chips).

Co-Authored-By: Claude Fable 5.1 <noreply@anthropic.com>
Claude-Session: https://claude.ai/code/session_01QpoMmygNy6VSnJkmoq279r
Parts:
- renumbered C42 to C47
Other:
- note added: "C40 input, C47 output (1 uF ceramic)."
- note removed: "C40 input, C42 output (1 uF ceramic)."
Changed lines of the file:
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@@
   (wire (pts (xy 254 88.9) (xy 254 91.44)) (stroke (width 0) (type default)))
   (symbol (lib_id "power:GND") (at 254 91.44 0) (unit 1) (in_bom yes) (on_board yes) (dnp no) (property "Reference" "#PWR0211" (at 254 91.44 0) (effects (font (size 1.27 1.27)) hide)) (property "Value" "GND" (at 254 97.79 0) (effects (font (size 2 2)) hide)) (property "Footprint" "" (at 254 91.44 0) (effects (font (size 1.27 1.27)) hide)) (property "Datasheet" "" (at 254 91.44 0) (effects (font (size 1.27 1.27)) hide)) (pin "1") (instances (project "placard" (path "/e3450542-4ffc-59d4-a4a7-45636233928a/f2696644-57a6-5352-a354-a3e1bf43cc65" (reference "#PWR0211") (unit 1)))))
-  (symbol (lib_id "placard_std:C") (at 254 85.09 0) (unit 1) (in_bom yes) (on_board yes) (dnp no) (property "Reference" "C42" (at 256.5 84.58 0) (effects (font (size 2.54 2.54) bold) (justify left bottom))) (property "Value" "1u" (at 256.5 87.68 0) (effects (font (size 2 2)) (justify left top))) (property "Footprint" "Capacitor_THT:C_Disc_D5.0mm_W2.5mm_P5.00mm" (at 254 85.09 0) (effects (font (size 1.27 1.27)) hide)) (property "Datasheet" "~" (at 254 85.09 0) (effects (font (size 1.27 1.27)) hide)) (property "Manufacturer" "KEMET" (at 254 85.09 0) (effects (font (size 1.27 1.27)) hide)) (property "MPN" "C330C105K5R5TA" (at 254 85.09 0) (effects (font (size 1.27 1.27)) hide)) (pin "1") (pin "2") (instances (project "placard" (path "/e3450542-4ffc-59d4-a4a7-45636233928a/f2696644-57a6-5352-a354-a3e1bf43cc65" (reference "C42") (unit 1)))))
+  (symbol (lib_id "placard_std:C") (at 254 85.09 0) (unit 1) (in_bom yes) (on_board yes) (dnp no) (property "Reference" "C47" (at 256.5 84.58 0) (effects (font (size 2.54 2.54) bold) (justify left bottom))) (property "Value" "1u" (at 256.5 87.68 0) (effects (font (size 2 2)) (justify left top))) (property "Footprint" "Capacitor_THT:C_Disc_D5.0mm_W2.5mm_P5.00mm" (at 254 85.09 0) (effects (font (size 1.27 1.27)) hide)) (property "Datasheet" "~" (at 254 85.09 0) (effects (font (size 1.27 1.27)) hide)) (property "Manufacturer" "KEMET" (at 254 85.09 0) (effects (font (size 1.27 1.27)) hide)) (property "MPN" "C330C105K5R5TA" (at 254 85.09 0) (effects (font (size 1.27 1.27)) hide)) (pin "1") (pin "2") (instances (project "placard" (path "/e3450542-4ffc-59d4-a4a7-45636233928a/f2696644-57a6-5352-a354-a3e1bf43cc65" (reference "C47") (unit 1)))))
   (wire (pts (xy 246.38 81.28) (xy 254 81.28)) (stroke (width 0) (type default)))
   (wire (pts (xy 254 81.28) (xy 264.16 81.28)) (stroke (width 0) (type default)))
@@
   (text "whose NC contact opens the 5 V line." (at 25 142 0) (effects (font (size 2.5 2.5)) (justify left bottom)))
   (text "U40: 3.3 V for the SD card only (sheet 10)." (at 200 112 0) (effects (font (size 2.5 2.5)) (justify left bottom)))
-  (text "C40 input, C42 output (1 uF ceramic)." (at 200 116 0) (effects (font (size 2.5 2.5)) (justify left bottom)))
+  (text "C40 input, C47 output (1 uF ceramic)." (at 200 116 0) (effects (font (size 2.5 2.5)) (justify left bottom)))
   (symbol (lib_id "power:+5V") (at 304.8 78.74 0) (unit 1) (in_bom yes) (on_board yes) (dnp no) (property "Reference" "#PWR0214" (at 304.8 78.74 0) (effects (font (size 1.27 1.27)) hide)) (property "Value" "+5V" (at 304.8 72.39 0) (effects (font (size 2 2)))) (property "Footprint" "" (at 304.8 78.74 0) (effects (font (size 1.27 1.27)) hide)) (property "Datasheet" "" (at 304.8 78.74 0) (effects (font (size 1.27 1.27)) hide)) (pin "1") (instances (project "placard" (path "/e3450542-4ffc-59d4-a4a7-45636233928a/f2696644-57a6-5352-a354-a3e1bf43cc65" (reference "#PWR0214") (unit 1)))))
   (symbol (lib_id "placard_std:R_US") (at 304.8 88.9 0) (unit 1) (in_bom yes) (on_board yes) (dnp no) (property "Reference" "R59" (at 306.8 88.4 0) (effects (font (size 2.54 2.54) bold) (justify left bottom))) (property "Value" "1k" (at 306.8 91.5 0) (effects (font (size 2 2)) (justify left top))) (property "Footprint" "placard:R_Axial_DIN0207_L6.3mm_D2.5mm_P10.16mm_Horizontal_Value" (at 304.8 88.9 0) (effects (font (size 1.27 1.27)) hide)) (property "Datasheet" "~" (at 304.8 88.9 0) (effects (font (size 1.27 1.27)) hide)) (property "Manufacturer" "Yageo" (at 304.8 88.9 0) (effects (font (size 1.27 1.27)) hide)) (property "MPN" "MFR-25FBF52-1K" (at 304.8 88.9 0) (effects (font (size 1.27 1.27)) hide)) (pin "1") (pin "2") (instances (project "placard" (path "/e3450542-4ffc-59d4-a4a7-45636233928a/f2696644-57a6-5352-a354-a3e1bf43cc65" (reference "R59") (unit 1)))))

Commit message: BOM/schematic: stocked substitutes from the first parts order
D18 Kingbright WP7113ID (LTL2R3KRD-EM out of stock), 100n TDK
FG28X7R1H104KNT00 (KEMET C320C104 $0.66 at Mouser), C45 TDK
FG24C0G1H153JNT06 (KEMET non-stocked), Vishay BAT85S-TAP and
1N4148-TAP, MF-RG300-0, USB4125-GF-A-0190; Mouser prices re-checked.

Co-Authored-By: Claude Opus 5.5 (1M context) <noreply@anthropic.com>
Claude-Session: https://claude.ai/code/session_017y5UgjExE8oeP7QrfvhCzb
Parts:
- C43: MPN C320C104K5R5TA -> FG28X7R1H104KNT00; Manufacturer KEMET -> TDK
- D18: value LTL2R3KRD-EM -> WP7113ID; MPN LTL2R3KRD-EM -> WP7113ID; Manufacturer Lite-On -> Kingbright
- D8: MPN BAT85 -> BAT85S-TAP
- F1: MPN MF-RG300 -> MF-RG300-0
- J13: MPN USB4125-GF-A -> USB4125-GF-A-0190

Commit message: K1: CIT J1071CS5VDC.36 replaces Omron G5LE-1 DC5
Same pin pattern and numbering as the G5LE (1 COM, 2/5 coil, 3 NO, 4 NC),
checked against the J107 bottom-view drawing. 7 A 30 V DC on NO and NC,
69 ohm 0.36 W coil (72 mA), sealed, through hole, $1.15 at Digi-Key.
New footprint placard:Relay_SPDT_CIT_J107 (same pads, smaller body,
1.4 mm COM hole) and 3D model; schematic, BOM, BRINGUP, SCHEMATIC_PLAN,
KITTING updated.

Co-Authored-By: Claude Opus 5.5 (1M context) <noreply@anthropic.com>
Claude-Session: https://claude.ai/code/session_01Te7NqPPYZrwzVnj3a1FyWV
Parts:
- K1: value G5LE-1 DC5 -> J1071CS5VDC.36; footprint Relay_THT:Relay_SPDT_Omron-G5LE-1 -> placard:Relay_SPDT_CIT_J107; MPN G5LE-1 DC5 -> J1071CS5VDC.36; Manufacturer Omron -> CIT Relay and Switch
Changed lines of the file:
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@@
   (junction (at 104.14 81.28) (diameter 0) (color 0 0 0 0))
   (no_connect (at 177.8 86.36))
-  (symbol (lib_id "placard_std:G5LE-1") (at 170.18 78.74 270) (unit 1) (in_bom yes) (on_board yes) (dnp no) (property "Reference" "K1" (at 167.68 89.78 90) (effects (font (size 2.54 2.54) bold) (justify left bottom))) (property "Value" "G5LE-1 DC5" (at 167.68 92.28 90) (effects (font (size 2 2)) (justify left top))) (property "Footprint" "Relay_THT:Relay_SPDT_Omron-G5LE-1" (at 170.18 78.74 0) (effects (font (size 1.27 1.27)) hide)) (property "Datasheet" "http://www.omron.com/ecb/products/pdf/en-g5le.pdf" (at 170.18 78.74 0) (effects (font (size 1.27 1.27)) hide)) (property "Manufacturer" "Omron" (at 170.18 78.74 0) (effects (font (size 1.27 1.27)) hide)) (property "MPN" "G5LE-1 DC5" (at 170.18 78.74 0) (effects (font (size 1.27 1.27)) hide)) (pin "1") (pin "2") (pin "3") (pin "4") (pin "5") (instances (project "placard" (path "/e3450542-4ffc-59d4-a4a7-45636233928a/f2696644-57a6-5352-a354-a3e1bf43cc65" (reference "K1") (unit 1)))))
+  (symbol (lib_id "placard_std:G5LE-1") (at 170.18 78.74 270) (unit 1) (in_bom yes) (on_board yes) (dnp no) (property "Reference" "K1" (at 167.68 89.78 90) (effects (font (size 2.54 2.54) bold) (justify left bottom))) (property "Value" "J1071CS5VDC.36" (at 167.68 92.28 90) (effects (font (size 2 2)) (justify left top))) (property "Footprint" "placard:Relay_SPDT_CIT_J107" (at 170.18 78.74 0) (effects (font (size 1.27 1.27)) hide)) (property "Datasheet" "http://www.omron.com/ecb/products/pdf/en-g5le.pdf" (at 170.18 78.74 0) (effects (font (size 1.27 1.27)) hide)) (property "Manufacturer" "CIT Relay and Switch" (at 170.18 78.74 0) (effects (font (size 1.27 1.27)) hide)) (property "MPN" "J1071CS5VDC.36" (at 170.18 78.74 0) (effects (font (size 1.27 1.27)) hide)) (pin "1") (pin "2") (pin "3") (pin "4") (pin "5") (instances (project "placard" (path "/e3450542-4ffc-59d4-a4a7-45636233928a/f2696644-57a6-5352-a354-a3e1bf43cc65" (reference "K1") (unit 1)))))
   (symbol (lib_id "placard_std:SW_Push") (at 157.48 73.66 0) (unit 1) (in_bom yes) (on_board yes) (dnp no) (property "Reference" "SW2" (at 154.9 68.68 0) (effects (font (size 2.54 2.54) bold) (justify left bottom))) (property "Value" "PTS645VL58-2 LFS" (at 144.4 54.78 0) (effects (font (size 2 2)) (justify left top))) (property "Footprint" "placard:SW_Tactile_SPST_Angled_PTS645Vx58-2LFS" (at 157.48 73.66 0) (effects (font (size 1.27 1.27)) hide)) (property "Datasheet" "~" (at 157.48 73.66 0) (effects (font (size 1.27 1.27)) hide)) (property "Manufacturer" "C&K" (at 157.48 73.66 0) (effects (font (size 1.27 1.27)) hide)) (property "MPN" "PTS645VL58-2 LFS" (at 157.48 73.66 0) (effects (font (size 1.27 1.27)) hide)) (pin "1") (pin "2") (instances (project "placard" (path "/e3450542-4ffc-59d4-a4a7-45636233928a/f2696644-57a6-5352-a354-a3e1bf43cc65" (reference "SW2") (unit 1)))))
   (symbol (lib_id "placard_std:D_Schottky") (at 170.18 63.5 0) (unit 1) (in_bom yes) (on_board yes) (dnp no) (property "Reference" "D8" (at 163.18 60.3 0) (effects (font (size 2.54 2.54) bold) (justify left bottom))) (property "Value" "BAT85" (at 171.18 60.3 0) (effects (font (size 2 2)) (justify left top))) (property "Footprint" "Diode_THT:D_DO-35_SOD27_P7.62mm_Horizontal" (at 170.18 63.5 0) (effects (font (size 1.27 1.27)) hide)) (property "Datasheet" "~" (at 170.18 63.5 0) (effects (font (size 1.27 1.27)) hide)) (property "Manufacturer" "Vishay" (at 170.18 63.5 0) (effects (font (size 1.27 1.27)) hide)) (property "MPN" "BAT85S-TAP" (at 170.18 63.5 0) (effects (font (size 1.27 1.27)) hide)) (pin "1") (pin "2") (instances (project "placard" (path "/e3450542-4ffc-59d4-a4a7-45636233928a/f2696644-57a6-5352-a354-a3e1bf43cc65" (reference "D8") (unit 1)))))

Commit message: Put every symbol, footprint and 3D model in the project library
- gen_kicad_stock_footprints.py: copies of the KiCad 9.0.6 footprints the
  boards use (C_Disc, CP_Radial, DO-15/DO-35, LED, pin header, oscillator,
  TO-92, SIP9, mounting holes, net tie) into placard.pretty, and KiCad's
  STEP models for them and for the DIP socket / resistor kit footprints
  into placard.3dshapes
- model paths use the PLACARD_LIB text variable (main board
  ${KIPRJMOD}/lib, cartridges ${KIPRJMOD}/../lib) so the shared footprints
  find their models in all three projects
- placard_std gains the 28C256 EEPROM and the power symbols; symbol
  Footprint defaults name placard footprints (relay, SIP9, oscillator,
  TO-92, EEPROM socket)
- schematics regenerated with placard_std power/EEPROM symbols and
  placard: footprints; BOM CSVs and PDFs regenerated
- cartridge .kicad_pro files take in Justin's local KiCad 9 settings

Co-Authored-By: Claude Opus 5.5 <noreply@anthropic.com>
Claude-Session: https://claude.ai/code/session_017okF1JiLRNFTfH7Az85hff
Parts:
- C40, C43, C47: footprint Capacitor_THT:C_Disc_D5.0mm_W2.5mm_P5.00mm -> placard:C_Disc_D5.0mm_W2.5mm_P5.00mm
- C41: footprint Capacitor_THT:CP_Radial_D8.0mm_P3.50mm -> placard:CP_Radial_D8.0mm_P3.50mm
- D18: footprint LED_THT:LED_D5.0mm -> placard:LED_D5.0mm
- D7: footprint Diode_THT:D_DO-15_P10.16mm_Horizontal -> placard:D_DO-15_P10.16mm_Horizontal
- D8: footprint Diode_THT:D_DO-35_SOD27_P7.62mm_Horizontal -> placard:D_DO-35_SOD27_P7.62mm_Horizontal
- JP1, JP2: footprint Connector_PinHeader_2.54mm:PinHeader_1x02_P2.54mm_Vertical -> placard:PinHeader_1x02_P2.54mm_Vertical
- NT1: footprint NetTie:NetTie-2_THT_Pad0.3mm -> placard:NetTie-2_THT_Pad0.3mm
- U40: footprint Package_TO_SOT_THT:TO-92_Inline -> placard:TO-92_Inline
- X1: footprint Oscillator:Oscillator_DIP-14 -> placard:Oscillator_DIP-14
