File: kicad/power.kicad_sch (KiCad schematic)
At the start: 22 parts, among them J13 USB4125-GF-A, K1 J1071CS5VDC.36, SW1 ANT11TFHQE, SW2 PTS645VL58-2 LFS, U40 MCP1700-3302E/TO, X1 25.175 MHz

Commit message: Option B: muxes take the enables as selects, /WE from an early clock tap
Removes the Sync PLD pass from every memory address (docs/FETCH_TIMING.md):
the instruction fetch gains 8.2 ns, X/Y/video/upper-32K reads 9.7 ns, the
zero-page store start 6.9 ns, and the address hold after /WE is +0.5 ns
from the datasheets alone.  No new parts, no extra clock, no PLCC.

- ATF22V10_QUAD_MUX.pld rev 02: two low + two high address bits per chip,
  PIXEL_ENABLE / PC_ENABLE / X_ENABLE / Y_ENABLE as the selects
- ATF22V10_SYNC.pld rev 10: ADDR_SEL outputs gone; /WE on pin 20 from the
  early clock tap CLK_E (pin 9), RW and RUN inputs, OE = RUN
- ATF22V10_MEM_CTRL.pld rev 10: /WE gone (pin 16 free)
- ATF22V10_IO_DECODE.pld rev 05: /CE_HI from the enables, RW dropped
- FPGA model and benches follow; GHDL: tb_cart_load (2 seeds), tb_top_load,
  tb_blank_line pass, and cpu_test makes the same 69,776 RAM writes as main
- Schematic: mux sheet rewired, /WE from U15, net tie NT2 between CLK_E and
  CLK on the power sheet (the 500 mm of track), symbols regenerated, PDFs
- Docs updated; docs/option_b_board.png shows the board rewiring (no chip
  has to move)

Co-Authored-By: Claude Fable 5.1 <noreply@anthropic.com>
Claude-Session: https://claude.ai/code/session_01DnW5SSBUc8XDbr4GrYdwj8
Parts:
- added NT2: CLK tap, placard:NetTie-2_THT_Pad0.3mm, symbol placard_std:NetTie_2
Connections:
- net CLK: now also NT2.2; no longer X1.8 (OUT)
- new net CLK_E: NT2.1, X1.8 (OUT)
Other:
- note added: "NT2: CLK_E (X1, U15 pin 9) to CLK (every other chip) through"
- note added: "at least 420 mm of track (500 nominal): the RAM /WE's early clock."
Changed lines of the file:
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@@
   (symbol (lib_id "placard_std:GND") (at 81.28 163.83 0) (unit 1) (in_bom yes) (on_board yes) (dnp no) (property "Reference" "#PWR0223" (at 81.28 163.83 0) (effects (font (size 1.27 1.27)) hide)) (property "Value" "GND" (at 81.28 170.18 0) (effects (font (size 2 2)) hide)) (property "Footprint" "" (at 81.28 163.83 0) (effects (font (size 1.27 1.27)) hide)) (property "Datasheet" "" (at 81.28 163.83 0) (effects (font (size 1.27 1.27)) hide)) (pin "1") (instances (project "placard" (path "/e3450542-4ffc-59d4-a4a7-45636233928a/f2696644-57a6-5352-a354-a3e1bf43cc65" (reference "#PWR0223") (unit 1)))))
   (symbol (lib_id "placard_std:C") (at 81.28 160.02 0) (unit 1) (in_bom yes) (on_board yes) (dnp no) (property "Reference" "C43" (at 83.28 159.52 0) (effects (font (size 2.54 2.54) bold) (justify left bottom))) (property "Value" "100n" (at 83.28 162.62 0) (effects (font (size 2 2)) (justify left top))) (property "Footprint" "placard:C_Disc_D5.0mm_W2.5mm_P5.00mm" (at 81.28 160.02 0) (effects (font (size 1.27 1.27)) hide)) (property "Datasheet" "~" (at 81.28 160.02 0) (effects (font (size 1.27 1.27)) hide)) (property "Manufacturer" "TDK" (at 81.28 160.02 0) (effects (font (size 1.27 1.27)) hide)) (property "MPN" "FG28X7R1H104KNT00" (at 81.28 160.02 0) (effects (font (size 1.27 1.27)) hide)) (pin "1") (pin "2") (instances (project "placard" (path "/e3450542-4ffc-59d4-a4a7-45636233928a/f2696644-57a6-5352-a354-a3e1bf43cc65" (reference "C43") (unit 1)))))
+  (symbol (lib_id "placard_std:NetTie_2") (at 109.22 187.96 0) (unit 1) (in_bom no) (on_board yes) (dnp no) (property "Reference" "NT2" (at 104 181 0) (effects (font (size 2.54 2.54) bold) (justify left bottom))) (property "Value" "CLK tap" (at 104.5 194 0) (effects (font (size 2 2)) (justify left top))) (property "Footprint" "placard:NetTie-2_THT_Pad0.3mm" (at 109.22 187.96 0) (effects (font (size 1.27 1.27)) hide)) (property "Datasheet" "~" (at 109.22 187.96 0) (effects (font (size 1.27 1.27)) hide)) (pin "1") (pin "2") (instances (project "placard" (path "/e3450542-4ffc-59d4-a4a7-45636233928a/f2696644-57a6-5352-a354-a3e1bf43cc65" (reference "NT2") (unit 1)))))
+  (wire (pts (xy 106.68 187.96) (xy 102.87 187.96)) (stroke (width 0) (type default)))
+  (wire (pts (xy 102.87 187.96) (xy 101.6 187.96)) (stroke (width 0) (type default)))
+  (wire (pts (xy 111.76 187.96) (xy 116.84 187.96)) (stroke (width 0) (type default)))
+  (text "NT2: CLK_E (X1, U15 pin 9) to CLK (every other chip) through" (at 40 224 0) (effects (font (size 2.2 2.2)) (justify left bottom)))
+  (text "at least 420 mm of track (500 nominal): the RAM /WE's early clock." (at 40 227.52 0) (effects (font (size 2.2 2.2)) (justify left bottom)))
   (wire (pts (xy 152.4 156.21) (xy 152.4 153.67)) (stroke (width 0) (type default)))
   (symbol (lib_id "placard_std:+5V") (at 152.4 153.67 0) (unit 1) (in_bom yes) (on_board yes) (dnp no) (property "Reference" "#PWR0224" (at 152.4 153.67 0) (effects (font (size 1.27 1.27)) hide)) (property "Value" "+5V" (at 152.4 147.32 0) (effects (font (size 2 2)))) (property "Footprint" "" (at 152.4 153.67 0) (effects (font (size 1.27 1.27)) hide)) (property "Datasheet" "" (at 152.4 153.67 0) (effects (font (size 1.27 1.27)) hide)) (pin "1") (instances (project "placard" (path "/e3450542-4ffc-59d4-a4a7-45636233928a/f2696644-57a6-5352-a354-a3e1bf43cc65" (reference "#PWR0224") (unit 1)))))
@@
   (text "Without one, fit JP1 and JP2 for bring-up" (at 130 208 0) (effects (font (size 2.5 2.5)) (justify left bottom)))
   (text "(BRINGUP.md); take them out with a cartridge." (at 130 212 0) (effects (font (size 2.5 2.5)) (justify left bottom)))
-  (wire (pts (xy 76.2 170.18) (xy 81.28 170.18)) (stroke (width 0) (type default)))
-  (global_label "CLK" (shape output) (at 81.28 170.18 0) (fields_autoplaced) (effects (font (size 2 2)) (justify left)) (property "Intersheetrefs" "${INTERSHEET_REFS}" (at 81.28 170.18 0) (effects (font (size 2 2)) (justify left) hide)))
+  (wire (pts (xy 76.2 170.18) (xy 78.74 170.18)) (stroke (width 0) (type default)))
   (wire (pts (xy 134.62 170.18) (xy 129.54 170.18)) (stroke (width 0) (type default)))
   (global_label "STALL_IN" (shape passive) (at 129.54 170.18 180) (fields_autoplaced) (effects (font (size 2 2)) (justify right)) (property "Intersheetrefs" "${INTERSHEET_REFS}" (at 129.54 170.18 0) (effects (font (size 2 2)) (justify left) hide)))
+  (global_label "CLK_E" (shape passive) (at 101.6 187.96 180) (fields_autoplaced) (effects (font (size 2 2)) (justify right)) (property "Intersheetrefs" "${INTERSHEET_REFS}" (at 101.6 187.96 0) (effects (font (size 2 2)) (justify left) hide)))
+  (global_label "CLK" (shape passive) (at 116.84 187.96 0) (fields_autoplaced) (effects (font (size 2 2)) (justify left)) (property "Intersheetrefs" "${INTERSHEET_REFS}" (at 116.84 187.96 0) (effects (font (size 2 2)) (justify left) hide)))
   (global_label "STALL_OUT" (shape passive) (at 162.56 170.18 0) (fields_autoplaced) (effects (font (size 2 2)) (justify left)) (property "Intersheetrefs" "${INTERSHEET_REFS}" (at 162.56 170.18 0) (effects (font (size 2 2)) (justify left) hide)))
   (global_label "RUN" (shape passive) (at 226.06 170.18 180) (fields_autoplaced) (effects (font (size 2 2)) (justify right)) (property "Intersheetrefs" "${INTERSHEET_REFS}" (at 226.06 170.18 0) (effects (font (size 2 2)) (justify left) hide)))
+  (wire (pts (xy 78.74 170.18) (xy 102.87 170.18)) (stroke (width 0) (type default)))
+  (wire (pts (xy 102.87 170.18) (xy 102.87 187.96)) (stroke (width 0) (type default)))
+  (wire (pts (xy 102.87 187.96) (xy 101.6 187.96)) (stroke (width 0) (type default)))
+  (junction (at 102.87 187.96) (diameter 0) (color 0 0 0 0))
   (junction (at 152.4 170.18) (diameter 0) (color 0 0 0 0))
   (junction (at 236.22 170.18) (diameter 0) (color 0 0 0 0))

Commit message: C41 and C44: one part, Rubycon 25YXJ220M6.3X11
Both 220 uF electrolytics are now the Rubycon YXJ (25 V, 6.3 x 11 mm,
2.5 mm pitch), Justin's Digi-Key pick since Panasonic EEU-FR1C221 is out
of stock. C41 drops the 8 mm / 3.5 mm footprint (and its stale "10V"
label) for the 6.3 mm / 2.5 mm one C44 already uses. Schematic, BOM,
bring-up list and main PDF regenerated; check 0 problems.

Co-Authored-By: Claude Opus 5.5 <noreply@anthropic.com>
Claude-Session: https://claude.ai/code/session_01DnW5SUH9ixqxRrdF9j2pr2
Parts:
- C41: value 220u 10V -> 220u; footprint placard:CP_Radial_D8.0mm_P3.50mm -> placard:CP_Radial_D6.3mm_P2.50mm; MPN EEU-FR1E221 -> 25YXJ220M6.3X11; Manufacturer Panasonic -> Rubycon
Changed lines of the file:
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@@
   (wire (pts (xy 142.24 88.9) (xy 142.24 91.44)) (stroke (width 0) (type default)))
   (symbol (lib_id "placard_std:GND") (at 142.24 91.44 0) (unit 1) (in_bom yes) (on_board yes) (dnp no) (property "Reference" "#PWR0203" (at 142.24 91.44 0) (effects (font (size 1.27 1.27)) hide)) (property "Value" "GND" (at 142.24 97.79 0) (effects (font (size 2 2)) hide)) (property "Footprint" "" (at 142.24 91.44 0) (effects (font (size 1.27 1.27)) hide)) (property "Datasheet" "" (at 142.24 91.44 0) (effects (font (size 1.27 1.27)) hide)) (pin "1") (instances (project "placard" (path "/e3450542-4ffc-59d4-a4a7-45636233928a/f2696644-57a6-5352-a354-a3e1bf43cc65" (reference "#PWR0203") (unit 1)))))
-  (symbol (lib_id "placard_std:C_Polarized") (at 142.24 85.09 0) (unit 1) (in_bom yes) (on_board yes) (dnp no) (property "Reference" "C41" (at 144.7 84.58 0) (effects (font (size 2.54 2.54) bold) (justify left bottom))) (property "Value" "220u 10V" (at 144.7 87.68 0) (effects (font (size 2 2)) (justify left top))) (property "Footprint" "placard:CP_Radial_D8.0mm_P3.50mm" (at 142.24 85.09 0) (effects (font (size 1.27 1.27)) hide)) (property "Datasheet" "~" (at 142.24 85.09 0) (effects (font (size 1.27 1.27)) hide)) (property "Manufacturer" "Panasonic" (at 142.24 85.09 0) (effects (font (size 1.27 1.27)) hide)) (property "MPN" "EEU-FR1E221" (at 142.24 85.09 0) (effects (font (size 1.27 1.27)) hide)) (pin "1") (pin "2") (instances (project "placard" (path "/e3450542-4ffc-59d4-a4a7-45636233928a/f2696644-57a6-5352-a354-a3e1bf43cc65" (reference "C41") (unit 1)))))
+  (symbol (lib_id "placard_std:C_Polarized") (at 142.24 85.09 0) (unit 1) (in_bom yes) (on_board yes) (dnp no) (property "Reference" "C41" (at 144.7 84.58 0) (effects (font (size 2.54 2.54) bold) (justify left bottom))) (property "Value" "220u" (at 144.7 87.68 0) (effects (font (size 2 2)) (justify left top))) (property "Footprint" "placard:CP_Radial_D6.3mm_P2.50mm" (at 142.24 85.09 0) (effects (font (size 1.27 1.27)) hide)) (property "Datasheet" "~" (at 142.24 85.09 0) (effects (font (size 1.27 1.27)) hide)) (property "Manufacturer" "Rubycon" (at 142.24 85.09 0) (effects (font (size 1.27 1.27)) hide)) (property "MPN" "25YXJ220M6.3X11" (at 142.24 85.09 0) (effects (font (size 1.27 1.27)) hide)) (pin "1") (pin "2") (instances (project "placard" (path "/e3450542-4ffc-59d4-a4a7-45636233928a/f2696644-57a6-5352-a354-a3e1bf43cc65" (reference "C41") (unit 1)))))
   (wire (pts (xy 129.54 81.28) (xy 142.24 81.28)) (stroke (width 0) (type default)))
   (wire (pts (xy 142.24 81.28) (xy 152.4 81.28)) (stroke (width 0) (type default)))

Commit message: Schottkys to black 1N5817 (DO-41) so they differ from the glass 1N4148s
- D1-D6, D8-D11, D19: BAT85 -> MCC 1N5817-TP. 1N4148s (D12-D17) unchanged.
- New footprint D_DO-41_SOD81_P7.62mm_Horizontal_Pad1.6 (KiCad 9.0.6 DO-41
  at 7.62 mm, pads 1.6 mm / drill 1.0 mm): same copper as the DO-35 places,
  so Update PCB from Schematic swaps them without touching the routing;
  checked for courtyard overlaps and silk over pads on the board.
- Schematic, main PDF, BOM, BRINGUP ("Two kinds of diode"), KITTING, IO,
  VIDEO and COLORS updated.

Co-Authored-By: Claude Opus 5.5 <noreply@anthropic.com>
Claude-Session: https://claude.ai/code/session_01DnW5STXEXm5h75y8sthpiM
Parts:
- D8: value BAT85 -> 1N5817; footprint placard:D_DO-35_SOD27_P7.62mm_Horizontal -> placard:D_DO-41_SOD81_P7.62mm_Horizontal_Pad1.6; MPN BAT85S-TAP -> 1N5817-TP; Manufacturer Vishay -> Micro Commercial Co
Changed lines of the file:
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@@
   (symbol (lib_id "placard_std:G5LE-1") (at 170.18 78.74 270) (unit 1) (in_bom yes) (on_board yes) (dnp no) (property "Reference" "K1" (at 167.68 89.78 90) (effects (font (size 2.54 2.54) bold) (justify left bottom))) (property "Value" "J1071CS5VDC.36" (at 167.68 92.28 90) (effects (font (size 2 2)) (justify left top))) (property "Footprint" "placard:Relay_SPDT_CIT_J107" (at 170.18 78.74 0) (effects (font (size 1.27 1.27)) hide)) (property "Datasheet" "http://www.omron.com/ecb/products/pdf/en-g5le.pdf" (at 170.18 78.74 0) (effects (font (size 1.27 1.27)) hide)) (property "Manufacturer" "CIT Relay and Switch" (at 170.18 78.74 0) (effects (font (size 1.27 1.27)) hide)) (property "MPN" "J1071CS5VDC.36" (at 170.18 78.74 0) (effects (font (size 1.27 1.27)) hide)) (pin "1") (pin "2") (pin "3") (pin "4") (pin "5") (instances (project "placard" (path "/e3450542-4ffc-59d4-a4a7-45636233928a/f2696644-57a6-5352-a354-a3e1bf43cc65" (reference "K1") (unit 1)))))
   (symbol (lib_id "placard_std:SW_Push") (at 157.48 73.66 0) (unit 1) (in_bom yes) (on_board yes) (dnp no) (property "Reference" "SW2" (at 154.9 68.68 0) (effects (font (size 2.54 2.54) bold) (justify left bottom))) (property "Value" "PTS645VL58-2 LFS" (at 144.4 54.78 0) (effects (font (size 2 2)) (justify left top))) (property "Footprint" "placard:SW_Tactile_SPST_Angled_PTS645Vx58-2LFS" (at 157.48 73.66 0) (effects (font (size 1.27 1.27)) hide)) (property "Datasheet" "~" (at 157.48 73.66 0) (effects (font (size 1.27 1.27)) hide)) (property "Manufacturer" "C&K" (at 157.48 73.66 0) (effects (font (size 1.27 1.27)) hide)) (property "MPN" "PTS645VL58-2 LFS" (at 157.48 73.66 0) (effects (font (size 1.27 1.27)) hide)) (pin "1") (pin "2") (instances (project "placard" (path "/e3450542-4ffc-59d4-a4a7-45636233928a/f2696644-57a6-5352-a354-a3e1bf43cc65" (reference "SW2") (unit 1)))))
-  (symbol (lib_id "placard_std:D_Schottky") (at 170.18 63.5 0) (unit 1) (in_bom yes) (on_board yes) (dnp no) (property "Reference" "D8" (at 163.18 60.3 0) (effects (font (size 2.54 2.54) bold) (justify left bottom))) (property "Value" "BAT85" (at 171.18 60.3 0) (effects (font (size 2 2)) (justify left top))) (property "Footprint" "placard:D_DO-35_SOD27_P7.62mm_Horizontal" (at 170.18 63.5 0) (effects (font (size 1.27 1.27)) hide)) (property "Datasheet" "~" (at 170.18 63.5 0) (effects (font (size 1.27 1.27)) hide)) (property "Manufacturer" "Vishay" (at 170.18 63.5 0) (effects (font (size 1.27 1.27)) hide)) (property "MPN" "BAT85S-TAP" (at 170.18 63.5 0) (effects (font (size 1.27 1.27)) hide)) (pin "1") (pin "2") (instances (project "placard" (path "/e3450542-4ffc-59d4-a4a7-45636233928a/f2696644-57a6-5352-a354-a3e1bf43cc65" (reference "D8") (unit 1)))))
+  (symbol (lib_id "placard_std:D_Schottky") (at 170.18 63.5 0) (unit 1) (in_bom yes) (on_board yes) (dnp no) (property "Reference" "D8" (at 163.18 60.3 0) (effects (font (size 2.54 2.54) bold) (justify left bottom))) (property "Value" "1N5817" (at 171.18 60.3 0) (effects (font (size 2 2)) (justify left top))) (property "Footprint" "placard:D_DO-41_SOD81_P7.62mm_Horizontal_Pad1.6" (at 170.18 63.5 0) (effects (font (size 1.27 1.27)) hide)) (property "Datasheet" "~" (at 170.18 63.5 0) (effects (font (size 1.27 1.27)) hide)) (property "Manufacturer" "Micro Commercial Co" (at 170.18 63.5 0) (effects (font (size 1.27 1.27)) hide)) (property "MPN" "1N5817-TP" (at 170.18 63.5 0) (effects (font (size 1.27 1.27)) hide)) (pin "1") (pin "2") (instances (project "placard" (path "/e3450542-4ffc-59d4-a4a7-45636233928a/f2696644-57a6-5352-a354-a3e1bf43cc65" (reference "D8") (unit 1)))))
   (wire (pts (xy 142.24 88.9) (xy 142.24 91.44)) (stroke (width 0) (type default)))
   (symbol (lib_id "placard_std:GND") (at 142.24 91.44 0) (unit 1) (in_bom yes) (on_board yes) (dnp no) (property "Reference" "#PWR0203" (at 142.24 91.44 0) (effects (font (size 1.27 1.27)) hide)) (property "Value" "GND" (at 142.24 97.79 0) (effects (font (size 2 2)) hide)) (property "Footprint" "" (at 142.24 91.44 0) (effects (font (size 1.27 1.27)) hide)) (property "Datasheet" "" (at 142.24 91.44 0) (effects (font (size 1.27 1.27)) hide)) (pin "1") (instances (project "placard" (path "/e3450542-4ffc-59d4-a4a7-45636233928a/f2696644-57a6-5352-a354-a3e1bf43cc65" (reference "#PWR0203") (unit 1)))))

Commit message: Bring-up test points TP1-TP3 and the ICTC-MP test leads
TP1, TP2 (GND, Keystone 5011 black) and TP3 (+5V after K1, Keystone
5010 red) on the power sheet, for the bring-up test lead clips.  The
TestPoint symbol and KiCad's Keystone 5010-5014 footprint are copied
into the project library (KiCad 9.0.6 ships no model for it, so the
copy has no model line).  BOM lines added; BRINGUP.md step 1 fits the
loops and uses them, step 12 clips to TP1; KITTING.md names the leads
(Twin Industries ICTC-MP, Digi-Key 438-1157-ND).

Board placement is Justin's: proposed spots TP1 (122,159),
TP2 (334,209), TP3 (78.5,75.5).

Co-Authored-By: Claude Opus 5.5 <noreply@anthropic.com>
Claude-Session: https://claude.ai/code/session_01DnW5STJr9GacgH1VpgnfMB
Parts:
- added TP1, TP2: GND, placard:TestPoint_Keystone_5010-5014_Multipurpose, symbol placard_std:TestPoint
- added TP3: +5V, placard:TestPoint_Keystone_5010-5014_Multipurpose, symbol placard_std:TestPoint
Connections:
- net +5V: now also TP3.1
- net GND: now also TP1.1, TP2.1
Other:
- note added: "(red 5010): clip points for the bring-up test leads."
- note added: "TP1, TP2 GND (black Keystone 5011), TP3 +5V after K1"
Changed lines of the file:
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@@
   (text "Without one, fit JP1 and JP2 for bring-up" (at 130 208 0) (effects (font (size 2.5 2.5)) (justify left bottom)))
   (text "(BRINGUP.md); take them out with a cartridge." (at 130 212 0) (effects (font (size 2.5 2.5)) (justify left bottom)))
+  (symbol (lib_id "placard_std:TestPoint") (at 304.8 190.5 0) (unit 1) (in_bom yes) (on_board yes) (dnp no) (property "Reference" "TP1" (at 306.8 184.5 0) (effects (font (size 2.54 2.54) bold) (justify left bottom))) (property "Value" "GND" (at 306.8 187 0) (effects (font (size 2 2)) (justify left top))) (property "Footprint" "placard:TestPoint_Keystone_5010-5014_Multipurpose" (at 304.8 190.5 0) (effects (font (size 1.27 1.27)) hide)) (property "Datasheet" "~" (at 304.8 190.5 0) (effects (font (size 1.27 1.27)) hide)) (property "Manufacturer" "Keystone Electronics" (at 304.8 190.5 0) (effects (font (size 1.27 1.27)) hide)) (property "MPN" "5011" (at 304.8 190.5 0) (effects (font (size 1.27 1.27)) hide)) (property "Description" "PC test point, multipurpose loop, through-hole" (at 304.8 190.5 0) (effects (font (size 1.27 1.27)) hide)) (pin "1") (instances (project "placard" (path "/e3450542-4ffc-59d4-a4a7-45636233928a/f2696644-57a6-5352-a354-a3e1bf43cc65" (reference "TP1") (unit 1)))))
+  (wire (pts (xy 304.8 190.5) (xy 304.8 195.58)) (stroke (width 0) (type default)))
+  (symbol (lib_id "placard_std:GND") (at 304.8 195.58 0) (unit 1) (in_bom yes) (on_board yes) (dnp no) (property "Reference" "#PWR0227" (at 304.8 195.58 0) (effects (font (size 1.27 1.27)) hide)) (property "Value" "GND" (at 304.8 201.93 0) (effects (font (size 2 2)) hide)) (property "Footprint" "" (at 304.8 195.58 0) (effects (font (size 1.27 1.27)) hide)) (property "Datasheet" "" (at 304.8 195.58 0) (effects (font (size 1.27 1.27)) hide)) (pin "1") (instances (project "placard" (path "/e3450542-4ffc-59d4-a4a7-45636233928a/f2696644-57a6-5352-a354-a3e1bf43cc65" (reference "#PWR0227") (unit 1)))))
+  (symbol (lib_id "placard_std:TestPoint") (at 322.58 190.5 0) (unit 1) (in_bom yes) (on_board yes) (dnp no) (property "Reference" "TP2" (at 324.58 184.5 0) (effects (font (size 2.54 2.54) bold) (justify left bottom))) (property "Value" "GND" (at 324.58 187 0) (effects (font (size 2 2)) (justify left top))) (property "Footprint" "placard:TestPoint_Keystone_5010-5014_Multipurpose" (at 322.58 190.5 0) (effects (font (size 1.27 1.27)) hide)) (property "Datasheet" "~" (at 322.58 190.5 0) (effects (font (size 1.27 1.27)) hide)) (property "Manufacturer" "Keystone Electronics" (at 322.58 190.5 0) (effects (font (size 1.27 1.27)) hide)) (property "MPN" "5011" (at 322.58 190.5 0) (effects (font (size 1.27 1.27)) hide)) (property "Description" "PC test point, multipurpose loop, through-hole" (at 322.58 190.5 0) (effects (font (size 1.27 1.27)) hide)) (pin "1") (instances (project "placard" (path "/e3450542-4ffc-59d4-a4a7-45636233928a/f2696644-57a6-5352-a354-a3e1bf43cc65" (reference "TP2") (unit 1)))))
+  (wire (pts (xy 322.58 190.5) (xy 322.58 195.58)) (stroke (width 0) (type default)))
+  (symbol (lib_id "placard_std:GND") (at 322.58 195.58 0) (unit 1) (in_bom yes) (on_board yes) (dnp no) (property "Reference" "#PWR0228" (at 322.58 195.58 0) (effects (font (size 1.27 1.27)) hide)) (property "Value" "GND" (at 322.58 201.93 0) (effects (font (size 2 2)) hide)) (property "Footprint" "" (at 322.58 195.58 0) (effects (font (size 1.27 1.27)) hide)) (property "Datasheet" "" (at 322.58 195.58 0) (effects (font (size 1.27 1.27)) hide)) (pin "1") (instances (project "placard" (path "/e3450542-4ffc-59d4-a4a7-45636233928a/f2696644-57a6-5352-a354-a3e1bf43cc65" (reference "#PWR0228") (unit 1)))))
+  (symbol (lib_id "placard_std:TestPoint") (at 340.36 195.58 180) (unit 1) (in_bom yes) (on_board yes) (dnp no) (property "Reference" "TP3" (at 342.36 199.5 0) (effects (font (size 2.54 2.54) bold) (justify right top))) (property "Value" "+5V" (at 342.36 202 0) (effects (font (size 2 2)) (justify right bottom))) (property "Footprint" "placard:TestPoint_Keystone_5010-5014_Multipurpose" (at 340.36 195.58 0) (effects (font (size 1.27 1.27)) hide)) (property "Datasheet" "~" (at 340.36 195.58 0) (effects (font (size 1.27 1.27)) hide)) (property "Manufacturer" "Keystone Electronics" (at 340.36 195.58 0) (effects (font (size 1.27 1.27)) hide)) (property "MPN" "5010" (at 340.36 195.58 0) (effects (font (size 1.27 1.27)) hide)) (property "Description" "PC test point, multipurpose loop, through-hole" (at 340.36 195.58 0) (effects (font (size 1.27 1.27)) hide)) (pin "1") (instances (project "placard" (path "/e3450542-4ffc-59d4-a4a7-45636233928a/f2696644-57a6-5352-a354-a3e1bf43cc65" (reference "TP3") (unit 1)))))
+  (wire (pts (xy 340.36 190.5) (xy 340.36 195.58)) (stroke (width 0) (type default)))
+  (symbol (lib_id "placard_std:+5V") (at 340.36 190.5 0) (unit 1) (in_bom yes) (on_board yes) (dnp no) (property "Reference" "#PWR0229" (at 340.36 190.5 0) (effects (font (size 1.27 1.27)) hide)) (property "Value" "+5V" (at 340.36 184.15 0) (effects (font (size 2 2)))) (property "Footprint" "" (at 340.36 190.5 0) (effects (font (size 1.27 1.27)) hide)) (property "Datasheet" "" (at 340.36 190.5 0) (effects (font (size 1.27 1.27)) hide)) (pin "1") (instances (project "placard" (path "/e3450542-4ffc-59d4-a4a7-45636233928a/f2696644-57a6-5352-a354-a3e1bf43cc65" (reference "#PWR0229") (unit 1)))))
+  (text "TP1, TP2 GND (black Keystone 5011), TP3 +5V after K1" (at 296 216 0) (effects (font (size 2.2 2.2)) (justify left bottom)))
+  (text "(red 5010): clip points for the bring-up test leads." (at 296 219.52 0) (effects (font (size 2.2 2.2)) (justify left bottom)))
   (wire (pts (xy 76.2 170.18) (xy 78.74 170.18)) (stroke (width 0) (type default)))
   (wire (pts (xy 134.62 170.18) (xy 129.54 170.18)) (stroke (width 0) (type default)))
