File: kicad/control.kicad_sch (KiCad schematic)
At the start: 6 parts, among them U1 ATF22V10C-7PX, U17 ATF22V10C-7PX, U2 ATF22V10C-10PU

Commit message: Tidy every schematic sheet: spread parts, straight runs, buses kept, horizontal tabs
Shared port, expansion and cartridge sheets laid out by hand; buses from
other sheets get a bus label at each chip, busy control nets a label at
each pin; some PLD and connector symbols reordered so wires run straight;
sideways power symbols read across. 0 netlist problems, no overlaps.

Co-Authored-By: Claude Opus 5.5 (1M context) <noreply@anthropic.com>
Claude-Session: https://claude.ai/code/session_01L9AkLuEg13EebxDmgXsaEp
Connections:
- net Q0: now reaches U1.18 (Q0), U2.10 (Q0)
- net BRANCH_BLOCK: now reaches U1.8 (BRANCH_BLOCK), U2.23 (BRANCH_BLOCK)
Other:
- moved on the sheet: C1, C17, C2, U1, U17, U2

Commit message: Bill of materials for the main board, cartridge and keyboard
Manufacturer and MPN fields on every schematic part (empty where none is
chosen), set from an MPN table in gen_kicad_schematic.py; net tie, cartridge
edge fingers and solder jumper excluded from the BOM.  gen_bom.py groups the
parts by part number into docs/BOM.md and docs/BOM.csv, adding sockets,
shunts, keyboard LEDs, keycaps, stabilizers and the keyboard ribbon cable.

Co-Authored-By: Claude Opus 5.5 (1M context) <noreply@anthropic.com>
Claude-Session: https://claude.ai/code/session_018iEnPngycbxX6Tt4Wzp3zN
Parts:
- U1, U17: MPN (none) -> ATF22V10C-7PX; Manufacturer (none) -> Microchip
- U2: MPN (none) -> ATF22V10C-10PU; Manufacturer (none) -> Microchip

Commit message: Part numbers for the remaining parts; J6 Tensility 54-00174; optional J1 and J9-J12
Every schematic part gets Manufacturer/MPN: Yageo MFR-25 resistors by value,
Bourns 4609X networks, KEMET/TDK ceramics, Panasonic FR electrolytics, ECS
oscillator, Assmann VGA, Sullins headers, Wurth box header, Cherry switches.
Sockets get On Shore numbers (0.3" 24/28-pin are ED241DT/ED281DT; ED28DT is
0.6"). J6 becomes the Tensility 54-00174 TRRS jack with a footprint drawn
from its datasheet. Digi-Key prices from Justin for the oscillator, VGA and
audio jack. The expansion slot sockets and the keyboard header are optional,
with a BOM total without them.

Co-Authored-By: Claude Opus 5.5 (1M context) <noreply@anthropic.com>
Claude-Session: https://claude.ai/code/session_01L9AkLuEg13EebxDmgXsaEp
Parts:
- C1, C17, C2: MPN (none) -> C320C104K5R5TA; Manufacturer (none) -> KEMET
Changed lines of the file:
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@@
   (symbol (lib_id "power:+5V") (at 91.44 118.11 0) (unit 1) (in_bom yes) (on_board yes) (dnp no) (property "Reference" "#PWR0303" (at 91.44 118.11 0) (effects (font (size 1.27 1.27)) hide)) (property "Value" "+5V" (at 91.44 111.76 0) (effects (font (size 2 2)))) (property "Footprint" "" (at 91.44 118.11 0) (effects (font (size 1.27 1.27)) hide)) (property "Datasheet" "" (at 91.44 118.11 0) (effects (font (size 1.27 1.27)) hide)) (pin "1") (instances (project "placard" (path "/e3450542-4ffc-59d4-a4a7-45636233928a/370d9988-af17-5e05-8c50-5ef0ca792654" (reference "#PWR0303") (unit 1)))))
   (symbol (lib_id "power:GND") (at 91.44 125.73 0) (unit 1) (in_bom yes) (on_board yes) (dnp no) (property "Reference" "#PWR0304" (at 91.44 125.73 0) (effects (font (size 1.27 1.27)) hide)) (property "Value" "GND" (at 91.44 132.08 0) (effects (font (size 2 2)) hide)) (property "Footprint" "" (at 91.44 125.73 0) (effects (font (size 1.27 1.27)) hide)) (property "Datasheet" "" (at 91.44 125.73 0) (effects (font (size 1.27 1.27)) hide)) (pin "1") (instances (project "placard" (path "/e3450542-4ffc-59d4-a4a7-45636233928a/370d9988-af17-5e05-8c50-5ef0ca792654" (reference "#PWR0304") (unit 1)))))
-  (symbol (lib_id "placard_std:C") (at 91.44 121.92 0) (unit 1) (in_bom yes) (on_board yes) (dnp no) (property "Reference" "C17" (at 93.44 121.42 0) (effects (font (size 2.54 2.54) bold) (justify left bottom))) (property "Value" "100n" (at 93.44 124.52 0) (effects (font (size 2 2)) (justify left top))) (property "Footprint" "Capacitor_THT:C_Disc_D5.0mm_W2.5mm_P5.00mm" (at 91.44 121.92 0) (effects (font (size 1.27 1.27)) hide)) (property "Datasheet" "~" (at 91.44 121.92 0) (effects (font (size 1.27 1.27)) hide)) (property "Manufacturer" "" (at 91.44 121.92 0) (effects (font (size 1.27 1.27)) hide)) (property "MPN" "" (at 91.44 121.92 0) (effects (font (size 1.27 1.27)) hide)) (pin "1") (pin "2") (instances (project "placard" (path "/e3450542-4ffc-59d4-a4a7-45636233928a/370d9988-af17-5e05-8c50-5ef0ca792654" (reference "C17") (unit 1)))))
+  (symbol (lib_id "placard_std:C") (at 91.44 121.92 0) (unit 1) (in_bom yes) (on_board yes) (dnp no) (property "Reference" "C17" (at 93.44 121.42 0) (effects (font (size 2.54 2.54) bold) (justify left bottom))) (property "Value" "100n" (at 93.44 124.52 0) (effects (font (size 2 2)) (justify left top))) (property "Footprint" "Capacitor_THT:C_Disc_D5.0mm_W2.5mm_P5.00mm" (at 91.44 121.92 0) (effects (font (size 1.27 1.27)) hide)) (property "Datasheet" "~" (at 91.44 121.92 0) (effects (font (size 1.27 1.27)) hide)) (property "Manufacturer" "KEMET" (at 91.44 121.92 0) (effects (font (size 1.27 1.27)) hide)) (property "MPN" "C320C104K5R5TA" (at 91.44 121.92 0) (effects (font (size 1.27 1.27)) hide)) (pin "1") (pin "2") (instances (project "placard" (path "/e3450542-4ffc-59d4-a4a7-45636233928a/370d9988-af17-5e05-8c50-5ef0ca792654" (reference "C17") (unit 1)))))
   (wire (pts (xy 172.72 134.62) (xy 172.72 132.08)) (stroke (width 0) (type default)))
   (symbol (lib_id "power:+5V") (at 172.72 132.08 0) (unit 1) (in_bom yes) (on_board yes) (dnp no) (property "Reference" "#PWR0305" (at 172.72 132.08 0) (effects (font (size 1.27 1.27)) hide)) (property "Value" "+5V" (at 172.72 125.73 0) (effects (font (size 2 2)))) (property "Footprint" "" (at 172.72 132.08 0) (effects (font (size 1.27 1.27)) hide)) (property "Datasheet" "" (at 172.72 132.08 0) (effects (font (size 1.27 1.27)) hide)) (pin "1") (instances (project "placard" (path "/e3450542-4ffc-59d4-a4a7-45636233928a/370d9988-af17-5e05-8c50-5ef0ca792654" (reference "#PWR0305") (unit 1)))))
@@
   (symbol (lib_id "power:+5V") (at 193.04 123.19 0) (unit 1) (in_bom yes) (on_board yes) (dnp no) (property "Reference" "#PWR0307" (at 193.04 123.19 0) (effects (font (size 1.27 1.27)) hide)) (property "Value" "+5V" (at 193.04 116.84 0) (effects (font (size 2 2)))) (property "Footprint" "" (at 193.04 123.19 0) (effects (font (size 1.27 1.27)) hide)) (property "Datasheet" "" (at 193.04 123.19 0) (effects (font (size 1.27 1.27)) hide)) (pin "1") (instances (project "placard" (path "/e3450542-4ffc-59d4-a4a7-45636233928a/370d9988-af17-5e05-8c50-5ef0ca792654" (reference "#PWR0307") (unit 1)))))
   (symbol (lib_id "power:GND") (at 193.04 130.81 0) (unit 1) (in_bom yes) (on_board yes) (dnp no) (property "Reference" "#PWR0308" (at 193.04 130.81 0) (effects (font (size 1.27 1.27)) hide)) (property "Value" "GND" (at 193.04 137.16 0) (effects (font (size 2 2)) hide)) (property "Footprint" "" (at 193.04 130.81 0) (effects (font (size 1.27 1.27)) hide)) (property "Datasheet" "" (at 193.04 130.81 0) (effects (font (size 1.27 1.27)) hide)) (pin "1") (instances (project "placard" (path "/e3450542-4ffc-59d4-a4a7-45636233928a/370d9988-af17-5e05-8c50-5ef0ca792654" (reference "#PWR0308") (unit 1)))))
-  (symbol (lib_id "placard_std:C") (at 193.04 127 0) (unit 1) (in_bom yes) (on_board yes) (dnp no) (property "Reference" "C1" (at 195.04 126.5 0) (effects (font (size 2.54 2.54) bold) (justify left bottom))) (property "Value" "100n" (at 195.04 129.6 0) (effects (font (size 2 2)) (justify left top))) (property "Footprint" "Capacitor_THT:C_Disc_D5.0mm_W2.5mm_P5.00mm" (at 193.04 127 0) (effects (font (size 1.27 1.27)) hide)) (property "Datasheet" "~" (at 193.04 127 0) (effects (font (size 1.27 1.27)) hide)) (property "Manufacturer" "" (at 193.04 127 0) (effects (font (size 1.27 1.27)) hide)) (property "MPN" "" (at 193.04 127 0) (effects (font (size 1.27 1.27)) hide)) (pin "1") (pin "2") (instances (project "placard" (path "/e3450542-4ffc-59d4-a4a7-45636233928a/370d9988-af17-5e05-8c50-5ef0ca792654" (reference "C1") (unit 1)))))
+  (symbol (lib_id "placard_std:C") (at 193.04 127 0) (unit 1) (in_bom yes) (on_board yes) (dnp no) (property "Reference" "C1" (at 195.04 126.5 0) (effects (font (size 2.54 2.54) bold) (justify left bottom))) (property "Value" "100n" (at 195.04 129.6 0) (effects (font (size 2 2)) (justify left top))) (property "Footprint" "Capacitor_THT:C_Disc_D5.0mm_W2.5mm_P5.00mm" (at 193.04 127 0) (effects (font (size 1.27 1.27)) hide)) (property "Datasheet" "~" (at 193.04 127 0) (effects (font (size 1.27 1.27)) hide)) (property "Manufacturer" "KEMET" (at 193.04 127 0) (effects (font (size 1.27 1.27)) hide)) (property "MPN" "C320C104K5R5TA" (at 193.04 127 0) (effects (font (size 1.27 1.27)) hide)) (pin "1") (pin "2") (instances (project "placard" (path "/e3450542-4ffc-59d4-a4a7-45636233928a/370d9988-af17-5e05-8c50-5ef0ca792654" (reference "C1") (unit 1)))))
   (no_connect (at 322.58 144.78))
   (no_connect (at 322.58 149.86))
@@
   (symbol (lib_id "power:+5V") (at 314.96 90.17 0) (unit 1) (in_bom yes) (on_board yes) (dnp no) (property "Reference" "#PWR0311" (at 314.96 90.17 0) (effects (font (size 1.27 1.27)) hide)) (property "Value" "+5V" (at 314.96 83.82 0) (effects (font (size 2 2)))) (property "Footprint" "" (at 314.96 90.17 0) (effects (font (size 1.27 1.27)) hide)) (property "Datasheet" "" (at 314.96 90.17 0) (effects (font (size 1.27 1.27)) hide)) (pin "1") (instances (project "placard" (path "/e3450542-4ffc-59d4-a4a7-45636233928a/370d9988-af17-5e05-8c50-5ef0ca792654" (reference "#PWR0311") (unit 1)))))
   (symbol (lib_id "power:GND") (at 314.96 97.79 0) (unit 1) (in_bom yes) (on_board yes) (dnp no) (property "Reference" "#PWR0312" (at 314.96 97.79 0) (effects (font (size 1.27 1.27)) hide)) (property "Value" "GND" (at 314.96 104.14 0) (effects (font (size 2 2)) hide)) (property "Footprint" "" (at 314.96 97.79 0) (effects (font (size 1.27 1.27)) hide)) (property "Datasheet" "" (at 314.96 97.79 0) (effects (font (size 1.27 1.27)) hide)) (pin "1") (instances (project "placard" (path "/e3450542-4ffc-59d4-a4a7-45636233928a/370d9988-af17-5e05-8c50-5ef0ca792654" (reference "#PWR0312") (unit 1)))))
-  (symbol (lib_id "placard_std:C") (at 314.96 93.98 0) (unit 1) (in_bom yes) (on_board yes) (dnp no) (property "Reference" "C2" (at 316.96 93.48 0) (effects (font (size 2.54 2.54) bold) (justify left bottom))) (property "Value" "100n" (at 316.96 96.58 0) (effects (font (size 2 2)) (justify left top))) (property "Footprint" "Capacitor_THT:C_Disc_D5.0mm_W2.5mm_P5.00mm" (at 314.96 93.98 0) (effects (font (size 1.27 1.27)) hide)) (property "Datasheet" "~" (at 314.96 93.98 0) (effects (font (size 1.27 1.27)) hide)) (property "Manufacturer" "" (at 314.96 93.98 0) (effects (font (size 1.27 1.27)) hide)) (property "MPN" "" (at 314.96 93.98 0) (effects (font (size 1.27 1.27)) hide)) (pin "1") (pin "2") (instances (project "placard" (path "/e3450542-4ffc-59d4-a4a7-45636233928a/370d9988-af17-5e05-8c50-5ef0ca792654" (reference "C2") (unit 1)))))
+  (symbol (lib_id "placard_std:C") (at 314.96 93.98 0) (unit 1) (in_bom yes) (on_board yes) (dnp no) (property "Reference" "C2" (at 316.96 93.48 0) (effects (font (size 2.54 2.54) bold) (justify left bottom))) (property "Value" "100n" (at 316.96 96.58 0) (effects (font (size 2 2)) (justify left top))) (property "Footprint" "Capacitor_THT:C_Disc_D5.0mm_W2.5mm_P5.00mm" (at 314.96 93.98 0) (effects (font (size 1.27 1.27)) hide)) (property "Datasheet" "~" (at 314.96 93.98 0) (effects (font (size 1.27 1.27)) hide)) (property "Manufacturer" "KEMET" (at 314.96 93.98 0) (effects (font (size 1.27 1.27)) hide)) (property "MPN" "C320C104K5R5TA" (at 314.96 93.98 0) (effects (font (size 1.27 1.27)) hide)) (pin "1") (pin "2") (instances (project "placard" (path "/e3450542-4ffc-59d4-a4a7-45636233928a/370d9988-af17-5e05-8c50-5ef0ca792654" (reference "C2") (unit 1)))))
   (wire (pts (xy 198.12 139.7) (xy 266.7 139.7)) (stroke (width 0) (type default)))
   (wire (pts (xy 198.12 142.24) (xy 208.28 142.24)) (stroke (width 0) (type default)))

Commit message: Every PLD is an ATF22V10C-7PX (one part number)
Justin: switch the seven main-board -10PU PLDs (Branch, PC x2, H, V,
color decoder, audio slot) and the cartridge loader to the -7PX, for one
part number to buy, program and kit (.52 more per main board). Symbols,
schematics, PDFs, BOM, docs and PLD comments updated; CHIPS.md keeps the
grade each PLD could use.

Co-Authored-By: Claude Opus 5.5 (1M context) <noreply@anthropic.com>
Claude-Session: https://claude.ai/code/session_01JnVuvUvdWezUUU6Sgmg16H
Parts:
- U2: value ATF22V10C-10PU -> ATF22V10C-7PX; MPN ATF22V10C-10PU -> ATF22V10C-7PX
Changed lines of the file:
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@@
   (wire (pts (xy 294.64 154.94) (xy 294.64 157.48)) (stroke (width 0) (type default)))
   (symbol (lib_id "power:GND") (at 294.64 157.48 0) (unit 1) (in_bom yes) (on_board yes) (dnp no) (property "Reference" "#PWR0310" (at 294.64 157.48 0) (effects (font (size 1.27 1.27)) hide)) (property "Value" "GND" (at 294.64 163.83 0) (effects (font (size 2 2)) hide)) (property "Footprint" "" (at 294.64 157.48 0) (effects (font (size 1.27 1.27)) hide)) (property "Datasheet" "" (at 294.64 157.48 0) (effects (font (size 1.27 1.27)) hide)) (pin "1") (instances (project "placard" (path "/e3450542-4ffc-59d4-a4a7-45636233928a/370d9988-af17-5e05-8c50-5ef0ca792654" (reference "#PWR0310") (unit 1)))))
-  (symbol (lib_id "placard:ATF22V10C_BRANCH") (at 294.64 127 0) (unit 1) (in_bom yes) (on_board yes) (dnp no) (property "Reference" "U2" (at 275.082 100.1 0) (effects (font (size 2.54 2.54) bold) (justify left bottom))) (property "Value" "ATF22V10C-10PU" (at 275.082 158.94 0) (effects (font (size 2 2)) (justify left top))) (property "Function" "Branch PLD" (at 275.082 162.34 0) (effects (font (size 2.54 2.54) bold) (justify left top))) (property "Footprint" "Package_DIP:DIP-24_W7.62mm" (at 294.64 127 0) (effects (font (size 1.27 1.27)) hide)) (property "Datasheet" "https://ww1.microchip.com/downloads/en/DeviceDoc/doc0735.pdf" (at 294.64 127 0) (effects (font (size 1.27 1.27)) hide)) (property "Manufacturer" "Microchip" (at 294.64 127 0) (effects (font (size 1.27 1.27)) hide)) (property "MPN" "ATF22V10C-10PU" (at 294.64 127 0) (effects (font (size 1.27 1.27)) hide)) (property "PLD" "ATF22V10_BRANCH.pld" (at 294.64 127 0) (effects (font (size 1.27 1.27)) hide)) (pin "17") (pin "2") (pin "3") (pin "4") (pin "5") (pin "6") (pin "7") (pin "13") (pin "8") (pin "1") (pin "10") (pin "11") (pin "9") (pin "14") (pin "23") (pin "21") (pin "22") (pin "19") (pin "16") (pin "15") (pin "18") (pin "20") (pin "24") (pin "12") (instances (project "placard" (path "/e3450542-4ffc-59d4-a4a7-45636233928a/370d9988-af17-5e05-8c50-5ef0ca792654" (reference "U2") (unit 1)))))
+  (symbol (lib_id "placard:ATF22V10C_BRANCH") (at 294.64 127 0) (unit 1) (in_bom yes) (on_board yes) (dnp no) (property "Reference" "U2" (at 275.082 100.1 0) (effects (font (size 2.54 2.54) bold) (justify left bottom))) (property "Value" "ATF22V10C-7PX" (at 275.082 158.94 0) (effects (font (size 2 2)) (justify left top))) (property "Function" "Branch PLD" (at 275.082 162.34 0) (effects (font (size 2.54 2.54) bold) (justify left top))) (property "Footprint" "Package_DIP:DIP-24_W7.62mm" (at 294.64 127 0) (effects (font (size 1.27 1.27)) hide)) (property "Datasheet" "https://ww1.microchip.com/downloads/en/DeviceDoc/doc0735.pdf" (at 294.64 127 0) (effects (font (size 1.27 1.27)) hide)) (property "Manufacturer" "Microchip" (at 294.64 127 0) (effects (font (size 1.27 1.27)) hide)) (property "MPN" "ATF22V10C-7PX" (at 294.64 127 0) (effects (font (size 1.27 1.27)) hide)) (property "PLD" "ATF22V10_BRANCH.pld" (at 294.64 127 0) (effects (font (size 1.27 1.27)) hide)) (pin "17") (pin "2") (pin "3") (pin "4") (pin "5") (pin "6") (pin "7") (pin "13") (pin "8") (pin "1") (pin "10") (pin "11") (pin "9") (pin "14") (pin "23") (pin "21") (pin "22") (pin "19") (pin "16") (pin "15") (pin "18") (pin "20") (pin "24") (pin "12") (instances (project "placard" (path "/e3450542-4ffc-59d4-a4a7-45636233928a/370d9988-af17-5e05-8c50-5ef0ca792654" (reference "U2") (unit 1)))))
   (symbol (lib_id "power:+5V") (at 314.96 90.17 0) (unit 1) (in_bom yes) (on_board yes) (dnp no) (property "Reference" "#PWR0311" (at 314.96 90.17 0) (effects (font (size 1.27 1.27)) hide)) (property "Value" "+5V" (at 314.96 83.82 0) (effects (font (size 2 2)))) (property "Footprint" "" (at 314.96 90.17 0) (effects (font (size 1.27 1.27)) hide)) (property "Datasheet" "" (at 314.96 90.17 0) (effects (font (size 1.27 1.27)) hide)) (pin "1") (instances (project "placard" (path "/e3450542-4ffc-59d4-a4a7-45636233928a/370d9988-af17-5e05-8c50-5ef0ca792654" (reference "#PWR0311") (unit 1)))))
   (symbol (lib_id "power:GND") (at 314.96 97.79 0) (unit 1) (in_bom yes) (on_board yes) (dnp no) (property "Reference" "#PWR0312" (at 314.96 97.79 0) (effects (font (size 1.27 1.27)) hide)) (property "Value" "GND" (at 314.96 104.14 0) (effects (font (size 2 2)) hide)) (property "Footprint" "" (at 314.96 97.79 0) (effects (font (size 1.27 1.27)) hide)) (property "Datasheet" "" (at 314.96 97.79 0) (effects (font (size 1.27 1.27)) hide)) (pin "1") (instances (project "placard" (path "/e3450542-4ffc-59d4-a4a7-45636233928a/370d9988-af17-5e05-8c50-5ef0ca792654" (reference "#PWR0312") (unit 1)))))

Commit message: Kit footprints: DIP sockets with puller room and part number, resistors with value
Justin: put the chip-puller room in the socket footprints (User.Eco1,
2.5 mm past each end) and the part number in silkscreen between the pin
rows; resistors get their value in silkscreen on the body. New
gen_kicad_kit_footprints.py derives them from KiCad's stock footprints;
schematic, symbols, BOM and PDFs now name them. The board file is left
as is (Justin is editing it): Update PCB from Schematic swaps them in.

Co-Authored-By: Claude Opus 5.5 (1M context) <noreply@anthropic.com>
Claude-Session: https://claude.ai/code/session_01JnVuvUvdWezUUU6Sgmg16H
Parts:
- U1, U17, U2: footprint Package_DIP:DIP-24_W7.62mm -> placard:DIP-24_W7.62mm_Socket_Puller
