File: kicad/control.kicad_sch (KiCad schematic)
At the start: 6 parts, among them U1 ATF22V10C-7PX, U17 ATF22V10C-7PX, U2 ATF22V10C-7PX

Commit message: BOM/schematic: stocked substitutes from the first parts order
D18 Kingbright WP7113ID (LTL2R3KRD-EM out of stock), 100n TDK
FG28X7R1H104KNT00 (KEMET C320C104 $0.66 at Mouser), C45 TDK
FG24C0G1H153JNT06 (KEMET non-stocked), Vishay BAT85S-TAP and
1N4148-TAP, MF-RG300-0, USB4125-GF-A-0190; Mouser prices re-checked.

Co-Authored-By: Claude Opus 5.5 (1M context) <noreply@anthropic.com>
Claude-Session: https://claude.ai/code/session_017y5UgjExE8oeP7QrfvhCzb
Parts:
- C1, C17, C2: MPN C320C104K5R5TA -> FG28X7R1H104KNT00; Manufacturer KEMET -> TDK
Changed lines of the file:
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@@
   (symbol (lib_id "power:+5V") (at 91.44 118.11 0) (unit 1) (in_bom yes) (on_board yes) (dnp no) (property "Reference" "#PWR0303" (at 91.44 118.11 0) (effects (font (size 1.27 1.27)) hide)) (property "Value" "+5V" (at 91.44 111.76 0) (effects (font (size 2 2)))) (property "Footprint" "" (at 91.44 118.11 0) (effects (font (size 1.27 1.27)) hide)) (property "Datasheet" "" (at 91.44 118.11 0) (effects (font (size 1.27 1.27)) hide)) (pin "1") (instances (project "placard" (path "/e3450542-4ffc-59d4-a4a7-45636233928a/370d9988-af17-5e05-8c50-5ef0ca792654" (reference "#PWR0303") (unit 1)))))
   (symbol (lib_id "power:GND") (at 91.44 125.73 0) (unit 1) (in_bom yes) (on_board yes) (dnp no) (property "Reference" "#PWR0304" (at 91.44 125.73 0) (effects (font (size 1.27 1.27)) hide)) (property "Value" "GND" (at 91.44 132.08 0) (effects (font (size 2 2)) hide)) (property "Footprint" "" (at 91.44 125.73 0) (effects (font (size 1.27 1.27)) hide)) (property "Datasheet" "" (at 91.44 125.73 0) (effects (font (size 1.27 1.27)) hide)) (pin "1") (instances (project "placard" (path "/e3450542-4ffc-59d4-a4a7-45636233928a/370d9988-af17-5e05-8c50-5ef0ca792654" (reference "#PWR0304") (unit 1)))))
-  (symbol (lib_id "placard_std:C") (at 91.44 121.92 0) (unit 1) (in_bom yes) (on_board yes) (dnp no) (property "Reference" "C17" (at 93.44 121.42 0) (effects (font (size 2.54 2.54) bold) (justify left bottom))) (property "Value" "100n" (at 93.44 124.52 0) (effects (font (size 2 2)) (justify left top))) (property "Footprint" "Capacitor_THT:C_Disc_D5.0mm_W2.5mm_P5.00mm" (at 91.44 121.92 0) (effects (font (size 1.27 1.27)) hide)) (property "Datasheet" "~" (at 91.44 121.92 0) (effects (font (size 1.27 1.27)) hide)) (property "Manufacturer" "KEMET" (at 91.44 121.92 0) (effects (font (size 1.27 1.27)) hide)) (property "MPN" "C320C104K5R5TA" (at 91.44 121.92 0) (effects (font (size 1.27 1.27)) hide)) (pin "1") (pin "2") (instances (project "placard" (path "/e3450542-4ffc-59d4-a4a7-45636233928a/370d9988-af17-5e05-8c50-5ef0ca792654" (reference "C17") (unit 1)))))
+  (symbol (lib_id "placard_std:C") (at 91.44 121.92 0) (unit 1) (in_bom yes) (on_board yes) (dnp no) (property "Reference" "C17" (at 93.44 121.42 0) (effects (font (size 2.54 2.54) bold) (justify left bottom))) (property "Value" "100n" (at 93.44 124.52 0) (effects (font (size 2 2)) (justify left top))) (property "Footprint" "Capacitor_THT:C_Disc_D5.0mm_W2.5mm_P5.00mm" (at 91.44 121.92 0) (effects (font (size 1.27 1.27)) hide)) (property "Datasheet" "~" (at 91.44 121.92 0) (effects (font (size 1.27 1.27)) hide)) (property "Manufacturer" "TDK" (at 91.44 121.92 0) (effects (font (size 1.27 1.27)) hide)) (property "MPN" "FG28X7R1H104KNT00" (at 91.44 121.92 0) (effects (font (size 1.27 1.27)) hide)) (pin "1") (pin "2") (instances (project "placard" (path "/e3450542-4ffc-59d4-a4a7-45636233928a/370d9988-af17-5e05-8c50-5ef0ca792654" (reference "C17") (unit 1)))))
   (wire (pts (xy 172.72 134.62) (xy 172.72 132.08)) (stroke (width 0) (type default)))
   (symbol (lib_id "power:+5V") (at 172.72 132.08 0) (unit 1) (in_bom yes) (on_board yes) (dnp no) (property "Reference" "#PWR0305" (at 172.72 132.08 0) (effects (font (size 1.27 1.27)) hide)) (property "Value" "+5V" (at 172.72 125.73 0) (effects (font (size 2 2)))) (property "Footprint" "" (at 172.72 132.08 0) (effects (font (size 1.27 1.27)) hide)) (property "Datasheet" "" (at 172.72 132.08 0) (effects (font (size 1.27 1.27)) hide)) (pin "1") (instances (project "placard" (path "/e3450542-4ffc-59d4-a4a7-45636233928a/370d9988-af17-5e05-8c50-5ef0ca792654" (reference "#PWR0305") (unit 1)))))
@@
   (symbol (lib_id "power:+5V") (at 193.04 123.19 0) (unit 1) (in_bom yes) (on_board yes) (dnp no) (property "Reference" "#PWR0307" (at 193.04 123.19 0) (effects (font (size 1.27 1.27)) hide)) (property "Value" "+5V" (at 193.04 116.84 0) (effects (font (size 2 2)))) (property "Footprint" "" (at 193.04 123.19 0) (effects (font (size 1.27 1.27)) hide)) (property "Datasheet" "" (at 193.04 123.19 0) (effects (font (size 1.27 1.27)) hide)) (pin "1") (instances (project "placard" (path "/e3450542-4ffc-59d4-a4a7-45636233928a/370d9988-af17-5e05-8c50-5ef0ca792654" (reference "#PWR0307") (unit 1)))))
   (symbol (lib_id "power:GND") (at 193.04 130.81 0) (unit 1) (in_bom yes) (on_board yes) (dnp no) (property "Reference" "#PWR0308" (at 193.04 130.81 0) (effects (font (size 1.27 1.27)) hide)) (property "Value" "GND" (at 193.04 137.16 0) (effects (font (size 2 2)) hide)) (property "Footprint" "" (at 193.04 130.81 0) (effects (font (size 1.27 1.27)) hide)) (property "Datasheet" "" (at 193.04 130.81 0) (effects (font (size 1.27 1.27)) hide)) (pin "1") (instances (project "placard" (path "/e3450542-4ffc-59d4-a4a7-45636233928a/370d9988-af17-5e05-8c50-5ef0ca792654" (reference "#PWR0308") (unit 1)))))
-  (symbol (lib_id "placard_std:C") (at 193.04 127 0) (unit 1) (in_bom yes) (on_board yes) (dnp no) (property "Reference" "C1" (at 195.04 126.5 0) (effects (font (size 2.54 2.54) bold) (justify left bottom))) (property "Value" "100n" (at 195.04 129.6 0) (effects (font (size 2 2)) (justify left top))) (property "Footprint" "Capacitor_THT:C_Disc_D5.0mm_W2.5mm_P5.00mm" (at 193.04 127 0) (effects (font (size 1.27 1.27)) hide)) (property "Datasheet" "~" (at 193.04 127 0) (effects (font (size 1.27 1.27)) hide)) (property "Manufacturer" "KEMET" (at 193.04 127 0) (effects (font (size 1.27 1.27)) hide)) (property "MPN" "C320C104K5R5TA" (at 193.04 127 0) (effects (font (size 1.27 1.27)) hide)) (pin "1") (pin "2") (instances (project "placard" (path "/e3450542-4ffc-59d4-a4a7-45636233928a/370d9988-af17-5e05-8c50-5ef0ca792654" (reference "C1") (unit 1)))))
+  (symbol (lib_id "placard_std:C") (at 193.04 127 0) (unit 1) (in_bom yes) (on_board yes) (dnp no) (property "Reference" "C1" (at 195.04 126.5 0) (effects (font (size 2.54 2.54) bold) (justify left bottom))) (property "Value" "100n" (at 195.04 129.6 0) (effects (font (size 2 2)) (justify left top))) (property "Footprint" "Capacitor_THT:C_Disc_D5.0mm_W2.5mm_P5.00mm" (at 193.04 127 0) (effects (font (size 1.27 1.27)) hide)) (property "Datasheet" "~" (at 193.04 127 0) (effects (font (size 1.27 1.27)) hide)) (property "Manufacturer" "TDK" (at 193.04 127 0) (effects (font (size 1.27 1.27)) hide)) (property "MPN" "FG28X7R1H104KNT00" (at 193.04 127 0) (effects (font (size 1.27 1.27)) hide)) (pin "1") (pin "2") (instances (project "placard" (path "/e3450542-4ffc-59d4-a4a7-45636233928a/370d9988-af17-5e05-8c50-5ef0ca792654" (reference "C1") (unit 1)))))
   (no_connect (at 322.58 144.78))
   (no_connect (at 322.58 149.86))
@@
   (symbol (lib_id "power:+5V") (at 314.96 90.17 0) (unit 1) (in_bom yes) (on_board yes) (dnp no) (property "Reference" "#PWR0311" (at 314.96 90.17 0) (effects (font (size 1.27 1.27)) hide)) (property "Value" "+5V" (at 314.96 83.82 0) (effects (font (size 2 2)))) (property "Footprint" "" (at 314.96 90.17 0) (effects (font (size 1.27 1.27)) hide)) (property "Datasheet" "" (at 314.96 90.17 0) (effects (font (size 1.27 1.27)) hide)) (pin "1") (instances (project "placard" (path "/e3450542-4ffc-59d4-a4a7-45636233928a/370d9988-af17-5e05-8c50-5ef0ca792654" (reference "#PWR0311") (unit 1)))))
   (symbol (lib_id "power:GND") (at 314.96 97.79 0) (unit 1) (in_bom yes) (on_board yes) (dnp no) (property "Reference" "#PWR0312" (at 314.96 97.79 0) (effects (font (size 1.27 1.27)) hide)) (property "Value" "GND" (at 314.96 104.14 0) (effects (font (size 2 2)) hide)) (property "Footprint" "" (at 314.96 97.79 0) (effects (font (size 1.27 1.27)) hide)) (property "Datasheet" "" (at 314.96 97.79 0) (effects (font (size 1.27 1.27)) hide)) (pin "1") (instances (project "placard" (path "/e3450542-4ffc-59d4-a4a7-45636233928a/370d9988-af17-5e05-8c50-5ef0ca792654" (reference "#PWR0312") (unit 1)))))
-  (symbol (lib_id "placard_std:C") (at 314.96 93.98 0) (unit 1) (in_bom yes) (on_board yes) (dnp no) (property "Reference" "C2" (at 316.96 93.48 0) (effects (font (size 2.54 2.54) bold) (justify left bottom))) (property "Value" "100n" (at 316.96 96.58 0) (effects (font (size 2 2)) (justify left top))) (property "Footprint" "Capacitor_THT:C_Disc_D5.0mm_W2.5mm_P5.00mm" (at 314.96 93.98 0) (effects (font (size 1.27 1.27)) hide)) (property "Datasheet" "~" (at 314.96 93.98 0) (effects (font (size 1.27 1.27)) hide)) (property "Manufacturer" "KEMET" (at 314.96 93.98 0) (effects (font (size 1.27 1.27)) hide)) (property "MPN" "C320C104K5R5TA" (at 314.96 93.98 0) (effects (font (size 1.27 1.27)) hide)) (pin "1") (pin "2") (instances (project "placard" (path "/e3450542-4ffc-59d4-a4a7-45636233928a/370d9988-af17-5e05-8c50-5ef0ca792654" (reference "C2") (unit 1)))))
+  (symbol (lib_id "placard_std:C") (at 314.96 93.98 0) (unit 1) (in_bom yes) (on_board yes) (dnp no) (property "Reference" "C2" (at 316.96 93.48 0) (effects (font (size 2.54 2.54) bold) (justify left bottom))) (property "Value" "100n" (at 316.96 96.58 0) (effects (font (size 2 2)) (justify left top))) (property "Footprint" "Capacitor_THT:C_Disc_D5.0mm_W2.5mm_P5.00mm" (at 314.96 93.98 0) (effects (font (size 1.27 1.27)) hide)) (property "Datasheet" "~" (at 314.96 93.98 0) (effects (font (size 1.27 1.27)) hide)) (property "Manufacturer" "TDK" (at 314.96 93.98 0) (effects (font (size 1.27 1.27)) hide)) (property "MPN" "FG28X7R1H104KNT00" (at 314.96 93.98 0) (effects (font (size 1.27 1.27)) hide)) (pin "1") (pin "2") (instances (project "placard" (path "/e3450542-4ffc-59d4-a4a7-45636233928a/370d9988-af17-5e05-8c50-5ef0ca792654" (reference "C2") (unit 1)))))
   (wire (pts (xy 198.12 139.7) (xy 266.7 139.7)) (stroke (width 0) (type default)))
   (wire (pts (xy 198.12 142.24) (xy 208.28 142.24)) (stroke (width 0) (type default)))

Commit message: Put every symbol, footprint and 3D model in the project library
- gen_kicad_stock_footprints.py: copies of the KiCad 9.0.6 footprints the
  boards use (C_Disc, CP_Radial, DO-15/DO-35, LED, pin header, oscillator,
  TO-92, SIP9, mounting holes, net tie) into placard.pretty, and KiCad's
  STEP models for them and for the DIP socket / resistor kit footprints
  into placard.3dshapes
- model paths use the PLACARD_LIB text variable (main board
  ${KIPRJMOD}/lib, cartridges ${KIPRJMOD}/../lib) so the shared footprints
  find their models in all three projects
- placard_std gains the 28C256 EEPROM and the power symbols; symbol
  Footprint defaults name placard footprints (relay, SIP9, oscillator,
  TO-92, EEPROM socket)
- schematics regenerated with placard_std power/EEPROM symbols and
  placard: footprints; BOM CSVs and PDFs regenerated
- cartridge .kicad_pro files take in Justin's local KiCad 9 settings

Co-Authored-By: Claude Opus 5.5 <noreply@anthropic.com>
Claude-Session: https://claude.ai/code/session_017okF1JiLRNFTfH7Az85hff
Parts:
- C1, C17, C2: footprint Capacitor_THT:C_Disc_D5.0mm_W2.5mm_P5.00mm -> placard:C_Disc_D5.0mm_W2.5mm_P5.00mm

Commit message: Schematic: rename buses to ADDR / DATABUS / D, wire the shared port outputs
- Address bus A15:A0 is now ADDR15:ADDR0, the data bus D7:D0 is DATABUS7:DATABUS0
  and the D register's outputs DR7:DR0 are D7:D0 (main board and both cartridges).
- Shared port sheet: U38's outputs P_SCK, P_MOSI, P_CS, P_PS2D and K0 are wired
  to the SNES pads, the SD dividers and the PS/2 hold diodes (K0 -> D6 ->
  keyboard CLK).  J3 now sits level with U38's SCK/MOSI pins, J2 above it.
- Parts moved so the longer labels fit: U3/U4 and the PC bus, U18, U22, U11,
  U31, U32, RN1, R5-R12; expansion slots in two rows.
- SCHEMATIC_PLAN.md: the bus names.

Co-Authored-By: Claude Opus 5.5 <noreply@anthropic.com>
Claude-Session: https://claude.ai/code/session_01DnW5SUv7E4nz9tGtPvD1qV
Connections:
- net D0 renamed DATABUS0
- net D1 renamed DATABUS1
- net D2 renamed DATABUS2
- net D3 renamed DATABUS3
- net D4 renamed DATABUS4
- net D5 renamed DATABUS5
- net D6 renamed DATABUS6
- net D7 renamed DATABUS7
