File: kicad/video_out.kicad_sch (KiCad schematic)
At the start: 55 parts, among them J6 3.5 mm, J7 VGA, U16 ATF22V10C-10PU, U22 SN74F377AN, U23 74HCT377, U36 SN74HCT574N

Commit message: Row tint and blank line: BOM, FPGA model, simulator, docs
- BOM: U23 CD74HCT377E, BAT85 D27-D29, 1N4148 D30-D35, 910 ohm R56-R58
- FPGA: hcount_pld revision 08 (LC7, BLANK_PULSE), vga_gen_pld lc7In,
  basys_top adds the row tint (+4 of 15) on the VGA outputs
- src/sim/tb_blank_line.vhd: GHDL check of blanked and shown lines
- placard_sim render(): bit 7 blanks a row, bits 6:4 tint it
- LIBRARY.md, memory map, CHIPS/KITTING/COLORS/SOUND/VIDEO part names

Co-Authored-By: Claude Opus 5.5 (1M context) <noreply@anthropic.com>
Claude-Session: https://claude.ai/code/session_01AyS52y3xy4qvxwvt915gG3
Parts:
- D30, D31, D32, D33, D34, D35: MPN (none) -> 1N4148; Manufacturer (none) -> Vishay
- R56, R57, R58: MPN (none) -> MFR-25FBF52-910R; Manufacturer (none) -> Yageo
- U23: value 74HCT377 -> CD74HCT377E; MPN (none) -> CD74HCT377E; Manufacturer (none) -> Texas Instruments

Commit message: Every PLD is an ATF22V10C-7PX (one part number)
Justin: switch the seven main-board -10PU PLDs (Branch, PC x2, H, V,
color decoder, audio slot) and the cartridge loader to the -7PX, for one
part number to buy, program and kit (.52 more per main board). Symbols,
schematics, PDFs, BOM, docs and PLD comments updated; CHIPS.md keeps the
grade each PLD could use.

Co-Authored-By: Claude Opus 5.5 (1M context) <noreply@anthropic.com>
Claude-Session: https://claude.ai/code/session_01JnVuvUvdWezUUU6Sgmg16H
Parts:
- U16: value ATF22V10C-10PU -> ATF22V10C-7PX; MPN ATF22V10C-10PU -> ATF22V10C-7PX
Changed lines of the file:
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@@
   (wire (pts (xy 190.5 134.62) (xy 190.5 137.16)) (stroke (width 0) (type default)))
   (symbol (lib_id "power:GND") (at 190.5 137.16 0) (unit 1) (in_bom yes) (on_board yes) (dnp no) (property "Reference" "#PWR0906" (at 190.5 137.16 0) (effects (font (size 1.27 1.27)) hide)) (property "Value" "GND" (at 190.5 143.51 0) (effects (font (size 2 2)) hide)) (property "Footprint" "" (at 190.5 137.16 0) (effects (font (size 1.27 1.27)) hide)) (property "Datasheet" "" (at 190.5 137.16 0) (effects (font (size 1.27 1.27)) hide)) (pin "1") (instances (project "placard" (path "/e3450542-4ffc-59d4-a4a7-45636233928a/53445658-004f-5a3f-8e51-bf0246e5367e" (reference "#PWR0906") (unit 1)))))
-  (symbol (lib_id "placard:ATF22V10C_COLORDECODER") (at 190.5 109.22 0) (unit 1) (in_bom yes) (on_board yes) (dnp no) (property "Reference" "U16" (at 179.832 82.32 0) (effects (font (size 2.54 2.54) bold) (justify left bottom))) (property "Value" "ATF22V10C-10PU" (at 179.832 138.62 0) (effects (font (size 2 2)) (justify left top))) (property "Function" "Color decoder PLD" (at 179.832 142.02 0) (effects (font (size 2.54 2.54) bold) (justify left top))) (property "Footprint" "Package_DIP:DIP-24_W7.62mm" (at 190.5 109.22 0) (effects (font (size 1.27 1.27)) hide)) (property "Datasheet" "https://ww1.microchip.com/downloads/en/DeviceDoc/doc0735.pdf" (at 190.5 109.22 0) (effects (font (size 1.27 1.27)) hide)) (property "Manufacturer" "Microchip" (at 190.5 109.22 0) (effects (font (size 1.27 1.27)) hide)) (property "MPN" "ATF22V10C-10PU" (at 190.5 109.22 0) (effects (font (size 1.27 1.27)) hide)) (property "PLD" "ATF22V10_COLORDECODER.pld" (at 190.5 109.22 0) (effects (font (size 1.27 1.27)) hide)) (pin "2") (pin "3") (pin "4") (pin "5") (pin "6") (pin "7") (pin "8") (pin "9") (pin "10") (pin "11") (pin "13") (pin "1") (pin "14") (pin "23") (pin "15") (pin "16") (pin "21") (pin "17") (pin "20") (pin "19") (pin "22") (pin "18") (pin "24") (pin "12") (instances (project "placard" (path "/e3450542-4ffc-59d4-a4a7-45636233928a/53445658-004f-5a3f-8e51-bf0246e5367e" (reference "U16") (unit 1)))))
+  (symbol (lib_id "placard:ATF22V10C_COLORDECODER") (at 190.5 109.22 0) (unit 1) (in_bom yes) (on_board yes) (dnp no) (property "Reference" "U16" (at 179.832 82.32 0) (effects (font (size 2.54 2.54) bold) (justify left bottom))) (property "Value" "ATF22V10C-7PX" (at 179.832 138.62 0) (effects (font (size 2 2)) (justify left top))) (property "Function" "Color decoder PLD" (at 179.832 142.02 0) (effects (font (size 2.54 2.54) bold) (justify left top))) (property "Footprint" "Package_DIP:DIP-24_W7.62mm" (at 190.5 109.22 0) (effects (font (size 1.27 1.27)) hide)) (property "Datasheet" "https://ww1.microchip.com/downloads/en/DeviceDoc/doc0735.pdf" (at 190.5 109.22 0) (effects (font (size 1.27 1.27)) hide)) (property "Manufacturer" "Microchip" (at 190.5 109.22 0) (effects (font (size 1.27 1.27)) hide)) (property "MPN" "ATF22V10C-7PX" (at 190.5 109.22 0) (effects (font (size 1.27 1.27)) hide)) (property "PLD" "ATF22V10_COLORDECODER.pld" (at 190.5 109.22 0) (effects (font (size 1.27 1.27)) hide)) (pin "2") (pin "3") (pin "4") (pin "5") (pin "6") (pin "7") (pin "8") (pin "9") (pin "10") (pin "11") (pin "13") (pin "1") (pin "14") (pin "23") (pin "15") (pin "16") (pin "21") (pin "17") (pin "20") (pin "19") (pin "22") (pin "18") (pin "24") (pin "12") (instances (project "placard" (path "/e3450542-4ffc-59d4-a4a7-45636233928a/53445658-004f-5a3f-8e51-bf0246e5367e" (reference "U16") (unit 1)))))
   (symbol (lib_id "power:+5V") (at 213.36 72.39 0) (unit 1) (in_bom yes) (on_board yes) (dnp no) (property "Reference" "#PWR0907" (at 213.36 72.39 0) (effects (font (size 1.27 1.27)) hide)) (property "Value" "+5V" (at 213.36 66.04 0) (effects (font (size 2 2)))) (property "Footprint" "" (at 213.36 72.39 0) (effects (font (size 1.27 1.27)) hide)) (property "Datasheet" "" (at 213.36 72.39 0) (effects (font (size 1.27 1.27)) hide)) (pin "1") (instances (project "placard" (path "/e3450542-4ffc-59d4-a4a7-45636233928a/53445658-004f-5a3f-8e51-bf0246e5367e" (reference "#PWR0907") (unit 1)))))
   (symbol (lib_id "power:GND") (at 213.36 80.01 0) (unit 1) (in_bom yes) (on_board yes) (dnp no) (property "Reference" "#PWR0908" (at 213.36 80.01 0) (effects (font (size 1.27 1.27)) hide)) (property "Value" "GND" (at 213.36 86.36 0) (effects (font (size 2 2)) hide)) (property "Footprint" "" (at 213.36 80.01 0) (effects (font (size 1.27 1.27)) hide)) (property "Datasheet" "" (at 213.36 80.01 0) (effects (font (size 1.27 1.27)) hide)) (pin "1") (instances (project "placard" (path "/e3450542-4ffc-59d4-a4a7-45636233928a/53445658-004f-5a3f-8e51-bf0246e5367e" (reference "#PWR0908") (unit 1)))))

Commit message: Relabel the audio output as line out in the schematic and diagrams
Sheet 9 heading, audio schematic PNG, block diagram, symbol render and
script comments now say audio line out.  PDFs regenerated (no outline).

Co-Authored-By: Claude Opus 5.5 (1M context) <noreply@anthropic.com>
Claude-Session: https://claude.ai/code/session_016v2oaxTs8Tr6RsYPNLtphh
Other:
- note added: "Pixel buffer, line code, color decoder and VGA DAC; audio DAC register, R-2R ladder, audio line out"
- note removed: "Pixel buffer, line code, color decoder and VGA DAC; audio DAC register, R-2R ladder, headphones"
Changed lines of the file:
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@@
 (kicad_sch (version 20230121) (generator eeschema)
   (paper "A3")
-  (title_block (title "Placard: Video and audio out") (date "2026-10-22") (rev "1") (company "Placard computer") (comment 1 "Generated by src/scripts/gen_kicad_schematic.py; plan in docs/SCHEMATIC_PLAN.md") (comment 2 "Chip numbers U1-U40 = docs/CHIPS.md; decoupling Cn goes with Un"))
+  (title_block (title "Placard: Video and audio out") (date "2026-10-23") (rev "1") (company "Placard computer") (comment 1 "Generated by src/scripts/gen_kicad_schematic.py; plan in docs/SCHEMATIC_PLAN.md") (comment 2 "Chip numbers U1-U40 = docs/CHIPS.md; decoupling Cn goes with Un"))
   (text "Video and audio out" (at 15 22 0) (effects (font (size 6 6) bold) (justify left bottom)))
-  (text "Pixel buffer, line code, color decoder and VGA DAC; audio DAC register, R-2R ladder, headphones" (at 15 30 0) (effects (font (size 3 3)) (justify left bottom)))
+  (text "Pixel buffer, line code, color decoder and VGA DAC; audio DAC register, R-2R ladder, audio line out" (at 15 30 0) (effects (font (size 3 3)) (justify left bottom)))
   (wire (pts (xy 63.5 121.92) (xy 63.5 124.46)) (stroke (width 0) (type default)))
   (symbol (lib_id "power:GND") (at 63.5 124.46 0) (unit 1) (in_bom yes) (on_board yes) (dnp no) (property "Reference" "#PWR0901" (at 63.5 124.46 0) (effects (font (size 1.27 1.27)) hide)) (property "Value" "GND" (at 63.5 130.81 0) (effects (font (size 2 2)) hide)) (property "Footprint" "" (at 63.5 124.46 0) (effects (font (size 1.27 1.27)) hide)) (property "Datasheet" "" (at 63.5 124.46 0) (effects (font (size 1.27 1.27)) hide)) (pin "1") (instances (project "placard" (path "/e3450542-4ffc-59d4-a4a7-45636233928a/53445658-004f-5a3f-8e51-bf0246e5367e" (reference "#PWR0901") (unit 1)))))

Commit message: Kit footprints: DIP sockets with puller room and part number, resistors with value
Justin: put the chip-puller room in the socket footprints (User.Eco1,
2.5 mm past each end) and the part number in silkscreen between the pin
rows; resistors get their value in silkscreen on the body. New
gen_kicad_kit_footprints.py derives them from KiCad's stock footprints;
schematic, symbols, BOM and PDFs now name them. The board file is left
as is (Justin is editing it): Update PCB from Schematic swaps them in.

Co-Authored-By: Claude Opus 5.5 (1M context) <noreply@anthropic.com>
Claude-Session: https://claude.ai/code/session_01JnVuvUvdWezUUU6Sgmg16H
Parts:
- R14, R15, R16, R17, R18, R19, R20, R21, R22, R23, R24, R25, R26, R27, R28, R29, R30, R31, R32, R33, R34, R35, R36, R37, R38, R39, R56, R57, R58: footprint Resistor_THT:R_Axial_DIN0207_L6.3mm_D2.5mm_P10.16mm_Horizontal -> placard:R_Axial_DIN0207_L6.3mm_D2.5mm_P10.16mm_Horizontal_Value
- U16: footprint Package_DIP:DIP-24_W7.62mm -> placard:DIP-24_W7.62mm_Socket_Puller
- U22, U23, U36: footprint Package_DIP:DIP-20_W7.62mm -> placard:DIP-20_W7.62mm_Socket_Puller

Commit message: Name the vertical sync /VSYNC like /HSYNC
Sync PLD rev 09 declares pin 18 active low (PIN 18 = !VSYNC) with the
equation written as logical true, the same way the H counter declares
!HSYNC.  The pin output is unchanged (low during counts 532-533) and the
equation drops from 6 product terms to 1.  Schematic net, symbol pin,
VHDL comments, bring-up labels and docs follow; main schematic PDF
regenerated.

Co-Authored-By: Claude Opus 5.5 (1M context) <noreply@anthropic.com>
Claude-Session: https://claude.ai/code/session_013veaZZUxC2KxHUx8e17FHP
Connections:
- net VSYNC renamed ~{VSYNC}
Changed lines of the file:
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@@
   (symbol (lib_id "placard_std:D_Schottky") (at 342.9 171.45 270) (unit 1) (in_bom yes) (on_board yes) (dnp no) (property "Reference" "D25" (at 332.9 173.94 90) (effects (font (size 2.54 2.54) bold) (justify left bottom))) (property "Value" "BAT85" (at 332.9 175.64 90) (effects (font (size 2 2)) (justify left top) hide)) (property "Footprint" "Diode_THT:D_DO-35_SOD27_P7.62mm_Horizontal" (at 342.9 171.45 0) (effects (font (size 1.27 1.27)) hide)) (property "Datasheet" "~" (at 342.9 171.45 0) (effects (font (size 1.27 1.27)) hide)) (property "Manufacturer" "Vishay" (at 342.9 171.45 0) (effects (font (size 1.27 1.27)) hide)) (property "MPN" "BAT85" (at 342.9 171.45 0) (effects (font (size 1.27 1.27)) hide)) (pin "1") (pin "2") (instances (project "placard" (path "/e3450542-4ffc-59d4-a4a7-45636233928a/53445658-004f-5a3f-8e51-bf0246e5367e" (reference "D25") (unit 1)))))
   (wire (pts (xy 342.9 167.64) (xy 345.44 167.64)) (stroke (width 0) (type default)))
-  (global_label "VSYNC" (shape passive) (at 345.44 167.64 0) (fields_autoplaced) (effects (font (size 2 2)) (justify left)) (property "Intersheetrefs" "${INTERSHEET_REFS}" (at 345.44 167.64 0) (effects (font (size 2 2)) (justify left) hide)))
+  (global_label "~{VSYNC}" (shape passive) (at 345.44 167.64 0) (fields_autoplaced) (effects (font (size 2 2)) (justify left)) (property "Intersheetrefs" "${INTERSHEET_REFS}" (at 345.44 167.64 0) (effects (font (size 2 2)) (justify left) hide)))
   (text "ESD clamps D22-D25 (BAT85): the syncs at J7 go to +5V" (at 297.18 185.42 0) (effects (font (size 2.2 2.2)) (justify left bottom)))
   (text "and GND through a Schottky." (at 297.18 188.94 0) (effects (font (size 2.2 2.2)) (justify left bottom)))
@@
   (global_label "~{HSYNC}" (shape passive) (at 328.93 101.6 0) (fields_autoplaced) (effects (font (size 2 2)) (justify left)) (property "Intersheetrefs" "${INTERSHEET_REFS}" (at 328.93 101.6 0) (effects (font (size 2 2)) (justify left) hide)))
   (wire (pts (xy 323.85 106.68) (xy 328.93 106.68)) (stroke (width 0) (type default)))
-  (global_label "VSYNC" (shape passive) (at 328.93 106.68 0) (fields_autoplaced) (effects (font (size 2 2)) (justify left)) (property "Intersheetrefs" "${INTERSHEET_REFS}" (at 328.93 106.68 0) (effects (font (size 2 2)) (justify left) hide)))
+  (global_label "~{VSYNC}" (shape passive) (at 328.93 106.68 0) (fields_autoplaced) (effects (font (size 2 2)) (justify left)) (property "Intersheetrefs" "${INTERSHEET_REFS}" (at 328.93 106.68 0) (effects (font (size 2 2)) (justify left) hide)))
   (wire (pts (xy 127 205.74) (xy 115.57 205.74)) (stroke (width 0) (type default)))
   (label "PIX0" (at 127 205.74 180) (fields_autoplaced) (effects (font (size 2 2)) (justify right bottom)))

Commit message: Remove the ESD clamps from PS/2, SNES and VGA
Justin decided to take the BAT85 steering pairs out entirely: D8-D21
(shared port sheet) and D22-D25 (video sheet sync lines), 18 diodes.
D7 (TVS on VBUS) stays.

The remaining diodes are renumbered so every kind is numbered from 1 with
no gaps: D26 -> D8 (relay coil), D27-D29 -> D9-D11 (tint BAT85),
D30-D35 -> D12-D17 (tint 1N4148).

The schematic generator now keeps each symbol's uuid from the files
already on disk (and RENUMBERED carries a renamed part's old uuid for one
run), so Update PCB from Schematic renames the renumbered footprints and
leaves every other footprint linked.  kicad/placard.kicad_pcb is not
touched.  BOM, PDFs (no bookmarks panel), placement lists and docs updated.

Co-Authored-By: Claude Opus 5.5 (1M context) <noreply@anthropic.com>
Claude-Session: https://claude.ai/code/session_01DRvpu48w1PN7avX3eFSFuQ
Parts:
- removed D22, D23, D24, D25: BAT85, Diode_THT:D_DO-35_SOD27_P7.62mm_Horizontal, symbol placard_std:D_Schottky
- renumbered D28 to D10, D29 to D11, D30 to D12, D31 to D13, D32 to D14, D33 to D15, D34 to D16, D35 to D17, D27 to D9
Other:
- note removed: "ESD clamps D22-D25 (BAT85): the syncs at J7 go to +5V"
- note removed: "and GND through a Schottky."

Commit message: Add 3D models for the connectors, switches and polyfuse
Every connector/switch footprint in kicad/lib/placard.pretty now names a
STEP model in kicad/lib/placard.3dshapes via ${KIPRJMOD}, so the board shows
them in any KiCad version without a 3D library path.

- gen_kicad_3d_models.py (CadQuery) generates models at typical dimensions
  for J8 cart slot, J9-J12 expansion slots, J5 stacked PS/2, J6 audio jack,
  SW1 toggle, J4 SD socket, F1 polyfuse and J2/J3 SNES ports; leads are put
  on the footprint pads. KiCad's own models are copied for SW2, J7, J13.
- gen_kicad_connectors.py adds the model to its footprints and makes
  project copies of KiCad's SD, MF-RG300, PTS645 and DSUB-15-HD footprints
  (same pads) pointing at the project models; removes a duplicated block.
- Schematic, BOM and gen_kicad_pcb.py use the placard: copies for J4, J7,
  F1, SW2. kicad/placard.kicad_pcb is not touched.
- docs/connector_3d_models.png: KiCad STEP export of the footprints.

Co-Authored-By: Claude Opus 5.5 (1M context) <noreply@anthropic.com>
Claude-Session: https://claude.ai/code/session_011CYV6fCf1RGSdDoH9HuCKo
Parts:
- J7: footprint Connector_Dsub:DSUB-15-HD_Female_Horizontal_P2.29x1.98mm_EdgePinOffset3.03mm_Housed_MountingHolesOffset4.94mm -> placard:DSUB-15-HD_Female_Horizontal_P2.29x1.98mm_EdgePinOffset3.03mm_Housed_MountingHolesOffset4.94mm
Changed lines of the file:
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@@
   (wire (pts (xy 306.07 109.22) (xy 306.07 111.76)) (stroke (width 0) (type default)))
   (symbol (lib_id "power:GND") (at 306.07 111.76 270) (unit 1) (in_bom yes) (on_board yes) (dnp no) (property "Reference" "#PWR0917" (at 306.07 111.76 0) (effects (font (size 1.27 1.27)) hide)) (property "Value" "GND" (at 297.72 111.76 90) (effects (font (size 2 2)) hide)) (property "Footprint" "" (at 306.07 111.76 0) (effects (font (size 1.27 1.27)) hide)) (property "Datasheet" "" (at 306.07 111.76 0) (effects (font (size 1.27 1.27)) hide)) (pin "1") (instances (project "placard" (path "/e3450542-4ffc-59d4-a4a7-45636233928a/53445658-004f-5a3f-8e51-bf0246e5367e" (reference "#PWR0917") (unit 1)))))
-  (symbol (lib_id "placard_std:DE15_Receptacle_HighDensity_MountingHoles") (at 316.23 101.6 0) (unit 1) (in_bom yes) (on_board yes) (dnp no) (property "Reference" "J7" (at 311 84 0) (effects (font (size 2.54 2.54) bold) (justify left bottom))) (property "Value" "VGA" (at 311 126 0) (effects (font (size 2 2)) (justify left top))) (property "Footprint" "Connector_Dsub:DSUB-15-HD_Female_Horizontal_P2.29x1.98mm_EdgePinOffset3.03mm_Housed_MountingHolesOffset4.94mm" (at 316.23 101.6 0) (effects (font (size 1.27 1.27)) hide)) (property "Datasheet" " ~" (at 316.23 101.6 0) (effects (font (size 1.27 1.27)) hide)) (property "Manufacturer" "Assmann WSW" (at 316.23 101.6 0) (effects (font (size 1.27 1.27)) hide)) (property "MPN" "A-HDF 15 A-KG/T" (at 316.23 101.6 0) (effects (font (size 1.27 1.27)) hide)) (pin "0") (pin "1") (pin "10") (pin "11") (pin "12") (pin "13") (pin "14") (pin "15") (pin "2") (pin "3") (pin "4") (pin "5") (pin "6") (pin "7") (pin "8") (pin "9") (instances (project "placard" (path "/e3450542-4ffc-59d4-a4a7-45636233928a/53445658-004f-5a3f-8e51-bf0246e5367e" (reference "J7") (unit 1)))))
+  (symbol (lib_id "placard_std:DE15_Receptacle_HighDensity_MountingHoles") (at 316.23 101.6 0) (unit 1) (in_bom yes) (on_board yes) (dnp no) (property "Reference" "J7" (at 311 84 0) (effects (font (size 2.54 2.54) bold) (justify left bottom))) (property "Value" "VGA" (at 311 126 0) (effects (font (size 2 2)) (justify left top))) (property "Footprint" "placard:DSUB-15-HD_Female_Horizontal_P2.29x1.98mm_EdgePinOffset3.03mm_Housed_MountingHolesOffset4.94mm" (at 316.23 101.6 0) (effects (font (size 1.27 1.27)) hide)) (property "Datasheet" " ~" (at 316.23 101.6 0) (effects (font (size 1.27 1.27)) hide)) (property "Manufacturer" "Assmann WSW" (at 316.23 101.6 0) (effects (font (size 1.27 1.27)) hide)) (property "MPN" "A-HDF 15 A-KG/T" (at 316.23 101.6 0) (effects (font (size 1.27 1.27)) hide)) (pin "0") (pin "1") (pin "10") (pin "11") (pin "12") (pin "13") (pin "14") (pin "15") (pin "2") (pin "3") (pin "4") (pin "5") (pin "6") (pin "7") (pin "8") (pin "9") (instances (project "placard" (path "/e3450542-4ffc-59d4-a4a7-45636233928a/53445658-004f-5a3f-8e51-bf0246e5367e" (reference "J7") (unit 1)))))
   (wire (pts (xy 248.92 88.9) (xy 264.16 88.9)) (stroke (width 0) (type default)))
   (wire (pts (xy 248.92 93.98) (xy 264.16 93.98)) (stroke (width 0) (type default)))
