File: kicad/video_out.kicad_sch (KiCad schematic)
At the start: 51 parts, among them J6 3.5 mm, J7 VGA, U16 ATF22V10C-7PX, U22 SN74F377AN, U23 CD74HCT377E, U36 SN74HCT574N

Commit message: VGA syncs: 47 ohm series resistors R61/R62 at the PLD pins
/HSYNC (U13 pin 21) and /VSYNC (U15 pin 18) now reach J7 through R61 and
R62 (47 ohm, Yageo MFR-25FBF52-47R, sharing R5-R12's BOM line); nets after
them are /VGA_HSYNC and /VGA_VSYNC.  Symbol uuids kept; board file untouched
(pull in with Update PCB from Schematic).  R60 22k gets its MPN.

Co-Authored-By: Claude Opus 5.5 (1M context) <noreply@anthropic.com>
Claude-Session: https://claude.ai/code/session_01B4M15KLwAcnVuRUejEFj2o
Connections:
- net ~{HSYNC} renamed ~{VGA_HSYNC}
- net ~{VSYNC} renamed ~{VGA_VSYNC}
Changed lines of the file:
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@@
   (global_label "LC7" (shape output) (at 149.86 157.48 0) (fields_autoplaced) (effects (font (size 2 2)) (justify left)) (property "Intersheetrefs" "${INTERSHEET_REFS}" (at 149.86 157.48 0) (effects (font (size 2 2)) (justify left) hide)))
   (wire (pts (xy 323.85 101.6) (xy 328.93 101.6)) (stroke (width 0) (type default)))
-  (global_label "~{HSYNC}" (shape passive) (at 328.93 101.6 0) (fields_autoplaced) (effects (font (size 2 2)) (justify left)) (property "Intersheetrefs" "${INTERSHEET_REFS}" (at 328.93 101.6 0) (effects (font (size 2 2)) (justify left) hide)))
+  (global_label "~{VGA_HSYNC}" (shape passive) (at 328.93 101.6 0) (fields_autoplaced) (effects (font (size 2 2)) (justify left)) (property "Intersheetrefs" "${INTERSHEET_REFS}" (at 328.93 101.6 0) (effects (font (size 2 2)) (justify left) hide)))
   (wire (pts (xy 323.85 106.68) (xy 328.93 106.68)) (stroke (width 0) (type default)))
-  (global_label "~{VSYNC}" (shape passive) (at 328.93 106.68 0) (fields_autoplaced) (effects (font (size 2 2)) (justify left)) (property "Intersheetrefs" "${INTERSHEET_REFS}" (at 328.93 106.68 0) (effects (font (size 2 2)) (justify left) hide)))
+  (global_label "~{VGA_VSYNC}" (shape passive) (at 328.93 106.68 0) (fields_autoplaced) (effects (font (size 2 2)) (justify left)) (property "Intersheetrefs" "${INTERSHEET_REFS}" (at 328.93 106.68 0) (effects (font (size 2 2)) (justify left) hide)))
   (wire (pts (xy 127 205.74) (xy 115.57 205.74)) (stroke (width 0) (type default)))
   (label "PIX0" (at 127 205.74 180) (fields_autoplaced) (effects (font (size 2 2)) (justify right bottom)))

Commit message: BOM/schematic: stocked substitutes from the first parts order
D18 Kingbright WP7113ID (LTL2R3KRD-EM out of stock), 100n TDK
FG28X7R1H104KNT00 (KEMET C320C104 $0.66 at Mouser), C45 TDK
FG24C0G1H153JNT06 (KEMET non-stocked), Vishay BAT85S-TAP and
1N4148-TAP, MF-RG300-0, USB4125-GF-A-0190; Mouser prices re-checked.

Co-Authored-By: Claude Opus 5.5 (1M context) <noreply@anthropic.com>
Claude-Session: https://claude.ai/code/session_017y5UgjExE8oeP7QrfvhCzb
Parts:
- C16, C22, C23, C36: MPN C320C104K5R5TA -> FG28X7R1H104KNT00; Manufacturer KEMET -> TDK
- C45: MPN C320C153K1G5TA -> FG24C0G1H153JNT06; Manufacturer KEMET -> TDK
- D10, D11, D9: MPN BAT85 -> BAT85S-TAP
- D12, D13, D14, D15, D16, D17: MPN 1N4148 -> 1N4148-TAP

Commit message: Put every symbol, footprint and 3D model in the project library
- gen_kicad_stock_footprints.py: copies of the KiCad 9.0.6 footprints the
  boards use (C_Disc, CP_Radial, DO-15/DO-35, LED, pin header, oscillator,
  TO-92, SIP9, mounting holes, net tie) into placard.pretty, and KiCad's
  STEP models for them and for the DIP socket / resistor kit footprints
  into placard.3dshapes
- model paths use the PLACARD_LIB text variable (main board
  ${KIPRJMOD}/lib, cartridges ${KIPRJMOD}/../lib) so the shared footprints
  find their models in all three projects
- placard_std gains the 28C256 EEPROM and the power symbols; symbol
  Footprint defaults name placard footprints (relay, SIP9, oscillator,
  TO-92, EEPROM socket)
- schematics regenerated with placard_std power/EEPROM symbols and
  placard: footprints; BOM CSVs and PDFs regenerated
- cartridge .kicad_pro files take in Justin's local KiCad 9 settings

Co-Authored-By: Claude Opus 5.5 <noreply@anthropic.com>
Claude-Session: https://claude.ai/code/session_017okF1JiLRNFTfH7Az85hff
Parts:
- C16, C22, C23, C36, C45, C46: footprint Capacitor_THT:C_Disc_D5.0mm_W2.5mm_P5.00mm -> placard:C_Disc_D5.0mm_W2.5mm_P5.00mm
- C44: footprint Capacitor_THT:CP_Radial_D6.3mm_P2.50mm -> placard:CP_Radial_D6.3mm_P2.50mm
- D10, D11, D12, D13, D14, D15, D16, D17, D9: footprint Diode_THT:D_DO-35_SOD27_P7.62mm_Horizontal -> placard:D_DO-35_SOD27_P7.62mm_Horizontal

Commit message: Schematic: rename buses to ADDR / DATABUS / D, wire the shared port outputs
- Address bus A15:A0 is now ADDR15:ADDR0, the data bus D7:D0 is DATABUS7:DATABUS0
  and the D register's outputs DR7:DR0 are D7:D0 (main board and both cartridges).
- Shared port sheet: U38's outputs P_SCK, P_MOSI, P_CS, P_PS2D and K0 are wired
  to the SNES pads, the SD dividers and the PS/2 hold diodes (K0 -> D6 ->
  keyboard CLK).  J3 now sits level with U38's SCK/MOSI pins, J2 above it.
- Parts moved so the longer labels fit: U3/U4 and the PC bus, U18, U22, U11,
  U31, U32, RN1, R5-R12; expansion slots in two rows.
- SCHEMATIC_PLAN.md: the bus names.

Co-Authored-By: Claude Opus 5.5 <noreply@anthropic.com>
Claude-Session: https://claude.ai/code/session_01DnW5SUv7E4nz9tGtPvD1qV
Connections:
- net D0 renamed DATABUS0
- net D1 renamed DATABUS1
- net D2 renamed DATABUS2
- net D3 renamed DATABUS3
- net D4 renamed DATABUS4
- net D5 renamed DATABUS5
- net D6 renamed DATABUS6
- net D7 renamed DATABUS7
Other:
- moved on the sheet: C22, U22

Commit message: Label the two 377 types on the board; red/green VGA DAC to E24 values
- Board silkscreen: "74F377" above U18-U22 and "74HCT377" above U23
  (bold 1.5 mm, outside the sockets so they stay visible with the
  sockets fitted); title block date 2026-10-28.
- BRINGUP.md: "Two kinds of 377" note and marking checks at U22, U23
  and U18. KITTING.md: CD74HCT377E packed in its own "U23 only" bag.
- Red/green DAC R14-R19: 3.3k / 1.6k / 820 (were 3.24k / 1.69k / 825);
  blue stays 1.43k / 715. Schematic, board values, BOM, COLORS.md and
  BRINGUP.md updated.

Co-Authored-By: Claude Opus 5.5 <noreply@anthropic.com>
Claude-Session: https://claude.ai/code/session_01DnW5STXEXm5h75y8sthpiM
Parts:
- R14, R17: value 3.24k -> 3.3k; MPN MFR-25FBF52-3K24 -> MFR-25FBF52-3K3
- R15, R18: value 1.69k -> 1.6k; MPN MFR-25FBF52-1K69 -> MFR-25FBF52-1K6
- R16, R19: value 825 -> 820; MPN MFR-25FBF52-825R -> MFR-25FBF52-820R
