File: kicad/placard.kicad_pcb (KiCad board)
At the start: 4 copper layers, 289.6 x 139.7 mm, 0 parts

Commit message: Main board layout: 290 x 140 mm outline, dimensions, connectors and slots placed
gen_kicad_pcb.py places the outline, dimensions, mounting holes, back-edge
I/O (USB-C, audio, VGA, PS/2), left-side SW1/SW2/SD, right-side SNES ports,
cartridge slot J8, expansion slots J9-J12 and keyboard header J1, linked to
the schematic symbols, and draws docs/placard_board_layout.png.
gen_kicad_connectors.py writes preliminary footprints for the parts KiCad
has none for; the schematic generator now assigns all connector footprints.

Co-Authored-By: Claude Opus 5.5 (1M context) <noreply@anthropic.com>
Claude-Session: https://claude.ai/code/session_013qXQudFqhMaBbYKyavQCXN
Parts:
- added H1: M3, MountingHole:MountingHole_3.2mm_M3_Pad_Via, F.Cu at (55.0, 55.0)
- added H2: M3, MountingHole:MountingHole_3.2mm_M3_Pad_Via, F.Cu at (335.0, 55.0)
- added H3: M3, MountingHole:MountingHole_3.2mm_M3_Pad_Via, F.Cu at (55.0, 185.0)
- added H4: M3, MountingHole:MountingHole_3.2mm_M3_Pad_Via, F.Cu at (335.0, 185.0)
- added H5: M3, MountingHole:MountingHole_3.2mm_M3_Pad_Via, F.Cu at (195.0, 185.0)
- added H6: M3, MountingHole:MountingHole_3.2mm_M3_Pad_Via, F.Cu at (290.0, 55.0)
- added J1: Keyboard (2x10 box), Connector_IDC:IDC-Header_2x10_P2.54mm_Vertical, F.Cu at (183.6, 133.3)
- added J10: Slot 2, placard:CardEdge_2x20_P2.54mm_Vertical, F.Cu at (112.3, 113.1)
- added J11: Slot 3, placard:CardEdge_2x20_P2.54mm_Vertical, F.Cu at (132.6, 113.1)
- added J12: Slot 4, placard:CardEdge_2x20_P2.54mm_Vertical, F.Cu at (153.0, 113.1)
- added J13: USB4125-GF-A, Connector_USB:USB_C_Receptacle_GCT_USB4125-xx-x_6P_TopMnt_Horizontal, F.Cu at (66.0, 53.4)
- added J2: SNES pad, placard:SNES_Pad_Socket_Horizontal, F.Cu at (340.0, 72.0)
- added J3: SNES pad, placard:SNES_Pad_Socket_Horizontal, F.Cu at (340.0, 100.0)
- added J4: SD (SPI), Connector_Card:SD_Kyocera_145638009511859+, F.Cu at (67.5, 109.5)
- added J5: PS/2 kbd + mouse, placard:PS2_Kycon_KMDGX-6S-6S-S4N, F.Cu at (255.0, 50.0)
- added J6: 3.5 mm, Connector_Audio:Jack_3.5mm_CUI_SJ1-3523N_Horizontal, F.Cu at (185.0, 54.5)
- added J7: VGA, Connector_Dsub:DSUB-15-HD_Female_Horizontal_P2.29x1.98mm_EdgePinOffset3.03mm_Housed_MountingHolesOffset4.94mm, F.Cu at (210.7, 57.0)
- added J8: Molex 87715-9106, placard:Molex_87715-9106_PCIe_x4_Vertical, F.Cu at (208.5, 105.0)
- added J9: Slot 1, placard:CardEdge_2x20_P2.54mm_Vertical, F.Cu at (92.0, 113.1)
- added SW1: ANT11TFHQE, placard:SW_Toggle_CIT_ANT11TFHQE, F.Cu at (50.0, 68.0)
- added SW2: E112SD1A3QE, placard:SW_Push_CK_E112SD1A3QE, F.Cu at (50.0, 84.0)
Other:
- board size 289.6 x 139.7 mm -> 290 x 140 mm
- board text added: "BACK"
- board text added: "Dimensions in mm from the back left corner to connector centre lines (edge connectors: middle of the face on the edge)"
- board text added: "EXPANSION BAY: cards stand up through the case top"
- board text added: "FRONT (keyboard side)"
- board text added: "Flat case top: user connectors, cartridge and cards in the back 75 mm"
- board text added: "H1-H6: M3 mounting holes, 3.2 mm, 5 mm in from the edges: (5,5) (285,5) (5,135) (285,135) (145,135) (240,5)"
- board text added: "J9-J12 at 20.32 (0.8") pitch"
- board text added: "KEYBOARD ABOVE (front 65 mm): low parts only"
- board text added: "LEFT SIDE"
- board text added: "PLACARD main board: 4 layers (In1 GND, In2 +5V), 1.6 mm, 290 x 140 mm, 3 mm corner radius"
- board text added: "PRELIMINARY footprints (check datasheets): J2 J3 J5 J8 J9-J12 SW1 SW2, see src/scripts/gen_kicad_connectors.py"
- board text added: "RIGHT SIDE"
- board text added: "SNES ports on the right side toward the back: not settled (the front is under the keyboard)"
- board text added: "cartridge shell"
- board text removed: "Placeholder outline 11.4 x 5.5 in (hardware/pcb_size_estimate.md)"

Commit message: Part numbers for the remaining parts; J6 Tensility 54-00174; optional J1 and J9-J12
Every schematic part gets Manufacturer/MPN: Yageo MFR-25 resistors by value,
Bourns 4609X networks, KEMET/TDK ceramics, Panasonic FR electrolytics, ECS
oscillator, Assmann VGA, Sullins headers, Wurth box header, Cherry switches.
Sockets get On Shore numbers (0.3" 24/28-pin are ED241DT/ED281DT; ED28DT is
0.6"). J6 becomes the Tensility 54-00174 TRRS jack with a footprint drawn
from its datasheet. Digi-Key prices from Justin for the oscillator, VGA and
audio jack. The expansion slot sockets and the keyboard header are optional,
with a BOM total without them.

Co-Authored-By: Claude Opus 5.5 (1M context) <noreply@anthropic.com>
Claude-Session: https://claude.ai/code/session_01L9AkLuEg13EebxDmgXsaEp
Parts:
- J6: footprint Connector_Audio:Jack_3.5mm_CUI_SJ1-3523N_Horizontal -> placard:Jack_3.5mm_Tensility_54-00174_Horizontal
- moved J6 4.50 mm to (185.0, 50.0), turned to 0 degrees

Commit message: Reset via relay: K1 G5LE-1 NC contact carries 5 V, tactile SW2 drives the coil
SW2 (C&K PTS645VL58-2 LFS) pulls in K1 (Omron G5LE-1 DC5) from VON, so
holding it opens the 5 V line; D26 (BAT85) across the coil. Replaces the
4 A E112SD1A3QE (about $11 -> $2). C41 moves ahead of K1 onto VON so the
board side drains faster on reset. Footprint, layout, BOM and docs updated.

Co-Authored-By: Claude Opus 5.5 (1M context) <noreply@anthropic.com>
Claude-Session: https://claude.ai/code/session_01L9AkLuEg13EebxDmgXsaEp
Parts:
- SW2: value E112SD1A3QE -> PTS645VL58-2 LFS; footprint placard:SW_Push_CK_E112SD1A3QE -> Button_Switch_THT:SW_Tactile_SPST_Angled_PTS645Vx58-2LFS
- moved SW2 3.43 mm to (52.6, 86.2)

Commit message: PCB: place every main-board part as a fit test (socket and puller clearance, no routing)
gen_kicad_pcb.py now places all 192 schematic parts: chip rows by sheet,
every DIP on a _Socket footprint with 2.5 mm puller room past each end,
Cn beside Un, passive blocks; checks courtyards (own + KiCad DRC), puller
room, off-board parts, and draws docs/placard_placement.png.

Co-Authored-By: Claude Opus 5.5 (1M context) <noreply@anthropic.com>
Claude-Session: https://claude.ai/code/session_01JnVuvUvdWezUUU6Sgmg16H
Parts:
- added C1: 100n, Capacitor_THT:C_Disc_D5.0mm_W2.5mm_P5.00mm, F.Cu at (82.1, 171.0)
- added C10: 100n, Capacitor_THT:C_Disc_D5.0mm_W2.5mm_P5.00mm, F.Cu at (250.6, 155.0)
- added C11: 100n, Capacitor_THT:C_Disc_D5.0mm_W2.5mm_P5.00mm, F.Cu at (263.7, 123.0)
- added C12: 100n, Capacitor_THT:C_Disc_D5.0mm_W2.5mm_P5.00mm, F.Cu at (259.3, 187.0)
- added C13: 100n, Capacitor_THT:C_Disc_D5.0mm_W2.5mm_P5.00mm, F.Cu at (86.1, 187.0)
- added C14: 100n, Capacitor_THT:C_Disc_D5.0mm_W2.5mm_P5.00mm, F.Cu at (119.8, 187.0)
- added C15: 100n, Capacitor_THT:C_Disc_D5.0mm_W2.5mm_P5.00mm, F.Cu at (153.5, 187.0)
- added C16: 100n, Capacitor_THT:C_Disc_D5.0mm_W2.5mm_P5.00mm, F.Cu at (186.1, 86.0)
- added C17: 100n, Capacitor_THT:C_Disc_D5.0mm_W2.5mm_P5.00mm, F.Cu at (284.3, 155.0)
- added C18: 100n, Capacitor_THT:C_Disc_D5.0mm_W2.5mm_P5.00mm, F.Cu at (91.0, 139.0)
- added C19: 100n, Capacitor_THT:C_Disc_D5.0mm_W2.5mm_P5.00mm, F.Cu at (211.8, 171.0)
- added C2: 100n, Capacitor_THT:C_Disc_D5.0mm_W2.5mm_P5.00mm, F.Cu at (115.8, 171.0)
- added C20: 100n, Capacitor_THT:C_Disc_D5.0mm_W2.5mm_P5.00mm, F.Cu at (240.4, 171.0)
- added C21: 100n, Capacitor_THT:C_Disc_D5.0mm_W2.5mm_P5.00mm, F.Cu at (269.0, 171.0)
- added C22: 100n, Capacitor_THT:C_Disc_D5.0mm_W2.5mm_P5.00mm, F.Cu at (214.7, 86.0)
- added C23: 100n, Capacitor_THT:C_Disc_D5.0mm_W2.5mm_P5.00mm, F.Cu at (243.3, 86.0)
- added C25: 100n, Capacitor_THT:C_Disc_D5.0mm_W2.5mm_P5.00mm, F.Cu at (292.3, 123.0)
- added C26: 100n, Capacitor_THT:C_Disc_D5.0mm_W2.5mm_P5.00mm, F.Cu at (119.6, 139.0)
- added C27: 100n, Capacitor_THT:C_Disc_D5.0mm_W2.5mm_P5.00mm, F.Cu at (148.2, 139.0)
- added C29: 100n, Capacitor_THT:C_Disc_D5.0mm_W2.5mm_P5.00mm, F.Cu at (182.1, 187.0)
- added C3: 100n, Capacitor_THT:C_Disc_D5.0mm_W2.5mm_P5.00mm, F.Cu at (82.1, 155.0)
- added C31: 100n, Capacitor_THT:C_Disc_D5.0mm_W2.5mm_P5.00mm, F.Cu at (191.2, 123.0)
- added C32: 100n, Capacitor_THT:C_Disc_D5.0mm_W2.5mm_P5.00mm, F.Cu at (230.0, 123.0)
- added C35: 100n, Capacitor_THT:C_Disc_D5.0mm_W2.5mm_P5.00mm, F.Cu at (225.6, 187.0)
- added C36: 100n, Capacitor_THT:C_Disc_D5.0mm_W2.5mm_P5.00mm, F.Cu at (271.9, 86.0)
- added C37: 100n, Capacitor_THT:C_Disc_D5.0mm_W2.5mm_P5.00mm, F.Cu at (267.2, 139.0)
- added C38: 100n, Capacitor_THT:C_Disc_D5.0mm_W2.5mm_P5.00mm, F.Cu at (238.6, 139.0)
- added C39: 100n, Capacitor_THT:C_Disc_D5.0mm_W2.5mm_P5.00mm, F.Cu at (295.8, 139.0)
- added C4: 100n, Capacitor_THT:C_Disc_D5.0mm_W2.5mm_P5.00mm, F.Cu at (115.8, 155.0)
- added C40: 1u, Capacitor_THT:C_Disc_D5.0mm_W2.5mm_P5.00mm, F.Cu at (64.6, 134.5)
- added C41: 220u 10V, Capacitor_THT:CP_Radial_D8.0mm_P3.50mm, F.Cu at (66.2, 81.8)
- added C42: 1u, Capacitor_THT:C_Disc_D5.0mm_W2.5mm_P5.00mm, F.Cu at (68.0, 134.5)
- added C43: 100n, Capacitor_THT:C_Disc_D5.0mm_W2.5mm_P5.00mm, F.Cu at (292.8, 172.2)
- added C44: 220u, Capacitor_THT:CP_Radial_D6.3mm_P2.50mm, F.Cu at (299.1, 78.2)
- added C45: 15n C0G, Capacitor_THT:C_Disc_D5.0mm_W2.5mm_P5.00mm, F.Cu at (293.9, 80.8)
- added C46: 22u, Capacitor_THT:C_Disc_D5.0mm_W2.5mm_P5.00mm, F.Cu at (299.1, 72.2)
- added C5: 100n, Capacitor_THT:C_Disc_D5.0mm_W2.5mm_P5.00mm, F.Cu at (149.5, 171.0)
- added C6: 100n, Capacitor_THT:C_Disc_D5.0mm_W2.5mm_P5.00mm, F.Cu at (183.2, 171.0)
- added C7: 100n, Capacitor_THT:C_Disc_D5.0mm_W2.5mm_P5.00mm, F.Cu at (149.5, 155.0)
- added C8: 100n, Capacitor_THT:C_Disc_D5.0mm_W2.5mm_P5.00mm, F.Cu at (183.2, 155.0)
- added C9: 100n, Capacitor_THT:C_Disc_D5.0mm_W2.5mm_P5.00mm, F.Cu at (216.9, 155.0)
- added D1: BAT85, Diode_THT:D_DO-35_SOD27_P7.62mm_Horizontal, F.Cu at (162.3, 108.8)
- added D10: BAT85, Diode_THT:D_DO-35_SOD27_P7.62mm_Horizontal, F.Cu at (185.1, 108.8)
- added D11: BAT85, Diode_THT:D_DO-35_SOD27_P7.62mm_Horizontal, F.Cu at (187.9, 108.8)
- added D12: BAT85, Diode_THT:D_DO-35_SOD27_P7.62mm_Horizontal, F.Cu at (190.8, 108.8)
- added D13: BAT85, Diode_THT:D_DO-35_SOD27_P7.62mm_Horizontal, F.Cu at (193.6, 108.8)
- added D14: BAT85, Diode_THT:D_DO-35_SOD27_P7.62mm_Horizontal, F.Cu at (247.3, 108.8)
- added D15: BAT85, Diode_THT:D_DO-35_SOD27_P7.62mm_Horizontal, F.Cu at (250.1, 108.8)
- added D16: BAT85, Diode_THT:D_DO-35_SOD27_P7.62mm_Horizontal, F.Cu at (253.0, 108.8)
- added D17: BAT85, Diode_THT:D_DO-35_SOD27_P7.62mm_Horizontal, F.Cu at (255.8, 108.8)
- added D18: BAT85, Diode_THT:D_DO-35_SOD27_P7.62mm_Horizontal, F.Cu at (258.7, 108.8)
- added D19: BAT85, Diode_THT:D_DO-35_SOD27_P7.62mm_Horizontal, F.Cu at (261.5, 108.8)
- added D2: BAT85, Diode_THT:D_DO-35_SOD27_P7.62mm_Horizontal, F.Cu at (165.1, 108.8)
- added D20: BAT85, Diode_THT:D_DO-35_SOD27_P7.62mm_Horizontal, F.Cu at (264.4, 108.8)
- added D21: BAT85, Diode_THT:D_DO-35_SOD27_P7.62mm_Horizontal, F.Cu at (267.2, 108.8)
- added D22: BAT85, Diode_THT:D_DO-35_SOD27_P7.62mm_Horizontal, F.Cu at (259.4, 77.1)
- added D23: BAT85, Diode_THT:D_DO-35_SOD27_P7.62mm_Horizontal, F.Cu at (262.3, 77.1)
- added D24: BAT85, Diode_THT:D_DO-35_SOD27_P7.62mm_Horizontal, F.Cu at (265.1, 77.1)
- added D25: BAT85, Diode_THT:D_DO-35_SOD27_P7.62mm_Horizontal, F.Cu at (268.0, 77.1)
- added D26: BAT85, Diode_THT:D_DO-35_SOD27_P7.62mm_Horizontal, F.Cu at (64.6, 89.2)
- added D27: BAT85, Diode_THT:D_DO-35_SOD27_P7.62mm_Horizontal, F.Cu at (270.8, 77.1)
- added D28: BAT85, Diode_THT:D_DO-35_SOD27_P7.62mm_Horizontal, F.Cu at (273.7, 77.1)
- added D29: BAT85, Diode_THT:D_DO-35_SOD27_P7.62mm_Horizontal, F.Cu at (276.5, 77.1)
- added D3: BAT85, Diode_THT:D_DO-35_SOD27_P7.62mm_Horizontal, F.Cu at (168.0, 108.8)
- added D30: 1N4148, Diode_THT:D_DO-35_SOD27_P7.62mm_Horizontal, F.Cu at (279.4, 77.1)
- added D31: 1N4148, Diode_THT:D_DO-35_SOD27_P7.62mm_Horizontal, F.Cu at (282.2, 77.1)
- added D32: 1N4148, Diode_THT:D_DO-35_SOD27_P7.62mm_Horizontal, F.Cu at (285.1, 77.1)
- added D33: 1N4148, Diode_THT:D_DO-35_SOD27_P7.62mm_Horizontal, F.Cu at (287.9, 77.1)
- added D34: 1N4148, Diode_THT:D_DO-35_SOD27_P7.62mm_Horizontal, F.Cu at (290.8, 77.1)
- added D35: 1N4148, Diode_THT:D_DO-35_SOD27_P7.62mm_Horizontal, F.Cu at (293.9, 73.3)
- added D4: BAT85, Diode_THT:D_DO-35_SOD27_P7.62mm_Horizontal, F.Cu at (170.8, 108.8)
- added D5: BAT85, Diode_THT:D_DO-35_SOD27_P7.62mm_Horizontal, F.Cu at (173.7, 108.8)
- added D6: BAT85, Diode_THT:D_DO-35_SOD27_P7.62mm_Horizontal, F.Cu at (176.5, 108.8)
- added D7: SA5.0A, Diode_THT:D_DO-15_P10.16mm_Horizontal, F.Cu at (83.4, 89.9)
- added D8: BAT85, Diode_THT:D_DO-35_SOD27_P7.62mm_Horizontal, F.Cu at (179.4, 108.8)
- added D9: BAT85, Diode_THT:D_DO-35_SOD27_P7.62mm_Horizontal, F.Cu at (182.2, 108.8)
- added F1: 3 A hold, Fuse:Fuse_Bourns_MF-RG300, F.Cu at (73.8, 84.3)
- added JP1: STALL, Connector_PinHeader_2.54mm:PinHeader_1x02_P2.54mm_Vertical, F.Cu at (302.4, 146.0)
- added JP2: RUN, Connector_PinHeader_2.54mm:PinHeader_1x02_P2.54mm_Vertical, F.Cu at (302.4, 150.0)
- added K1: G5LE-1 DC5, Relay_THT:Relay_SPDT_Omron-G5LE-1, F.Cu at (66.0, 68.0)
- added NT1: AGND tie, NetTie:NetTie-2_THT_Pad0.3mm, F.Cu at (77.4, 90.0)
- added R1: 5.1k, Resistor_THT:R_Axial_DIN0207_L6.3mm_D2.5mm_P10.16mm_Horizontal, F.Cu at (73.4, 53.2)
- added R10: 47, Resistor_THT:R_Axial_DIN0207_L6.3mm_D2.5mm_P10.16mm_Horizontal, F.Cu at (287.2, 185.1)
- added R11: 47, Resistor_THT:R_Axial_DIN0207_L6.3mm_D2.5mm_P10.16mm_Horizontal, F.Cu at (290.5, 185.1)
- added R12: 47, Resistor_THT:R_Axial_DIN0207_L6.3mm_D2.5mm_P10.16mm_Horizontal, F.Cu at (293.9, 185.1)
- added R13: 10k, Resistor_THT:R_Axial_DIN0207_L6.3mm_D2.5mm_P10.16mm_Horizontal, F.Cu at (308.6, 153.1)
- added R14: 3.24k, Resistor_THT:R_Axial_DIN0207_L6.3mm_D2.5mm_P10.16mm_Horizontal, F.Cu at (162.5, 78.3)
- added R15: 1.69k, Resistor_THT:R_Axial_DIN0207_L6.3mm_D2.5mm_P10.16mm_Horizontal, F.Cu at (165.9, 78.3)
- added R16: 825, Resistor_THT:R_Axial_DIN0207_L6.3mm_D2.5mm_P10.16mm_Horizontal, F.Cu at (169.2, 78.3)
- added R17: 3.24k, Resistor_THT:R_Axial_DIN0207_L6.3mm_D2.5mm_P10.16mm_Horizontal, F.Cu at (172.6, 78.3)
- added R18: 1.69k, Resistor_THT:R_Axial_DIN0207_L6.3mm_D2.5mm_P10.16mm_Horizontal, F.Cu at (175.9, 78.3)
- added R19: 825, Resistor_THT:R_Axial_DIN0207_L6.3mm_D2.5mm_P10.16mm_Horizontal, F.Cu at (179.3, 78.3)
- added R2: 5.1k, Resistor_THT:R_Axial_DIN0207_L6.3mm_D2.5mm_P10.16mm_Horizontal, F.Cu at (73.4, 56.6)
- added R20: 1.43k, Resistor_THT:R_Axial_DIN0207_L6.3mm_D2.5mm_P10.16mm_Horizontal, F.Cu at (182.6, 78.3)
- added R21: 715, Resistor_THT:R_Axial_DIN0207_L6.3mm_D2.5mm_P10.16mm_Horizontal, F.Cu at (186.0, 78.3)
- added R22: 2.2, Resistor_THT:R_Axial_DIN0207_L6.3mm_D2.5mm_P10.16mm_Horizontal, F.Cu at (189.3, 78.3)
- added R23: 2k, Resistor_THT:R_Axial_DIN0207_L6.3mm_D2.5mm_P10.16mm_Horizontal, F.Cu at (192.7, 78.3)
- added R24: 2k, Resistor_THT:R_Axial_DIN0207_L6.3mm_D2.5mm_P10.16mm_Horizontal, F.Cu at (196.0, 78.3)
- added R25: 2k, Resistor_THT:R_Axial_DIN0207_L6.3mm_D2.5mm_P10.16mm_Horizontal, F.Cu at (199.4, 78.3)
- added R26: 2k, Resistor_THT:R_Axial_DIN0207_L6.3mm_D2.5mm_P10.16mm_Horizontal, F.Cu at (202.7, 78.3)
- added R27: 2k, Resistor_THT:R_Axial_DIN0207_L6.3mm_D2.5mm_P10.16mm_Horizontal, F.Cu at (206.1, 78.3)
- added R28: 2k, Resistor_THT:R_Axial_DIN0207_L6.3mm_D2.5mm_P10.16mm_Horizontal, F.Cu at (209.4, 78.3)
- added R29: 2k, Resistor_THT:R_Axial_DIN0207_L6.3mm_D2.5mm_P10.16mm_Horizontal, F.Cu at (212.8, 78.3)
- added R3: 10k, Resistor_THT:R_Axial_DIN0207_L6.3mm_D2.5mm_P10.16mm_Horizontal, F.Cu at (295.4, 153.1)
- added R30: 2k, Resistor_THT:R_Axial_DIN0207_L6.3mm_D2.5mm_P10.16mm_Horizontal, F.Cu at (216.1, 78.3)
- added R31: 2k, Resistor_THT:R_Axial_DIN0207_L6.3mm_D2.5mm_P10.16mm_Horizontal, F.Cu at (219.5, 78.3)
- added R32: 1k, Resistor_THT:R_Axial_DIN0207_L6.3mm_D2.5mm_P10.16mm_Horizontal, F.Cu at (222.8, 78.3)
- added R33: 1k, Resistor_THT:R_Axial_DIN0207_L6.3mm_D2.5mm_P10.16mm_Horizontal, F.Cu at (226.2, 78.3)
- added R34: 1k, Resistor_THT:R_Axial_DIN0207_L6.3mm_D2.5mm_P10.16mm_Horizontal, F.Cu at (229.5, 78.3)
- added R35: 1k, Resistor_THT:R_Axial_DIN0207_L6.3mm_D2.5mm_P10.16mm_Horizontal, F.Cu at (232.9, 78.3)
- added R36: 1k, Resistor_THT:R_Axial_DIN0207_L6.3mm_D2.5mm_P10.16mm_Horizontal, F.Cu at (236.2, 78.3)
- added R37: 1k, Resistor_THT:R_Axial_DIN0207_L6.3mm_D2.5mm_P10.16mm_Horizontal, F.Cu at (239.6, 78.3)
- added R38: 1k, Resistor_THT:R_Axial_DIN0207_L6.3mm_D2.5mm_P10.16mm_Horizontal, F.Cu at (242.9, 78.3)
- added R39: 10k, Resistor_THT:R_Axial_DIN0207_L6.3mm_D2.5mm_P10.16mm_Horizontal, F.Cu at (246.3, 78.3)
- added R4: 10k, Resistor_THT:R_Axial_DIN0207_L6.3mm_D2.5mm_P10.16mm_Horizontal, F.Cu at (298.8, 153.1)
- added R40: 10k, Resistor_THT:R_Axial_DIN0207_L6.3mm_D2.5mm_P10.16mm_Horizontal, F.Cu at (273.1, 101.7)
- added R41: 10k, Resistor_THT:R_Axial_DIN0207_L6.3mm_D2.5mm_P10.16mm_Horizontal, F.Cu at (273.1, 105.0)
- added R42: 1.8k, Resistor_THT:R_Axial_DIN0207_L6.3mm_D2.5mm_P10.16mm_Horizontal, F.Cu at (273.1, 108.3)
- added R43: 1.8k, Resistor_THT:R_Axial_DIN0207_L6.3mm_D2.5mm_P10.16mm_Horizontal, F.Cu at (285.7, 101.7)
- added R44: 1.8k, Resistor_THT:R_Axial_DIN0207_L6.3mm_D2.5mm_P10.16mm_Horizontal, F.Cu at (285.7, 105.0)
- added R45: 3.3k, Resistor_THT:R_Axial_DIN0207_L6.3mm_D2.5mm_P10.16mm_Horizontal, F.Cu at (285.7, 108.3)
- added R46: 3.3k, Resistor_THT:R_Axial_DIN0207_L6.3mm_D2.5mm_P10.16mm_Horizontal, F.Cu at (298.3, 101.7)
- added R47: 3.3k, Resistor_THT:R_Axial_DIN0207_L6.3mm_D2.5mm_P10.16mm_Horizontal, F.Cu at (298.3, 105.0)
- added R48: 10k, Resistor_THT:R_Axial_DIN0207_L6.3mm_D2.5mm_P10.16mm_Horizontal, F.Cu at (298.3, 108.3)
- added R49: 4.7k, Resistor_THT:R_Axial_DIN0207_L6.3mm_D2.5mm_P10.16mm_Horizontal, F.Cu at (310.9, 101.7)
- added R5: 47, Resistor_THT:R_Axial_DIN0207_L6.3mm_D2.5mm_P10.16mm_Horizontal, F.Cu at (270.4, 185.1)
- added R50: 4.7k, Resistor_THT:R_Axial_DIN0207_L6.3mm_D2.5mm_P10.16mm_Horizontal, F.Cu at (310.9, 105.0)
- added R51: 1k, Resistor_THT:R_Axial_DIN0207_L6.3mm_D2.5mm_P10.16mm_Horizontal, F.Cu at (312.0, 153.1)
- added R52: 1k, Resistor_THT:R_Axial_DIN0207_L6.3mm_D2.5mm_P10.16mm_Horizontal, F.Cu at (315.3, 153.1)
- added R53: 1k, Resistor_THT:R_Axial_DIN0207_L6.3mm_D2.5mm_P10.16mm_Horizontal, F.Cu at (318.7, 153.1)
- added R54: 1k, Resistor_THT:R_Axial_DIN0207_L6.3mm_D2.5mm_P10.16mm_Horizontal, F.Cu at (322.0, 153.1)
- added R55: 4.7k, Resistor_THT:R_Axial_DIN0207_L6.3mm_D2.5mm_P10.16mm_Horizontal, F.Cu at (310.9, 108.3)
- added R56: 910, Resistor_THT:R_Axial_DIN0207_L6.3mm_D2.5mm_P10.16mm_Horizontal, F.Cu at (249.6, 78.3)
- added R57: 910, Resistor_THT:R_Axial_DIN0207_L6.3mm_D2.5mm_P10.16mm_Horizontal, F.Cu at (253.0, 78.3)
- added R58: 910, Resistor_THT:R_Axial_DIN0207_L6.3mm_D2.5mm_P10.16mm_Horizontal, F.Cu at (256.3, 78.3)
- added R6: 47, Resistor_THT:R_Axial_DIN0207_L6.3mm_D2.5mm_P10.16mm_Horizontal, F.Cu at (273.8, 185.1)
- added R7: 47, Resistor_THT:R_Axial_DIN0207_L6.3mm_D2.5mm_P10.16mm_Horizontal, F.Cu at (277.1, 185.1)
- added R8: 47, Resistor_THT:R_Axial_DIN0207_L6.3mm_D2.5mm_P10.16mm_Horizontal, F.Cu at (280.5, 185.1)
- added R9: 47, Resistor_THT:R_Axial_DIN0207_L6.3mm_D2.5mm_P10.16mm_Horizontal, F.Cu at (283.8, 185.1)
- added RN1: 10k, Resistor_THT:R_Array_SIP9, F.Cu at (299.6, 178.2)
- added RN2: 4.7k, Resistor_THT:R_Array_SIP9, F.Cu at (299.6, 181.8)
- added U1: ATF22V10C-7PX, Package_DIP:DIP-24_W7.62mm_Socket, F.Cu at (59.6, 167.8)
- added U10: ATF22V10C-7PX, Package_DIP:DIP-24_W7.62mm_Socket, F.Cu at (228.1, 151.8)
- added U11: ATF22V10C-7PX, Package_DIP:DIP-24_W7.62mm_Socket, F.Cu at (241.2, 119.8)
- added U12: ATF22V10C-7PX, Package_DIP:DIP-24_W7.62mm_Socket, F.Cu at (236.8, 183.8)
- added U13: ATF22V10C-10PU, Package_DIP:DIP-24_W7.62mm_Socket, F.Cu at (63.6, 183.8)
- added U14: ATF22V10C-10PU, Package_DIP:DIP-24_W7.62mm_Socket, F.Cu at (97.3, 183.8)
- added U15: ATF22V10C-7PX, Package_DIP:DIP-24_W7.62mm_Socket, F.Cu at (131.0, 183.8)
- added U16: ATF22V10C-10PU, Package_DIP:DIP-24_W7.62mm_Socket, F.Cu at (163.6, 96.8)
- added U17: ATF22V10C-7PX, Package_DIP:DIP-24_W7.62mm_Socket, F.Cu at (261.8, 151.8)
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Other:
- board text added: "Behind the keyboard: memory under the cartridge slot, video out chips, video/audio passives along the back edge, shared-port protection beside J8; power at the back left"
- board text added: "Chip rows, front to back: video timing + data bus resistors and networks | control + ALU + oscillator | PC + address mux | data bus + shared port (J1 between)"
- board text added: "Dashed boxes: expansion bay (cards stand up through the case top) and the cartridge shell around J8"
- board text added: "Dashed line: keyboard's back edge; the keyboard lies over the front 65 mm (low parts only); the back 75 mm is under the flat case top (user connectors, cartridge, cards)"
- board text added: "Placement test (no routing): every chip socketed (KiCad _Socket footprints); hatched boxes at the socket ends = 2.5 mm chip-puller room, kept clear"
- board text removed: "EXPANSION BAY: cards stand up through the case top"
- board text removed: "Flat case top: user connectors, cartridge and cards in the back 75 mm"
- board text removed: "KEYBOARD ABOVE (front 65 mm): low parts only"
- board text removed: "cartridge shell"

Commit message: Every PLD is an ATF22V10C-7PX (one part number)
Justin: switch the seven main-board -10PU PLDs (Branch, PC x2, H, V,
color decoder, audio slot) and the cartridge loader to the -7PX, for one
part number to buy, program and kit (.52 more per main board). Symbols,
schematics, PDFs, BOM, docs and PLD comments updated; CHIPS.md keeps the
grade each PLD could use.

Co-Authored-By: Claude Opus 5.5 (1M context) <noreply@anthropic.com>
Claude-Session: https://claude.ai/code/session_01JnVuvUvdWezUUU6Sgmg16H
Parts:
- U13, U14, U16, U2, U3, U35, U4: value ATF22V10C-10PU -> ATF22V10C-7PX

Commit message: J13: USB4125 footprint with longer SMD pads for hand soldering
New placard:USB_C_Receptacle_GCT_USB4125_6P_HandSolder, made by
gen_kicad_connectors.py from KiCad's USB4125 footprint with the six SMD
pads lengthened 1.5 mm away from the board edge (inner ends unchanged),
so the iron has room to touch each pad. Symbol, power sheet and board
now use it; board drawings regenerated.

Co-Authored-By: Claude Opus 5.5 (1M context) <noreply@anthropic.com>
Claude-Session: https://claude.ai/code/session_01SPs5Hx9ixxAAqtEGqiE4Ba
Parts:
- J13: footprint Connector_USB:USB_C_Receptacle_GCT_USB4125-xx-x_6P_TopMnt_Horizontal -> placard:USB_C_Receptacle_GCT_USB4125_6P_HandSolder

Commit message: PCB: 290 x 290 mm board, parts spread out for kit builders
Justin: the placement was too congested for amateur assembly; keep the
290 mm width and double the depth. Six chip rows 35 mm apart, each spread
across the width; 6 mm minimum between sockets, 1.5 mm between passives,
decaps 1 mm from their chips; keyboard header J1 in the front row; two
more mounting holes at mid-depth (H7, H8). No courtyard overlaps.

Co-Authored-By: Claude Opus 5.5 (1M context) <noreply@anthropic.com>
Claude-Session: https://claude.ai/code/session_01JnVuvUvdWezUUU6Sgmg16H
Parts:
- added H7: M3, MountingHole:MountingHole_3.2mm_M3_Pad_Via, F.Cu at (55.0, 195.0)
- added H8: M3, MountingHole:MountingHole_3.2mm_M3_Pad_Via, F.Cu at (335.0, 195.0)
- moved C38 228.2 mm to (112.1, 328.9)
- moved U38 227.4 mm to (89.6, 324.8)
- moved C37 226.3 mm to (144.2, 328.9)
- moved U37 225.5 mm to (126.8, 324.8)
- moved C39 224.4 mm to (176.3, 328.9)
- moved U39 223.6 mm to (158.9, 324.8)
- moved J1 196.8 mm to (238.6, 322.3)
- moved C42 189.1 mm to (72.4, 323.5)
- moved C40 189.0 mm to (67.8, 323.5)
- moved U40 189.0 mm to (62.8, 322.3)
- moved C12 179.0 mm to (84.1, 223.9)
- moved U12 178.9 mm to (61.6, 219.8)
- moved U15 172.8 mm to (300.4, 149.8)
- moved C26 172.6 mm to (269.9, 223.9)
- moved C15 172.6 mm to (322.9, 153.9)
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Other:
- board size 290 x 140 mm -> 290 x 290 mm
- board text added: "Back: video/audio passives along the back edge, shared-port protection and pull-ups around J8, power at the back left"
- board text added: "Chip rows, back to front: video | audio slot, oscillator, memory | I/O decode, control, data bus | ALU, data bus | PC + address mux | shared port + keyboard header J1"
- board text added: "Dashed line: keyboard's back edge; the keyboard lies over the front 65 mm (low parts only); the back 225 mm is under the flat case top (user connectors, cartridge, cards)"
- board text added: "H1-H8: M3 mounting holes, 3.2 mm, 5 mm in from the edges: (5,5) (285,5) (5,285) (285,285) (145,285) (240,5) (5,145) (285,145)"
- board text added: "PLACARD main board: 4 layers (In1 GND, In2 +5V), 1.6 mm, 290 x 290 mm, 3 mm corner radius"
- board text removed: "Behind the keyboard: memory under the cartridge slot, video out chips, video/audio passives along the back edge, shared-port protection beside J8; power at the back left"
- board text removed: "Chip rows, front to back: video timing + data bus resistors and networks | control + ALU + oscillator | PC + address mux | data bus + shared port (J1 between)"
- board text removed: "Dashed line: keyboard's back edge; the keyboard lies over the front 65 mm (low parts only); the back 75 mm is under the flat case top (user connectors, cartridge, cards)"
- board text removed: "H1-H6: M3 mounting holes, 3.2 mm, 5 mm in from the edges: (5,5) (285,5) (5,135) (285,135) (145,135) (240,5)"
- board text removed: "PLACARD main board: 4 layers (In1 GND, In2 +5V), 1.6 mm, 290 x 140 mm, 3 mm corner radius"

Commit message: Check in Justin's local work: board, project, CLAUDE.md, PLD files
- kicad/placard.kicad_pcb: Justin's hand layout and routing as of
  2026-10-25 with the silkscreen trimmed off pads and the board edge
  (DRC clean in KiCad 9).
- kicad/placard.kicad_pro: KiCad 9 project settings saved with it.
- CLAUDE.md, reference/ATF22V10C.pdf, src/pld/Counter499EN.si,
  src/pld/gen_vectors.py: files that were only on Justin's PC.

Co-Authored-By: Claude Opus 5.5 (1M context) <noreply@anthropic.com>
Claude-Session: https://claude.ai/code/session_01393wxHftXkXBUKTbGjayj9
Parts:
- removed C37, C39: 100n, Capacitor_THT:C_Disc_D5.0mm_W2.5mm_P5.00mm
- removed the D10 at (194.7, 108.8)
- removed the D11 at (198.7, 108.8)
- removed the D12 at (247.3, 108.8)
- removed the D13 at (251.3, 108.8)
- removed the D14 at (255.4, 108.8)
- removed the D15 at (259.4, 108.8)
- removed the D16 at (263.5, 108.8)
- removed the D17 at (267.5, 108.8)
- removed D20, D21, D22, D23, D24, D25: BAT85, Diode_THT:D_DO-35_SOD27_P7.62mm_Horizontal
- removed the D8 at (186.6, 108.8)
- removed the D9 at (190.6, 108.8)
- removed J1: Keyboard (2x10 box), Connector_IDC:IDC-Header_2x10_P2.54mm_Vertical
- removed RN2: 4.7k, Resistor_THT:R_Array_SIP9
- removed U37: SN74HC574N, Package_DIP:DIP-20_W7.62mm_Socket
- removed U39: SN74F541N, Package_DIP:DIP-20_W7.62mm_Socket
- added C42: 100n, Capacitor_THT:C_Disc_D5.0mm_W2.5mm_P5.00mm, F.Cu at (170.3, 137.5)
- added R59: 1k, placard:R_Axial_DIN0207_L6.3mm_D2.5mm_P10.16mm_Horizontal_Value, F.Cu at (54.8, 167.7)
- added R60: 22k, placard:R_Axial_DIN0207_L6.3mm_D2.5mm_P10.16mm_Horizontal_Value, F.Cu at (310.0, 98.1)
- added U42: ATF22V10C-7PX, placard:DIP-24_W7.62mm_Socket_Puller, F.Cu at (175.7, 143.5)
- D18: value BAT85 -> LTL2R3KRD-EM; footprint Diode_THT:D_DO-35_SOD27_P7.62mm_Horizontal -> LED_THT:LED_D5.0mm
- F1: footprint Fuse:Fuse_Bourns_MF-RG300 -> placard:Fuse_Bourns_MF-RG300
- J4: footprint Connector_Card:SD_Kyocera_145638009511859+ -> placard:SD_Kyocera_145638009511859+
- J7: footprint Connector_Dsub:DSUB-15-HD_Female_Horizontal_P2.29x1.98mm_EdgePinOffset3.03mm_Housed_MountingHolesOffset4.94mm -> placard:DSUB-15-HD_Female_Horizontal_P2.29x1.98mm_EdgePinOffset3.03mm_Housed_MountingHolesOffset4.94mm
- R1, R10, R11, R12, R13, R14, R15, R16, R17, R18, R19, R2, R20, R21, R22, R23, R24, R25, R26, R27, R28, R29, R3, R30, R31, R32, R33, R34, R35, R36, R37, R38, R39, R4, R40, R41, R42, R43, R44, R45, R46, R47, R48, R49, R5, R50, R51, R52, R53, R54, R55, R56, R57, R58, R6, R7, R8, R9: footprint Resistor_THT:R_Axial_DIN0207_L6.3mm_D2.5mm_P10.16mm_Horizontal -> placard:R_Axial_DIN0207_L6.3mm_D2.5mm_P10.16mm_Horizontal_Value
- SW2: footprint Button_Switch_THT:SW_Tactile_SPST_Angled_PTS645Vx58-2LFS -> placard:SW_Tactile_SPST_Angled_PTS645Vx58-2LFS
- U1, U10, U11, U12, U13, U14, U15, U16, U17, U2, U3, U35, U38, U4, U5, U6, U7, U8, U9: footprint Package_DIP:DIP-24_W7.62mm_Socket -> placard:DIP-24_W7.62mm_Socket_Puller
- U18, U19, U20, U21, U22, U23, U25, U26, U27, U29, U36: footprint Package_DIP:DIP-20_W7.62mm_Socket -> placard:DIP-20_W7.62mm_Socket_Puller
- U31, U32: footprint Package_DIP:DIP-28_W7.62mm_Socket -> placard:DIP-28_W7.62mm_Socket_Puller
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- renumbered C42 to C47, D28 to D10, D29 to D11, D30 to D12, D31 to D13, D32 to D14, D33 to D15, D34 to D16, D35 to D17, D26 to D8, D27 to D9
Connections:
- C1 pad 1: (no net) -> +5V
- C1 pad 2: (no net) -> GND
- C10 pad 1: (no net) -> +5V
- C10 pad 2: (no net) -> GND
- C11 pad 1: (no net) -> +5V
- C11 pad 2: (no net) -> GND
- C12 pad 1: (no net) -> +5V
- C12 pad 2: (no net) -> GND
- C13 pad 1: (no net) -> +5V
- C13 pad 2: (no net) -> GND
- C14 pad 1: (no net) -> +5V
- C14 pad 2: (no net) -> GND
- C15 pad 1: (no net) -> +5V
- C15 pad 2: (no net) -> GND
- C16 pad 1: (no net) -> +5V
- C16 pad 2: (no net) -> GND
- C17 pad 1: (no net) -> +5V
- C17 pad 2: (no net) -> GND
- C18 pad 1: (no net) -> +5V
- C18 pad 2: (no net) -> GND
- C19 pad 1: (no net) -> +5V
- C19 pad 2: (no net) -> GND
- C2 pad 1: (no net) -> +5V
- C2 pad 2: (no net) -> GND
- C20 pad 1: (no net) -> +5V
- C20 pad 2: (no net) -> GND
- C21 pad 1: (no net) -> +5V
- C21 pad 2: (no net) -> GND
- C22 pad 1: (no net) -> +5V
- C22 pad 2: (no net) -> GND
- C23 pad 1: (no net) -> +5V
- C23 pad 2: (no net) -> GND
- C25 pad 1: (no net) -> +5V
- C25 pad 2: (no net) -> GND
- C26 pad 1: (no net) -> +5V
- C26 pad 2: (no net) -> GND
- C27 pad 1: (no net) -> +5V
- C27 pad 2: (no net) -> GND
- C29 pad 1: (no net) -> +5V
- C29 pad 2: (no net) -> GND
- C3 pad 1: (no net) -> +5V
- C3 pad 2: (no net) -> GND
- C31 pad 1: (no net) -> +5V
- C31 pad 2: (no net) -> GND
- C32 pad 1: (no net) -> +5V
- C32 pad 2: (no net) -> GND
- C35 pad 1: (no net) -> +5V
- C35 pad 2: (no net) -> GND
- C36 pad 1: (no net) -> /Video and audio out/DAC_5V
- C36 pad 2: (no net) -> GNDA
- C38 pad 1: (no net) -> +5V
- C38 pad 2: (no net) -> GND
- C4 pad 1: (no net) -> +5V
- C4 pad 2: (no net) -> GND
- C40 pad 1: (no net) -> +5V
- C40 pad 2: (no net) -> GND
- C41 pad 1: (no net) -> Net-(SW1-B)
- C41 pad 2: (no net) -> GND
- C43 pad 1: (no net) -> +5V
- C43 pad 2: (no net) -> GND
- C44 pad 1: (no net) -> /Video and audio out/DAC_5V
- C44 pad 2: (no net) -> GNDA
- C45 pad 1: (no net) -> /Video and audio out/LAD7
- C45 pad 2: (no net) -> GNDA
- C46 pad 1: (no net) -> /Video and audio out/LAD7
- C46 pad 2: (no net) -> /Video and audio out/AUDIO
- C47 pad 1: (no net) -> +3V3
- C47 pad 2: (no net) -> GND
- C5 pad 1: (no net) -> +5V
- C5 pad 2: (no net) -> GND
- C6 pad 1: (no net) -> +5V
- C6 pad 2: (no net) -> GND
- C7 pad 1: (no net) -> +5V
- C7 pad 2: (no net) -> GND
- C8 pad 1: (no net) -> +5V
- C8 pad 2: (no net) -> GND
- C9 pad 1: (no net) -> +5V
- C9 pad 2: (no net) -> GND
- D1 pad 1: (no net) -> /Shared port/RXCLK
- D1 pad 2: (no net) -> /Shared port/KBD_CLK
- D10 pad 1: (no net) -> VIDEN
- D10 pad 2: (no net) -> Net-(D10-A)
- D11 pad 1: (no net) -> VIDEN
- D11 pad 2: (no net) -> Net-(D11-A)
- D12 pad 1: (no net) -> Net-(D12-K)
- D12 pad 2: (no net) -> Net-(D12-A)
- D13 pad 1: (no net) -> /Video and audio out/VGA_R
- D13 pad 2: (no net) -> Net-(D12-K)
- D14 pad 1: (no net) -> Net-(D14-K)
- D14 pad 2: (no net) -> Net-(D10-A)
- D15 pad 1: (no net) -> /Video and audio out/VGA_G
- D15 pad 2: (no net) -> Net-(D14-K)
- D16 pad 1: (no net) -> Net-(D16-K)
- D16 pad 2: (no net) -> Net-(D11-A)
- D17 pad 1: (no net) -> /Video and audio out/VGA_B
- D17 pad 2: (no net) -> Net-(D16-K)
- D18 pad 1: (no net) -> GND
- D18 pad 2: (no net) -> Net-(D18-A)
- D19 pad 1: (no net) -> /Shared port/PS2_INH
- D19 pad 2: (no net) -> /Shared port/KBD_CLK
- D2 pad 1: (no net) -> /Shared port/P_CS
- D2 pad 2: (no net) -> /Shared port/MOUS_CLK
- D3 pad 1: (no net) -> /Shared port/P_PS2D
- D3 pad 2: (no net) -> /Shared port/PS2_DATA
- D4 pad 1: (no net) -> /Shared port/RXCLK
- D4 pad 2: (no net) -> /Shared port/MOUS_CLK
- D5 pad 1: (no net) -> /Shared port/PS2_INH
- D5 pad 2: (no net) -> /Shared port/MOUS_CLK
- D6 pad 1: (no net) -> /Shared port/K0
- D6 pad 2: (no net) -> /Shared port/KBD_CLK
- D7 pad 1: (no net) -> Net-(D7-K)
- D7 pad 2: (no net) -> GND
- D8 pad 1: (no net) -> Net-(D8-K)
- D8 pad 2: (no net) -> GND
- D9 pad 1: (no net) -> VIDEN
- D9 pad 2: (no net) -> Net-(D12-A)
- F1 pad 1: (no net) -> Net-(F1-Pad1)
- F1 pad 2: (no net) -> Net-(D7-K)
- J10 pad A1: (no net) -> GND
- J10 pad A10: (no net) -> SRC4
- J10 pad A11: (no net) -> SRC6
- J10 pad A12: (no net) -> GND
- J10 pad A13: (no net) -> A0
- J10 pad A14: (no net) -> A2
- J10 pad A15: (no net) -> A4
- J10 pad A16: (no net) -> A6
- J10 pad A17: (no net) -> ~{EXP2}
- J10 pad A18: (no net) -> RW
- J10 pad A19: (no net) -> ~{WE}
- J10 pad A2: (no net) -> +5V
- J10 pad A20: (no net) -> GND
- J10 pad A3: (no net) -> D0
- J10 pad A4: (no net) -> D2
- J10 pad A5: (no net) -> D4
- J10 pad A6: (no net) -> D6
- J10 pad A7: (no net) -> GND
- J10 pad A8: (no net) -> SRC0
- J10 pad A9: (no net) -> SRC2
- J10 pad B1: (no net) -> GND
- J10 pad B10: (no net) -> SRC5
- J10 pad B11: (no net) -> SRC7
- J10 pad B12: (no net) -> CLK
- J10 pad B13: (no net) -> A1
- J10 pad B14: (no net) -> A3
- J10 pad B15: (no net) -> A5
- J10 pad B16: (no net) -> A7
- J10 pad B17: (no net) -> Net-(J10-SEL)
- J10 pad B18: (no net) -> ~{LOAD_IMM}
- J10 pad B19: (no net) -> RUN
- J10 pad B2: (no net) -> +5V
- J10 pad B20: (no net) -> GND
- J10 pad B3: (no net) -> D1
- J10 pad B4: (no net) -> D3
- J10 pad B5: (no net) -> D5
- J10 pad B6: (no net) -> D7
- J10 pad B7: (no net) -> GND
- J10 pad B8: (no net) -> SRC1
- J10 pad B9: (no net) -> SRC3
- J11 pad A1: (no net) -> GND
- J11 pad A10: (no net) -> SRC4
- J11 pad A11: (no net) -> SRC6
- J11 pad A12: (no net) -> GND
- J11 pad A13: (no net) -> A0
- J11 pad A14: (no net) -> A2
- J11 pad A15: (no net) -> A4
- J11 pad A16: (no net) -> A6
- J11 pad A17: (no net) -> ~{EXP1}
- J11 pad A18: (no net) -> RW
- J11 pad A19: (no net) -> ~{WE}
- J11 pad A2: (no net) -> +5V
- J11 pad A20: (no net) -> GND
- J11 pad A3: (no net) -> D0
- J11 pad A4: (no net) -> D2
- J11 pad A5: (no net) -> D4
- J11 pad A6: (no net) -> D6
- J11 pad A7: (no net) -> GND
- J11 pad A8: (no net) -> SRC0
- J11 pad A9: (no net) -> SRC2
- J11 pad B1: (no net) -> GND
- J11 pad B10: (no net) -> SRC5
- J11 pad B11: (no net) -> SRC7
- J11 pad B12: (no net) -> CLK
- J11 pad B13: (no net) -> A1
- J11 pad B14: (no net) -> A3
- J11 pad B15: (no net) -> A5
- J11 pad B16: (no net) -> A7
- J11 pad B17: (no net) -> Net-(J11-SEL)
- J11 pad B18: (no net) -> ~{LOAD_IMM}
- J11 pad B19: (no net) -> RUN
- J11 pad B2: (no net) -> +5V
- J11 pad B20: (no net) -> GND
- J11 pad B3: (no net) -> D1
- J11 pad B4: (no net) -> D3
- J11 pad B5: (no net) -> D5
- J11 pad B6: (no net) -> D7
- J11 pad B7: (no net) -> GND
- J11 pad B8: (no net) -> SRC1
- J11 pad B9: (no net) -> SRC3
- J12 pad A1: (no net) -> GND
- J12 pad A10: (no net) -> SRC4
- J12 pad A11: (no net) -> SRC6
- J12 pad A12: (no net) -> GND
- J12 pad A13: (no net) -> A0
- J12 pad A14: (no net) -> A2
- J12 pad A15: (no net) -> A4
- J12 pad A16: (no net) -> A6
- J12 pad A17: (no net) -> ~{EXP2}
- J12 pad A18: (no net) -> RW
- J12 pad A19: (no net) -> ~{WE}
- J12 pad A2: (no net) -> +5V
- J12 pad A20: (no net) -> GND
- J12 pad A3: (no net) -> D0
- J12 pad A4: (no net) -> D2
- J12 pad A5: (no net) -> D4
- J12 pad A6: (no net) -> D6
- J12 pad A7: (no net) -> GND
- J12 pad A8: (no net) -> SRC0
- J12 pad A9: (no net) -> SRC2
- J12 pad B1: (no net) -> GND
- J12 pad B10: (no net) -> SRC5
- J12 pad B11: (no net) -> SRC7
- J12 pad B12: (no net) -> CLK
- J12 pad B13: (no net) -> A1
- J12 pad B14: (no net) -> A3
- J12 pad B15: (no net) -> A5
- J12 pad B16: (no net) -> A7
- J12 pad B17: (no net) -> Net-(J12-SEL)
- J12 pad B18: (no net) -> ~{LOAD_IMM}
- J12 pad B19: (no net) -> RUN
- J12 pad B2: (no net) -> +5V
- J12 pad B20: (no net) -> GND
- J12 pad B3: (no net) -> D1
- J12 pad B4: (no net) -> D3
- J12 pad B5: (no net) -> D5
- J12 pad B6: (no net) -> D7
- J12 pad B7: (no net) -> GND
- J12 pad B8: (no net) -> SRC1
- J12 pad B9: (no net) -> SRC3
- J13 pad A12: (no net) -> GND
- J13 pad A5: (no net) -> Net-(J13-CC1)
- J13 pad A9: (no net) -> Net-(F1-Pad1)
- J13 pad B12: (no net) -> GND
- J13 pad B5: (no net) -> Net-(J13-CC2)
- J13 pad B9: (no net) -> Net-(F1-Pad1)
- J13 pad S1: (no net) -> GND
- J2 pad 1: (no net) -> +5V
- J2 pad 2: (no net) -> /Shared port/P_SCK
- J2 pad 3: (no net) -> /Shared port/P_MOSI
- J2 pad 4: (no net) -> /Shared port/PAD1_DATA
- J2 pad 5: (no net) -> unconnected-(J2-nc-Pad5)
- J2 pad 6: (no net) -> unconnected-(J2-nc-Pad6)
- J2 pad 7: (no net) -> GND
- J3 pad 1: (no net) -> +5V
- J3 pad 2: (no net) -> /Shared port/P_SCK
- J3 pad 3: (no net) -> /Shared port/P_MOSI
- J3 pad 4: (no net) -> /Shared port/PAD2_DATA
- J3 pad 5: (no net) -> unconnected-(J3-nc-Pad5)
- J3 pad 6: (no net) -> unconnected-(J3-nc-Pad6)
- J3 pad 7: (no net) -> GND
- J4 pad 1: (no net) -> Net-(J4-CD/DAT3)
- J4 pad 10: (no net) -> unconnected-(J4-CARD_DETECT-Pad10)
- J4 pad 11: (no net) -> unconnected-(J4-WRITE_PROTECT-Pad11)
- J4 pad 12: (no net) -> GND
- J4 pad 13: (no net) -> GND
- J4 pad 2: (no net) -> Net-(J4-CMD)
- J4 pad 3: (no net) -> GND
- J4 pad 4: (no net) -> +3V3
- J4 pad 5: (no net) -> Net-(J4-CLK)
- J4 pad 6: (no net) -> GND
- J4 pad 7: (no net) -> /Shared port/SD_MISO
- J4 pad 8: (no net) -> unconnected-(J4-DAT1-Pad8)
- J4 pad 9: (no net) -> unconnected-(J4-DAT2-Pad9)
- J5 pad A1: (no net) -> /Shared port/PS2_DATA
- J5 pad A2: (no net) -> unconnected-(J5-nc-PadA2)
- J5 pad A3: (no net) -> GND
- J5 pad A4: (no net) -> +5V
- J5 pad A5: (no net) -> /Shared port/MOUS_CLK
- J5 pad A6: (no net) -> unconnected-(J5-nc-PadA6)
- J5 pad B1: (no net) -> /Shared port/PS2_DATA
- J5 pad B2: (no net) -> unconnected-(J5-nc-PadB2)
- J5 pad B3: (no net) -> GND
- J5 pad B4: (no net) -> +5V
- J5 pad B5: (no net) -> /Shared port/KBD_CLK
- J5 pad B6: (no net) -> unconnected-(J5-nc-PadB6)
- J5 pad SH: (no net) -> GND
- J6 pad R1: (no net) -> /Video and audio out/AUDIO
- J6 pad R2: (no net) -> GNDA
- J6 pad S: (no net) -> GNDA
- J6 pad T: (no net) -> /Video and audio out/AUDIO
- J7 pad 0: (no net) -> GND
- J7 pad 1: (no net) -> /Video and audio out/VGA_R
- J7 pad 10: (no net) -> GND
- J7 pad 11: (no net) -> unconnected-(J7-Pad11)
- J7 pad 12: (no net) -> unconnected-(J7-Pad12)
- J7 pad 13: (no net) -> ~{HSYNC}
- J7 pad 14: (no net) -> ~{VSYNC}
- J7 pad 15: (no net) -> unconnected-(J7-Pad15)
- J7 pad 2: (no net) -> /Video and audio out/VGA_G
- J7 pad 3: (no net) -> /Video and audio out/VGA_B
- J7 pad 4: (no net) -> unconnected-(J7-Pad4)
- J7 pad 5: (no net) -> GND
- J7 pad 6: (no net) -> GND
- J7 pad 7: (no net) -> GND
- J7 pad 8: (no net) -> GND
- J7 pad 9: (no net) -> unconnected-(J7-Pad9)
- J8 pad A1: (no net) -> GND
- J8 pad A10: (no net) -> A14
- J8 pad A11: (no net) -> GND
- J8 pad A12: (no net) -> D0
- J8 pad A13: (no net) -> D2
- J8 pad A14: (no net) -> D4
- J8 pad A15: (no net) -> D6
- J8 pad A16: (no net) -> A15
- J8 pad A17: (no net) -> Net-(J8-/ROM_OE)
- J8 pad A18: (no net) -> PIXEL_ENABLE
- J8 pad A19: (no net) -> RUN
- J8 pad A2: (no net) -> +5V
- J8 pad A20: (no net) -> CLK
- J8 pad A21: (no net) -> GND
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Routing:
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- added copper zone on In2.Cu, net +5V
- added copper zone on In1.Cu, net GND
Other:
- board size 290 x 290 mm -> 290 x 215 mm
- board text added: "25.175 MHz"
- board text added: "AC Buffer"
- board text added: "AC Register"
- board text added: "ALU High"
- board text added: "ALU Low"
- board text added: "Audio Driver"
- board text added: "Audio Enable"
- board text added: "Audio R-2R DAC"
- board text added: "Bank Selector"
- board text added: "Blue"
- board text added: "Branch Handler"
- board text added: "Cartridge ROM"
- board text added: "Color Decoder"
- board text added: "D Buffer"
- board text added: "D Register"
- board text added: "Green"
- board text added: "H Counter"
- board text added: "I/O Decoder"
- board text added: "Inst Register"
- board text added: "Line Readback"
- board text added: "Memory Control"
- board text added: "Pixel Register"
- board text added: "Port Driver"
- board text added: "Port Receiver"
- board text added: "Program Counter High"
- board text added: "Program Counter Low"
- board text added: "Quad 4:1 Mux"
- board text added: "RAM High"
- board text added: "RAM Low"
- board text added: "Red"
- board text added: "Slot 1"
- board text added: "Slot 2"
- board text added: "Slot 3"
- board text added: "Slot 4"
- board text added: "State Machine"
- board text added: "V Counter"
- board text added: "Video Mode"
- board text added: "Video Sync"
- board text added: "X Register"
- board text added: "Y Register"
