File: kicad/placard.kicad_pcb (KiCad board)
At the start: 4 copper layers, 290 x 215 mm, 183 parts, among them J10 Slot 2, J11 Slot 3, J12 Slot 4, J13 USB4125-GF-A, J2 SNES pad, J3 SNES pad, J4 SD (SPI), J5 PS/2 kbd + mouse, J6 3.5 mm, J7 VGA, J8 Molex 87715-9106, J9 Slot 1, K1 G5LE-1 DC5, SW1 ANT11TFHQE, SW2 PTS645VL58-2 LFS, U1 ATF22V10C-7PX, U10 ATF22V10C-7PX, U11 ATF22V10C-7PX, U12 ATF22V10C-7PX, U13 ATF22V10C-7PX, U14 ATF22V10C-7PX, U15 ATF22V10C-7PX, U16 ATF22V10C-7PX, U17 ATF22V10C-7PX, U18 SN74F377AN, U19 SN74F377AN, U2 ATF22V10C-7PX, U20 SN74F377AN, U21 SN74F377AN, U22 SN74F377AN, U23 CD74HCT377E, U25 CD74ACT273E, U26 SN74F541N, U27 SN74F541N, U29 SN74F541N, U3 ATF22V10C-7PX, U31 AS7C256C-15PCN, U32 AS7C256C-15PCN, U35 ATF22V10C-7PX, U36 SN74HCT574N, U38 ATF22V10C-7PX, U4 ATF22V10C-7PX, U40 MCP1700-3302E/TO, U42 ATF22V10C-7PX, U5 ATF22V10C-7PX, U6 ATF22V10C-7PX, U7 ATF22V10C-7PX, U8 ATF22V10C-7PX, U9 ATF22V10C-7PX, X1 25.175 MHz

Commit message: Main board: 5 mm corner radius, concentric with the corner mounting holes
Edge.Cuts arcs 3 -> 5 mm (centres at the H1-H4 M3 hole centres, 5 mm in
from each edge, so the pads keep 1.8 mm to the edge all round). In1 GND /
In2 +5V zone outlines chamfered to match so they stay inside the board.
Board note corrected to 290 x 215 mm. gen_kicad_pcb.py radius updated.

Co-Authored-By: Claude Opus 5.5 (1M context) <noreply@anthropic.com>
Claude-Session: https://claude.ai/code/session_01Kqq4hXKDNbPYn2hxTugYn8
Other:
- outline, holes or cut-outs redrawn
- board text added: "PLACARD main board: 4 layers (In1 GND, In2 +5V), 1.6 mm, 290 x 215 mm, 5 mm corner radius"
- board text removed: "PLACARD main board: 4 layers (In1 GND, In2 +5V), 1.6 mm, 290 x 290 mm, 3 mm corner radius"
Changed lines of the file:
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@@
 	)
 	(gr_line
-		(start 337 265)
-		(end 53 265)
+		(start 335 265)
+		(end 55 265)
 		(stroke
 			(width 0.1)
@@
 	)
 	(gr_line
-		(start 53 50)
-		(end 337 50)
+		(start 55 50)
+		(end 335 50)
 		(stroke
 			(width 0.1)
@@
 	)
 	(gr_arc
-		(start 53 265)
-		(mid 50.87868 264.12132)
-		(end 50 262)
+		(start 55 265)
+		(mid 51.464466 263.535534)
+		(end 50 260)
 		(stroke
 			(width 0.1)
@@
 	)
 	(gr_arc
-		(start 50 53)
-		(mid 50.87868 50.87868)
-		(end 53 50)
+		(start 50 55)
+		(mid 51.464466 51.464466)
+		(end 55 50)
 		(stroke
 			(width 0.1)
@@
 	)
 	(gr_arc
-		(start 340 262)
-		(mid 339.12132 264.12132)
-		(end 337 265)
+		(start 340 260)
+		(mid 338.535534 263.535534)
+		(end 335 265)
 		(stroke
 			(width 0.1)
@@
 	)
 	(gr_line
-		(start 50 262)
-		(end 50 53)
+		(start 50 260)
+		(end 50 55)
 		(stroke
 			(width 0.1)
@@
 	)
 	(gr_line
-		(start 340 53)
-		(end 340 262)
+		(start 340 55)
+		(end 340 260)
 		(stroke
 			(width 0.1)
@@
 	)
 	(gr_arc
-		(start 337 50)
-		(mid 339.12132 50.87868)
-		(end 340 53)
+		(start 335 50)
+		(mid 338.535534 51.464466)
+		(end 340 55)
 		(stroke
 			(width 0.1)
@@
 		)
 	)
-	(gr_text "PLACARD main board: 4 layers (In1 GND, In2 +5V), 1.6 mm, 290 x 290 mm, 3 mm corner radius"
+	(gr_text "PLACARD main board: 4 layers (In1 GND, In2 +5V), 1.6 mm, 290 x 215 mm, 5 mm corner radius"
 		(at 54 329 0)
 		(layer "Cmts.User")
@@
 		(polygon
 			(pts
-				(xy 53 50) (xy 337 50) (xy 340 53) (xy 340 262) (xy 337 265) (xy 53 265) (xy 50 262) (xy 50 53)
+				(xy 55 50) (xy 335 50) (xy 340 55) (xy 340 260) (xy 335 265) (xy 55 265) (xy 50 260) (xy 50 55)
 			)
 		)
@@
 		(polygon
 			(pts
-				(xy 53 50) (xy 337 50) (xy 340 53) (xy 340 262) (xy 337 265) (xy 53 265) (xy 50 262) (xy 50 53)
+				(xy 55 50) (xy 335 50) (xy 340 55) (xy 340 260) (xy 335 265) (xy 55 265) (xy 50 260) (xy 50 55)
 			)
 		)
