File: kicad/data_bus.kicad_sch (KiCad schematic)
At the start: 15 parts, among them U18 SN74F377AN, U26 SN74F541N, U27 SN74F541N

Commit message: BOM/schematic: stocked substitutes from the first parts order
D18 Kingbright WP7113ID (LTL2R3KRD-EM out of stock), 100n TDK
FG28X7R1H104KNT00 (KEMET C320C104 $0.66 at Mouser), C45 TDK
FG24C0G1H153JNT06 (KEMET non-stocked), Vishay BAT85S-TAP and
1N4148-TAP, MF-RG300-0, USB4125-GF-A-0190; Mouser prices re-checked.

Co-Authored-By: Claude Opus 5.5 (1M context) <noreply@anthropic.com>
Claude-Session: https://claude.ai/code/session_017y5UgjExE8oeP7QrfvhCzb
Parts:
- C18, C26, C27: MPN C320C104K5R5TA -> FG28X7R1H104KNT00; Manufacturer KEMET -> TDK

Commit message: Schematic: expansion slot contacts A8-B11 become BT1-BT8 (slot-1 boot)
Cards latch D7:D0, so the slots no longer carry SRC7:SRC0.  Slot 1's
BT1-BT5 carry STALL_IN, STALL_OUT, PC_ENABLE, PIXEL_ENABLE and /CART;
BT6-BT8 and slots 2-4's boot contacts are not connected
(EXPANSION.md, "Booting from slot 1").  Slots respaced to keep the labels
on the page.

Co-Authored-By: Claude Opus 5.5 (1M context) <noreply@anthropic.com>
Claude-Session: https://claude.ai/code/session_016q7L8WUy2bLsrwHss8WZwY
Changed lines of the file:
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@@
   (bus (pts (xy 313.69 163.83) (xy 313.69 162.56)) (stroke (width 0) (type default)))
   (bus (pts (xy 320.04 162.56) (xy 322.58 162.56)) (stroke (width 0) (type default)))
-  (global_label "SRC[0..7]" (shape bidirectional) (at 322.58 162.56 0) (fields_autoplaced) (effects (font (size 2 2)) (justify left)) (property "Intersheetrefs" "${INTERSHEET_REFS}" (at 322.58 162.56 0) (effects (font (size 2 2)) (justify left) hide)))
+  (label "SRC[0..7]" (at 322.58 162.56 0) (fields_autoplaced) (effects (font (size 2 2)) (justify left bottom)))
   (bus (pts (xy 134.62 189.23) (xy 132.08 189.23)) (stroke (width 0) (type default)))
   (junction (at 134.62 189.23) (diameter 0) (color 0 0 0 0))

Commit message: Put every symbol, footprint and 3D model in the project library
- gen_kicad_stock_footprints.py: copies of the KiCad 9.0.6 footprints the
  boards use (C_Disc, CP_Radial, DO-15/DO-35, LED, pin header, oscillator,
  TO-92, SIP9, mounting holes, net tie) into placard.pretty, and KiCad's
  STEP models for them and for the DIP socket / resistor kit footprints
  into placard.3dshapes
- model paths use the PLACARD_LIB text variable (main board
  ${KIPRJMOD}/lib, cartridges ${KIPRJMOD}/../lib) so the shared footprints
  find their models in all three projects
- placard_std gains the 28C256 EEPROM and the power symbols; symbol
  Footprint defaults name placard footprints (relay, SIP9, oscillator,
  TO-92, EEPROM socket)
- schematics regenerated with placard_std power/EEPROM symbols and
  placard: footprints; BOM CSVs and PDFs regenerated
- cartridge .kicad_pro files take in Justin's local KiCad 9 settings

Co-Authored-By: Claude Opus 5.5 <noreply@anthropic.com>
Claude-Session: https://claude.ai/code/session_017okF1JiLRNFTfH7Az85hff
Parts:
- C18, C26, C27: footprint Capacitor_THT:C_Disc_D5.0mm_W2.5mm_P5.00mm -> placard:C_Disc_D5.0mm_W2.5mm_P5.00mm
- RN1: footprint Resistor_THT:R_Array_SIP9 -> placard:R_Array_SIP9

Commit message: Schematic: rename buses to ADDR / DATABUS / D, wire the shared port outputs
- Address bus A15:A0 is now ADDR15:ADDR0, the data bus D7:D0 is DATABUS7:DATABUS0
  and the D register's outputs DR7:DR0 are D7:D0 (main board and both cartridges).
- Shared port sheet: U38's outputs P_SCK, P_MOSI, P_CS, P_PS2D and K0 are wired
  to the SNES pads, the SD dividers and the PS/2 hold diodes (K0 -> D6 ->
  keyboard CLK).  J3 now sits level with U38's SCK/MOSI pins, J2 above it.
- Parts moved so the longer labels fit: U3/U4 and the PC bus, U18, U22, U11,
  U31, U32, RN1, R5-R12; expansion slots in two rows.
- SCHEMATIC_PLAN.md: the bus names.

Co-Authored-By: Claude Opus 5.5 <noreply@anthropic.com>
Claude-Session: https://claude.ai/code/session_01DnW5SUv7E4nz9tGtPvD1qV
Connections:
- net DR0 is gone; now on net D0: U18.2 (Q0), U26.2 (A0)
- net DR1 is gone; now on net D1: U18.5 (Q1), U26.3 (A1)
- net DR2 is gone; now on net D2: U18.6 (Q2), U26.4 (A2)
- net DR3 is gone; now on net D3: U18.9 (Q3), U26.5 (A3)
- net DR4 is gone; now on net D4: U18.12 (Q4), U26.6 (A4)
- net DR5 is gone; now on net D5: U18.15 (Q5), U26.7 (A5)
- net DR6 is gone; now on net D6: U18.16 (Q6), U26.8 (A6)
- net DR7 is gone; now on net D7: U18.19 (Q7), U26.9 (A7)
- net D0: no longer R5.1, RN1.2 (R1), U18.3 (D0)
- net D1: no longer R6.1, RN1.3 (R2), U18.4 (D1)
- net D2: no longer R7.1, RN1.4 (R3), U18.7 (D2)
- net D3: no longer R8.1, RN1.5 (R4), U18.8 (D3)
- net D4: no longer R9.1, RN1.6 (R5), U18.13 (D4)
- net D5: no longer R10.1, RN1.7 (R6), U18.14 (D5)
- net D6: no longer R11.1, RN1.8 (R7), U18.17 (D6)
- net D7: no longer R12.1, RN1.9 (R8), U18.18 (D7)
- new net DATABUS0: R5.1, RN1.2 (R1), U18.3 (D0)
- new net DATABUS1: R6.1, RN1.3 (R2), U18.4 (D1)
- new net DATABUS2: R7.1, RN1.4 (R3), U18.7 (D2)
- new net DATABUS3: R8.1, RN1.5 (R4), U18.8 (D3)
- new net DATABUS4: R9.1, RN1.6 (R5), U18.13 (D4)
- new net DATABUS5: R10.1, RN1.7 (R6), U18.14 (D5)
- new net DATABUS6: R11.1, RN1.8 (R7), U18.17 (D6)
- new net DATABUS7: R12.1, RN1.9 (R8), U18.18 (D7)
Other:
- note added: "RN1: DATABUS7:0 read FFh when nothing drives it"
- note removed: "RN1: D7:D0 read FFh when nothing drives them"
- moved on the sheet: C18, R10, R11, R12, R5, R6, R7, R8, R9, RN1, U18
