File: kicad/pc_mux.kicad_sch (KiCad schematic)
At the start: 12 parts, among them U10 ATF22V10C-7PX, U3 ATF22V10C-7PX, U4 ATF22V10C-7PX, U7 ATF22V10C-7PX, U8 ATF22V10C-7PX, U9 ATF22V10C-7PX

Commit message: BOM/schematic: stocked substitutes from the first parts order
D18 Kingbright WP7113ID (LTL2R3KRD-EM out of stock), 100n TDK
FG28X7R1H104KNT00 (KEMET C320C104 $0.66 at Mouser), C45 TDK
FG24C0G1H153JNT06 (KEMET non-stocked), Vishay BAT85S-TAP and
1N4148-TAP, MF-RG300-0, USB4125-GF-A-0190; Mouser prices re-checked.

Co-Authored-By: Claude Opus 5.5 (1M context) <noreply@anthropic.com>
Claude-Session: https://claude.ai/code/session_017y5UgjExE8oeP7QrfvhCzb
Parts:
- C10, C3, C4, C7, C8, C9: MPN C320C104K5R5TA -> FG28X7R1H104KNT00; Manufacturer KEMET -> TDK

Commit message: Put every symbol, footprint and 3D model in the project library
- gen_kicad_stock_footprints.py: copies of the KiCad 9.0.6 footprints the
  boards use (C_Disc, CP_Radial, DO-15/DO-35, LED, pin header, oscillator,
  TO-92, SIP9, mounting holes, net tie) into placard.pretty, and KiCad's
  STEP models for them and for the DIP socket / resistor kit footprints
  into placard.3dshapes
- model paths use the PLACARD_LIB text variable (main board
  ${KIPRJMOD}/lib, cartridges ${KIPRJMOD}/../lib) so the shared footprints
  find their models in all three projects
- placard_std gains the 28C256 EEPROM and the power symbols; symbol
  Footprint defaults name placard footprints (relay, SIP9, oscillator,
  TO-92, EEPROM socket)
- schematics regenerated with placard_std power/EEPROM symbols and
  placard: footprints; BOM CSVs and PDFs regenerated
- cartridge .kicad_pro files take in Justin's local KiCad 9 settings

Co-Authored-By: Claude Opus 5.5 <noreply@anthropic.com>
Claude-Session: https://claude.ai/code/session_017okF1JiLRNFTfH7Az85hff
Parts:
- C10, C3, C4, C7, C8, C9: footprint Capacitor_THT:C_Disc_D5.0mm_W2.5mm_P5.00mm -> placard:C_Disc_D5.0mm_W2.5mm_P5.00mm

Commit message: Schematic: rename buses to ADDR / DATABUS / D, wire the shared port outputs
- Address bus A15:A0 is now ADDR15:ADDR0, the data bus D7:D0 is DATABUS7:DATABUS0
  and the D register's outputs DR7:DR0 are D7:D0 (main board and both cartridges).
- Shared port sheet: U38's outputs P_SCK, P_MOSI, P_CS, P_PS2D and K0 are wired
  to the SNES pads, the SD dividers and the PS/2 hold diodes (K0 -> D6 ->
  keyboard CLK).  J3 now sits level with U38's SCK/MOSI pins, J2 above it.
- Parts moved so the longer labels fit: U3/U4 and the PC bus, U18, U22, U11,
  U31, U32, RN1, R5-R12; expansion slots in two rows.
- SCHEMATIC_PLAN.md: the bus names.

Co-Authored-By: Claude Opus 5.5 <noreply@anthropic.com>
Claude-Session: https://claude.ai/code/session_01DnW5SUv7E4nz9tGtPvD1qV
Connections:
- net DR0 is gone; now on net D0: U7.1 (A0)
- net DR1 is gone; now on net D1: U7.5 (A1)
- net DR2 is gone; now on net D2: U7.11 (A2)
- net DR3 is gone; now on net D3: U7.16 (A3)
- net DR4 is gone; now on net D4: U8.1 (A0)
- net DR5 is gone; now on net D5: U8.5 (A1)
- net DR6 is gone; now on net D6: U8.11 (A2)
- net DR7 is gone; now on net D7: U8.16 (A3)
- net D0: no longer U3.2 (D0)
- net D1: no longer U3.3 (D1)
- net D2: no longer U3.4 (D2)
- net D3: no longer U3.5 (D3)
- net D4: no longer U3.6 (D4)
- net D5: no longer U3.7 (D5)
- net D6: no longer U3.8 (D6)
- net D7: no longer U3.9 (D7)
- net A0 renamed ADDR0
- net A1 renamed ADDR1
- net A10 renamed ADDR10
- net A11 renamed ADDR11
- net A12 renamed ADDR12
- net A13 renamed ADDR13
- net A14 renamed ADDR14
- net A15 renamed ADDR15
- net A2 renamed ADDR2
- net A3 renamed ADDR3
- net A4 renamed ADDR4
- net A5 renamed ADDR5
- net A6 renamed ADDR6
- net A7 renamed ADDR7
- net A8 renamed ADDR8
- net A9 renamed ADDR9
- new net DATABUS0: U3.2 (D0)
- new net DATABUS1: U3.3 (D1)
- new net DATABUS2: U3.4 (D2)
- new net DATABUS3: U3.5 (D3)
- new net DATABUS4: U3.6 (D4)
- new net DATABUS5: U3.7 (D5)
- new net DATABUS6: U3.8 (D6)
- new net DATABUS7: U3.9 (D7)
Other:
- note added: "Video address: VA0, VA1, VA7, VA8 from the audio slot PLD (line repeat), ADDR6:2 = V6:V2, ADDR15:9 = H9:H3."
- note removed: "Video address: VA0, VA1, VA7, VA8 from the audio slot PLD (line repeat), A6:A2 = V6:V2, A15:A9 = H9:H3."
- moved on the sheet: C3, C4, U3, U4

Commit message: Option B: muxes take the enables as selects, /WE from an early clock tap
Removes the Sync PLD pass from every memory address (docs/FETCH_TIMING.md):
the instruction fetch gains 8.2 ns, X/Y/video/upper-32K reads 9.7 ns, the
zero-page store start 6.9 ns, and the address hold after /WE is +0.5 ns
from the datasheets alone.  No new parts, no extra clock, no PLCC.

- ATF22V10_QUAD_MUX.pld rev 02: two low + two high address bits per chip,
  PIXEL_ENABLE / PC_ENABLE / X_ENABLE / Y_ENABLE as the selects
- ATF22V10_SYNC.pld rev 10: ADDR_SEL outputs gone; /WE on pin 20 from the
  early clock tap CLK_E (pin 9), RW and RUN inputs, OE = RUN
- ATF22V10_MEM_CTRL.pld rev 10: /WE gone (pin 16 free)
- ATF22V10_IO_DECODE.pld rev 05: /CE_HI from the enables, RW dropped
- FPGA model and benches follow; GHDL: tb_cart_load (2 seeds), tb_top_load,
  tb_blank_line pass, and cpu_test makes the same 69,776 RAM writes as main
- Schematic: mux sheet rewired, /WE from U15, net tie NT2 between CLK_E and
  CLK on the power sheet (the 500 mm of track), symbols regenerated, PDFs
- Docs updated; docs/option_b_board.png shows the board rewiring (no chip
  has to move)

Co-Authored-By: Claude Fable 5.1 <noreply@anthropic.com>
Claude-Session: https://claude.ai/code/session_01DnW5SSBUc8XDbr4GrYdwj8
Parts:
- U10: Function Address mux 15:12 -> Address mux 7:6, 15:14
- U7: Function Address mux 3:0 -> Address mux 1:0, 9:8
- U8: Function Address mux 7:4 -> Address mux 3:2, 11:10
- U9: Function Address mux 11:8 -> Address mux 5:4, 13:12
Connections:
- net ADDR10: now also U8.22 (HI0); no longer U9.22 (Y2)
- net ADDR11: now also U8.23 (HI1); no longer U9.23 (Y3)
- net ADDR12: now also U9.22 (HI0); no longer U10.20 (Y0)
- net ADDR13: now also U9.23 (HI1); no longer U10.21 (Y1)
- net ADDR2: now also U8.20 (LO0); no longer U7.22 (Y2)
- net ADDR3: now also U8.21 (LO1); no longer U7.23 (Y3)
- net ADDR4: now also U9.20 (LO0); no longer U8.20 (Y0)
- net ADDR5: now also U9.21 (LO1); no longer U8.21 (Y1)
- net ADDR6: now also U10.20 (LO0); no longer U8.22 (Y2)
- net ADDR7: now also U10.21 (LO1); no longer U8.23 (Y3)
- net ADDR8: now also U7.22 (HI0); no longer U9.20 (Y0)
- net ADDR9: now also U7.23 (HI1); no longer U9.21 (Y1)
- net D0: now also U7.5 (D0); no longer U7.1 (A0)
- net D1: now also U7.9 (D1); no longer U7.5 (A1)
- net D2: now also U8.5 (D0); no longer U7.11 (A2)
- net D3: now also U8.9 (D1); no longer U7.16 (A3)
- net D4: now also U9.5 (D0); no longer U8.1 (A0)
- net D5: now also U9.9 (D1); no longer U8.5 (A1)
- net D6: now also U10.5 (D0); no longer U8.11 (A2)
- net D7: now also U10.9 (D1); no longer U8.16 (A3)
- net GND: no longer U10.1 (A0), U10.11 (A2), U10.16 (A3), U10.5 (A1), U9.1 (A0), U9.11 (A2), U9.16 (A3), U9.5 (A1)
- net H3: now also U7.18 (V3); no longer U9.7 (C1)
- net H4: now also U8.15 (V2); no longer U9.14 (C2)
- net H5: now also U8.18 (V3); no longer U9.18 (C3)
- net H6: now also U9.15 (V2); no longer U10.3 (C0)
- net H7: now also U9.18 (V3); no longer U10.7 (C1)
- net H8: now also U10.15 (V2); no longer U10.14 (C2)
- net PC0: now also U7.8 (PC0); no longer U7.4 (D0)
- net PC1: now also U7.13 (PC1); no longer U7.8 (D1)
- net PC10: now also U8.16 (PC2); no longer U9.15 (D2)
- net PC11: now also U8.19 (PC3); no longer U9.19 (D3)
- net PC12: now also U9.16 (PC2); no longer U10.4 (D0)
- net PC13: now also U9.19 (PC3); no longer U10.8 (D1)
- net PC14: now also U10.16 (PC2); no longer U10.15 (D2)
- net PC2: now also U8.8 (PC0); no longer U7.15 (D2)
- net PC3: now also U8.13 (PC1); no longer U7.19 (D3)
- net PC4: now also U9.8 (PC0); no longer U8.4 (D0)
- net PC5: now also U9.13 (PC1); no longer U8.8 (D1)
- net PC6: now also U10.8 (PC0); no longer U8.15 (D2)
- net PC7: now also U10.13 (PC1); no longer U8.19 (D3)
- net PC8: now also U7.16 (PC2); no longer U9.4 (D0)
- net PC9: now also U7.19 (PC3); no longer U9.8 (D1)
- net PC_ENABLE: now also U10.2 (PC_ENABLE), U7.2 (PC_ENABLE), U8.2 (PC_ENABLE), U9.2 (PC_ENABLE)
- net V2: now also U8.7 (V0); no longer U7.14 (C2)
- net V3: now also U8.11 (V1); no longer U7.18 (C3)
- net V4: now also U9.7 (V0); no longer U8.3 (C0)
- net V5: now also U9.11 (V1); no longer U8.7 (C1)
- net V6: now also U10.7 (V0); no longer U8.14 (C2)
- net VA0: now also U7.7 (V0); no longer U7.3 (C0)
- net VA1: now also U7.11 (V1); no longer U7.7 (C1)
- net VA7: now also U10.11 (V1); no longer U8.18 (C3)
- net VA8: now also U7.15 (V2); no longer U9.3 (C0)
- net X0: now also U7.6 (X0); no longer U7.2 (B0)
- net X1: now also U7.10 (X1); no longer U7.6 (B1)
- net X2: now also U8.6 (X0); no longer U7.13 (B2)
- net X3: now also U8.10 (X1); no longer U7.17 (B3)
- net X4: now also U9.6 (X0); no longer U8.2 (B0)
- net X5: now also U9.10 (X1); no longer U8.6 (B1)
- net X6: now also U10.6 (X0); no longer U8.13 (B2)
- net X7: now also U10.10 (X1); no longer U8.17 (B3)
- net Y0: now also U7.14 (Y2); no longer U9.2 (B0)
- net Y1: now also U7.17 (Y3); no longer U9.6 (B1)
- net Y2: now also U8.14 (Y2); no longer U9.13 (B2)
- net Y3: now also U8.17 (Y3); no longer U9.17 (B3)
- net Y4: now also U9.14 (Y2); no longer U10.2 (B0)
- net Y5: now also U9.17 (Y3); no longer U10.6 (B1)
- net Y6: now also U10.14 (Y2); no longer U10.13 (B2)
- removed net ADDR_SEL: U10.10 (S1), U7.10 (S1), U8.10 (S1), U9.10 (S1)
- removed net ADDR_SEL_HI: U10.9 (S0), U9.9 (S0)
- removed net ADDR_SEL_LO: U7.9 (S0), U8.9 (S0)
- new net PIXEL_ENABLE: U10.1 (PIXEL_ENABLE), U7.1 (PIXEL_ENABLE), U8.1 (PIXEL_ENABLE), U9.1 (PIXEL_ENABLE)
- new net X_ENABLE: U10.3 (X_ENABLE), U7.3 (X_ENABLE), U8.3 (X_ENABLE), U9.3 (X_ENABLE)
- new net Y_ENABLE: U10.4 (Y_ENABLE), U7.4 (Y_ENABLE), U8.4 (Y_ENABLE), U9.4 (Y_ENABLE)
Other:
- note added: "Each mux: two low bits (D, X, video, PC) and two high bits (0, Y, video, PC); the enables select"
- note added: "Selects: PIXEL_ENABLE (U15) = video address; else PC_ENABLE = PC; else X_ENABLE / Y_ENABLE = X / Y register; else D / 00h."
- note removed: "Mux inputs: A = D / 0, B = X / Y, C = video address, D = PC"
- moved on the sheet: C10, C7, C8, C9
