File: kicad/shared_port.kicad_sch (KiCad schematic)
At the start: 28 parts, among them J2 SNES pad, J3 SNES pad, J4 SD (SPI), J5 PS/2 kbd + mouse, U38 ATF22V10C-7PX, U42 ATF22V10C-7PX

Commit message: VGA syncs: 47 ohm series resistors R61/R62 at the PLD pins
/HSYNC (U13 pin 21) and /VSYNC (U15 pin 18) now reach J7 through R61 and
R62 (47 ohm, Yageo MFR-25FBF52-47R, sharing R5-R12's BOM line); nets after
them are /VGA_HSYNC and /VGA_VSYNC.  Symbol uuids kept; board file untouched
(pull in with Update PCB from Schematic).  R60 22k gets its MPN.

Co-Authored-By: Claude Opus 5.5 (1M context) <noreply@anthropic.com>
Claude-Session: https://claude.ai/code/session_01B4M15KLwAcnVuRUejEFj2o
Parts:
- R60: MPN (none) -> MFR-25FBF52-22K; Manufacturer (none) -> Yageo
Changed lines of the file:
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@@
   (wire (pts (xy 223.52 218.44) (xy 223.52 220.98)) (stroke (width 0) (type default)))
   (symbol (lib_id "power:GND") (at 223.52 220.98 0) (unit 1) (in_bom yes) (on_board yes) (dnp no) (property "Reference" "#PWR1012" (at 223.52 220.98 0) (effects (font (size 1.27 1.27)) hide)) (property "Value" "GND" (at 223.52 227.33 0) (effects (font (size 2 2)) hide)) (property "Footprint" "" (at 223.52 220.98 0) (effects (font (size 1.27 1.27)) hide)) (property "Datasheet" "" (at 223.52 220.98 0) (effects (font (size 1.27 1.27)) hide)) (pin "1") (instances (project "placard" (path "/e3450542-4ffc-59d4-a4a7-45636233928a/b3c80de0-82bc-5f69-87f9-71f84480d1b8" (reference "#PWR1012") (unit 1)))))
-  (symbol (lib_id "placard_std:R_US") (at 223.52 214.63 0) (unit 1) (in_bom yes) (on_board yes) (dnp no) (property "Reference" "R60" (at 225.52 213.33 0) (effects (font (size 2.54 2.54) bold) (justify left bottom))) (property "Value" "22k" (at 225.52 216.13 0) (effects (font (size 2 2)) (justify left top))) (property "Footprint" "placard:R_Axial_DIN0207_L6.3mm_D2.5mm_P10.16mm_Horizontal_Value" (at 223.52 214.63 0) (effects (font (size 1.27 1.27)) hide)) (property "Datasheet" "~" (at 223.52 214.63 0) (effects (font (size 1.27 1.27)) hide)) (property "Manufacturer" "" (at 223.52 214.63 0) (effects (font (size 1.27 1.27)) hide)) (property "MPN" "" (at 223.52 214.63 0) (effects (font (size 1.27 1.27)) hide)) (pin "1") (pin "2") (instances (project "placard" (path "/e3450542-4ffc-59d4-a4a7-45636233928a/b3c80de0-82bc-5f69-87f9-71f84480d1b8" (reference "R60") (unit 1)))))
+  (symbol (lib_id "placard_std:R_US") (at 223.52 214.63 0) (unit 1) (in_bom yes) (on_board yes) (dnp no) (property "Reference" "R60" (at 225.52 213.33 0) (effects (font (size 2.54 2.54) bold) (justify left bottom))) (property "Value" "22k" (at 225.52 216.13 0) (effects (font (size 2 2)) (justify left top))) (property "Footprint" "placard:R_Axial_DIN0207_L6.3mm_D2.5mm_P10.16mm_Horizontal_Value" (at 223.52 214.63 0) (effects (font (size 1.27 1.27)) hide)) (property "Datasheet" "~" (at 223.52 214.63 0) (effects (font (size 1.27 1.27)) hide)) (property "Manufacturer" "Yageo" (at 223.52 214.63 0) (effects (font (size 1.27 1.27)) hide)) (property "MPN" "MFR-25FBF52-22K" (at 223.52 214.63 0) (effects (font (size 1.27 1.27)) hide)) (pin "1") (pin "2") (instances (project "placard" (path "/e3450542-4ffc-59d4-a4a7-45636233928a/b3c80de0-82bc-5f69-87f9-71f84480d1b8" (reference "R60") (unit 1)))))
   (wire (pts (xy 307.34 208.28) (xy 307.34 205.74)) (stroke (width 0) (type default)))
   (symbol (lib_id "power:+5V") (at 307.34 205.74 0) (unit 1) (in_bom yes) (on_board yes) (dnp no) (property "Reference" "#PWR1013" (at 307.34 205.74 0) (effects (font (size 1.27 1.27)) hide)) (property "Value" "+5V" (at 307.34 199.39 0) (effects (font (size 2 2)))) (property "Footprint" "" (at 307.34 205.74 0) (effects (font (size 1.27 1.27)) hide)) (property "Datasheet" "" (at 307.34 205.74 0) (effects (font (size 1.27 1.27)) hide)) (pin "1") (instances (project "placard" (path "/e3450542-4ffc-59d4-a4a7-45636233928a/b3c80de0-82bc-5f69-87f9-71f84480d1b8" (reference "#PWR1013") (unit 1)))))

Commit message: BOM/schematic: stocked substitutes from the first parts order
D18 Kingbright WP7113ID (LTL2R3KRD-EM out of stock), 100n TDK
FG28X7R1H104KNT00 (KEMET C320C104 $0.66 at Mouser), C45 TDK
FG24C0G1H153JNT06 (KEMET non-stocked), Vishay BAT85S-TAP and
1N4148-TAP, MF-RG300-0, USB4125-GF-A-0190; Mouser prices re-checked.

Co-Authored-By: Claude Opus 5.5 (1M context) <noreply@anthropic.com>
Claude-Session: https://claude.ai/code/session_017y5UgjExE8oeP7QrfvhCzb
Parts:
- C38, C42: MPN C320C104K5R5TA -> FG28X7R1H104KNT00; Manufacturer KEMET -> TDK
- D1, D19, D2, D3, D4, D5, D6: MPN BAT85 -> BAT85S-TAP

Commit message: J4: Hirose DM1AA-SF-PEJ(82) replaces the obsolete Kyocera SD socket
Kyocera 145638009511859+ is obsolete (and 145638109211859+ is a
mirrored footprint, not a drop-in). KiCad's Hirose footprint copied
into placard.pretty with pads renamed to the SD_Card symbol (SW 10,
WP 11, shield 12/13), generated 3D model, BOM price from Mouser,
schematic PDFs and CASE.md J4 note updated.

Co-Authored-By: Claude Opus 5.5 (1M context) <noreply@anthropic.com>
Claude-Session: https://claude.ai/code/session_017y5UgjExE8oeP7QrfvhCzb
Parts:
- J4: footprint placard:SD_Kyocera_145638009511859+ -> placard:SD_Hirose_DM1AA_SF_PEJ82; MPN 145638009511859+ -> DM1AA-SF-PEJ(82); Manufacturer Kyocera AVX -> Hirose
Changed lines of the file:
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@@
   (wire (pts (xy 350.52 170.18) (xy 347.98 170.18)) (stroke (width 0) (type default)))
   (symbol (lib_id "power:+3V3") (at 347.98 170.18 90) (unit 1) (in_bom yes) (on_board yes) (dnp no) (property "Reference" "#PWR1021" (at 347.98 170.18 0) (effects (font (size 1.27 1.27)) hide)) (property "Value" "+3V3" (at 338.68 170.18 90) (effects (font (size 2 2)))) (property "Footprint" "" (at 347.98 170.18 0) (effects (font (size 1.27 1.27)) hide)) (property "Datasheet" "" (at 347.98 170.18 0) (effects (font (size 1.27 1.27)) hide)) (pin "1") (instances (project "placard" (path "/e3450542-4ffc-59d4-a4a7-45636233928a/b3c80de0-82bc-5f69-87f9-71f84480d1b8" (reference "#PWR1021") (unit 1)))))
-  (symbol (lib_id "placard_std:SD_Card") (at 373.38 170.18 0) (unit 1) (in_bom yes) (on_board yes) (dnp no) (property "Reference" "J4" (at 353 153 0) (effects (font (size 2.54 2.54) bold) (justify left bottom))) (property "Value" "SD (SPI)" (at 353 187 0) (effects (font (size 2 2)) (justify left top))) (property "Footprint" "placard:SD_Kyocera_145638009511859+" (at 373.38 170.18 0) (effects (font (size 1.27 1.27)) hide)) (property "Datasheet" "http://portal.fciconnect.com/Comergent//fci/drawing/10067847.pdf" (at 373.38 170.18 0) (effects (font (size 1.27 1.27)) hide)) (property "Manufacturer" "Kyocera AVX" (at 373.38 170.18 0) (effects (font (size 1.27 1.27)) hide)) (property "MPN" "145638009511859+" (at 373.38 170.18 0) (effects (font (size 1.27 1.27)) hide)) (pin "1") (pin "10") (pin "11") (pin "12") (pin "13") (pin "2") (pin "3") (pin "4") (pin "5") (pin "6") (pin "7") (pin "8") (pin "9") (instances (project "placard" (path "/e3450542-4ffc-59d4-a4a7-45636233928a/b3c80de0-82bc-5f69-87f9-71f84480d1b8" (reference "J4") (unit 1)))))
+  (symbol (lib_id "placard_std:SD_Card") (at 373.38 170.18 0) (unit 1) (in_bom yes) (on_board yes) (dnp no) (property "Reference" "J4" (at 353 153 0) (effects (font (size 2.54 2.54) bold) (justify left bottom))) (property "Value" "SD (SPI)" (at 353 187 0) (effects (font (size 2 2)) (justify left top))) (property "Footprint" "placard:SD_Hirose_DM1AA_SF_PEJ82" (at 373.38 170.18 0) (effects (font (size 1.27 1.27)) hide)) (property "Datasheet" "http://portal.fciconnect.com/Comergent//fci/drawing/10067847.pdf" (at 373.38 170.18 0) (effects (font (size 1.27 1.27)) hide)) (property "Manufacturer" "Hirose" (at 373.38 170.18 0) (effects (font (size 1.27 1.27)) hide)) (property "MPN" "DM1AA-SF-PEJ(82)" (at 373.38 170.18 0) (effects (font (size 1.27 1.27)) hide)) (pin "1") (pin "10") (pin "11") (pin "12") (pin "13") (pin "2") (pin "3") (pin "4") (pin "5") (pin "6") (pin "7") (pin "8") (pin "9") (instances (project "placard" (path "/e3450542-4ffc-59d4-a4a7-45636233928a/b3c80de0-82bc-5f69-87f9-71f84480d1b8" (reference "J4") (unit 1)))))
   (wire (pts (xy 350.52 177.8) (xy 345.44 177.8)) (stroke (width 0) (type default)))
   (wire (pts (xy 345.44 177.8) (xy 345.44 208.28)) (stroke (width 0) (type default)))

Commit message: Put every symbol, footprint and 3D model in the project library
- gen_kicad_stock_footprints.py: copies of the KiCad 9.0.6 footprints the
  boards use (C_Disc, CP_Radial, DO-15/DO-35, LED, pin header, oscillator,
  TO-92, SIP9, mounting holes, net tie) into placard.pretty, and KiCad's
  STEP models for them and for the DIP socket / resistor kit footprints
  into placard.3dshapes
- model paths use the PLACARD_LIB text variable (main board
  ${KIPRJMOD}/lib, cartridges ${KIPRJMOD}/../lib) so the shared footprints
  find their models in all three projects
- placard_std gains the 28C256 EEPROM and the power symbols; symbol
  Footprint defaults name placard footprints (relay, SIP9, oscillator,
  TO-92, EEPROM socket)
- schematics regenerated with placard_std power/EEPROM symbols and
  placard: footprints; BOM CSVs and PDFs regenerated
- cartridge .kicad_pro files take in Justin's local KiCad 9 settings

Co-Authored-By: Claude Opus 5.5 <noreply@anthropic.com>
Claude-Session: https://claude.ai/code/session_017okF1JiLRNFTfH7Az85hff
Parts:
- C38, C42: footprint Capacitor_THT:C_Disc_D5.0mm_W2.5mm_P5.00mm -> placard:C_Disc_D5.0mm_W2.5mm_P5.00mm
- D1, D19, D2, D3, D4, D5, D6: footprint Diode_THT:D_DO-35_SOD27_P7.62mm_Horizontal -> placard:D_DO-35_SOD27_P7.62mm_Horizontal

Commit message: Schematic: rename buses to ADDR / DATABUS / D, wire the shared port outputs
- Address bus A15:A0 is now ADDR15:ADDR0, the data bus D7:D0 is DATABUS7:DATABUS0
  and the D register's outputs DR7:DR0 are D7:D0 (main board and both cartridges).
- Shared port sheet: U38's outputs P_SCK, P_MOSI, P_CS, P_PS2D and K0 are wired
  to the SNES pads, the SD dividers and the PS/2 hold diodes (K0 -> D6 ->
  keyboard CLK).  J3 now sits level with U38's SCK/MOSI pins, J2 above it.
- Parts moved so the longer labels fit: U3/U4 and the PC bus, U18, U22, U11,
  U31, U32, RN1, R5-R12; expansion slots in two rows.
- SCHEMATIC_PLAN.md: the bus names.

Co-Authored-By: Claude Opus 5.5 <noreply@anthropic.com>
Claude-Session: https://claude.ai/code/session_01DnW5SUv7E4nz9tGtPvD1qV
Connections:
- net A0 renamed ADDR0
- net A1 renamed ADDR1
- net D0 renamed DATABUS0
- net D1 renamed DATABUS1
- net D2 renamed DATABUS2
- net D3 renamed DATABUS3
- net D4 renamed DATABUS4
- net D5 renamed DATABUS5
- net D6 renamed DATABUS6
- net D7 renamed DATABUS7
Other:
- moved on the sheet: J2, J3, R40, R41

Commit message: Schottkys to black 1N5817 (DO-41) so they differ from the glass 1N4148s
- D1-D6, D8-D11, D19: BAT85 -> MCC 1N5817-TP. 1N4148s (D12-D17) unchanged.
- New footprint D_DO-41_SOD81_P7.62mm_Horizontal_Pad1.6 (KiCad 9.0.6 DO-41
  at 7.62 mm, pads 1.6 mm / drill 1.0 mm): same copper as the DO-35 places,
  so Update PCB from Schematic swaps them without touching the routing;
  checked for courtyard overlaps and silk over pads on the board.
- Schematic, main PDF, BOM, BRINGUP ("Two kinds of diode"), KITTING, IO,
  VIDEO and COLORS updated.

Co-Authored-By: Claude Opus 5.5 <noreply@anthropic.com>
Claude-Session: https://claude.ai/code/session_01DnW5STXEXm5h75y8sthpiM
Parts:
- D1, D19, D2, D3, D4, D5, D6: value BAT85 -> 1N5817; footprint placard:D_DO-35_SOD27_P7.62mm_Horizontal -> placard:D_DO-41_SOD81_P7.62mm_Horizontal_Pad1.6; MPN BAT85S-TAP -> 1N5817-TP; Manufacturer Vishay -> Micro Commercial Co
