File: kicad/placard.kicad_sch (KiCad schematic)
At the start: 0 parts

Commit message: Carry the PS/2 receiver PLD and the dropped matrix keyboard through the design
The matrix keyboard (U37, U39, J1, RN2, the keyboard board) is gone and the
PS/2 receiver PLD U42 (ATF22V10_PS2.pld rev 02) is added everywhere except
the hand-edited board layout:

- Drivers: receiver-based kbd_scan / mouse_poll / ps2_poll, PS2_LSN listened
  device, ps2_pause waits for a half-received mouse byte and holds the line
  at least 100 us; pad_read frees the mouse clock only briefly.
- Simulator: PS/2 keyboard and mouse models with abort/resend; tests pass.
- Bring-up ROM polls the PS/2 keyboard; BRINGUP.md step 18 rewritten.
- FPGA: port_pld rev 04, new ps2_pld, basys_top wired to both, matrix gone.
- Schematic: shared port sheet redrawn (U38, U42, D1/D4/D5/D19, R60),
  keyboard project, key switch footprints and header removed, C42 -> C47,
  PDFs and I/O PNG regenerated (netlist and ERC clean).
- BOM: keyboard board removed, U42 and C42 added; main board $184.77.
- Docs: IO, CHIPS, PLD_USAGE, LIBRARY, MENU, SCHEMATIC_PLAN, KITTING,
  EXPANSION, ROM, README, kicad README; dated notes in KIT_PRICING and CASE
  (keyboard kit and keyboard bay are moot, re-cost and case rethink pending).
- Block diagram regenerated (33 chips).

Co-Authored-By: Claude Fable 5.1 <noreply@anthropic.com>
Claude-Session: https://claude.ai/code/session_01QpoMmygNy6VSnJkmoq279r
Other:
- note added: "J2-J5"
- note added: "U38 port PLD, U42 PS/2 receiver"
- note removed: "U37 latch, U38 port PLD"
- note removed: "U39 rows, J1-J5"
Changed lines of the file:
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@@
   (text "U16 color decoder, VGA" (at 23 177 0) (effects (font (size 2.5 2.5)) (justify left bottom)))
   (text "U36 audio DAC, J6" (at 23 184 0) (effects (font (size 2.5 2.5)) (justify left bottom)))
-  (text "U37 latch, U38 port PLD" (at 118 170 0) (effects (font (size 2.5 2.5)) (justify left bottom)))
-  (text "U39 rows, J1-J5" (at 118 177 0) (effects (font (size 2.5 2.5)) (justify left bottom)))
+  (text "U38 port PLD, U42 PS/2 receiver" (at 118 170 0) (effects (font (size 2.5 2.5)) (justify left bottom)))
+  (text "J2-J5" (at 118 177 0) (effects (font (size 2.5 2.5)) (justify left bottom)))
   (text "J9-J12 card-edge slots" (at 308 115 0) (effects (font (size 2.5 2.5)) (justify left bottom)))
   (text "34 chips + U40 regulator (docs/CHIPS.md numbers; U24, U28, U30, U33, U34 are not used)." (at 20 220 0) (effects (font (size 3 3)) (justify left bottom)))
