File: kicad/cartridge/cartridge.kicad_sch (KiCad schematic)
At the start: 12 parts, among them J1 Card edge (87715-9106 mate), U1 ATF22V10C-7PX, U2 AT28C256-15PU, U3 AT28C256-15PU, U4 AS7C256C-15PCN, U5 AS7C256C-15PCN

Commit message: Kit footprints: DIP sockets with puller room and part number, resistors with value
Justin: put the chip-puller room in the socket footprints (User.Eco1,
2.5 mm past each end) and the part number in silkscreen between the pin
rows; resistors get their value in silkscreen on the body. New
gen_kicad_kit_footprints.py derives them from KiCad's stock footprints;
schematic, symbols, BOM and PDFs now name them. The board file is left
as is (Justin is editing it): Update PCB from Schematic swaps them in.

Co-Authored-By: Claude Opus 5.5 (1M context) <noreply@anthropic.com>
Claude-Session: https://claude.ai/code/session_01JnVuvUvdWezUUU6Sgmg16H
Parts:
- U1: footprint Package_DIP:DIP-24_W7.62mm -> placard:DIP-24_W7.62mm_Socket_Puller
- U2, U3: footprint Package_DIP:DIP-28_W15.24mm -> placard:DIP-28_W15.24mm_Socket_Puller
- U4, U5: footprint Package_DIP:DIP-28_W7.62mm -> placard:DIP-28_W7.62mm_Socket_Puller
