File: kicad/cartridge_32k/cartridge_32k.kicad_sch (KiCad schematic)
At the start: 7 parts, among them J1 Card edge (87715-9106 mate), U1 ATF22V10C-7PX, U2 AT28C256-15PU, U3 AS7C256C-15PCN

Commit message: BOM/schematic: stocked substitutes from the first parts order
D18 Kingbright WP7113ID (LTL2R3KRD-EM out of stock), 100n TDK
FG28X7R1H104KNT00 (KEMET C320C104 $0.66 at Mouser), C45 TDK
FG24C0G1H153JNT06 (KEMET non-stocked), Vishay BAT85S-TAP and
1N4148-TAP, MF-RG300-0, USB4125-GF-A-0190; Mouser prices re-checked.

Co-Authored-By: Claude Opus 5.5 (1M context) <noreply@anthropic.com>
Claude-Session: https://claude.ai/code/session_017y5UgjExE8oeP7QrfvhCzb
Parts:
- C1, C2, C3: MPN C320C104K5R5TA -> FG28X7R1H104KNT00; Manufacturer KEMET -> TDK
Changed lines of the file:
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@@
   (symbol (lib_id "power:+5V") (at 149.86 82.55 0) (unit 1) (in_bom yes) (on_board yes) (dnp no) (property "Reference" "#PWR0106" (at 149.86 82.55 0) (effects (font (size 1.27 1.27)) hide)) (property "Value" "+5V" (at 149.86 76.2 0) (effects (font (size 2 2)))) (property "Footprint" "" (at 149.86 82.55 0) (effects (font (size 1.27 1.27)) hide)) (property "Datasheet" "" (at 149.86 82.55 0) (effects (font (size 1.27 1.27)) hide)) (pin "1") (instances (project "cartridge_32k" (path "/7406a4ab-9e40-5a47-bfe2-c7a63f89be7c" (reference "#PWR0106") (unit 1)))))
   (symbol (lib_id "power:GND") (at 149.86 90.17 0) (unit 1) (in_bom yes) (on_board yes) (dnp no) (property "Reference" "#PWR0107" (at 149.86 90.17 0) (effects (font (size 1.27 1.27)) hide)) (property "Value" "GND" (at 149.86 96.52 0) (effects (font (size 2 2)) hide)) (property "Footprint" "" (at 149.86 90.17 0) (effects (font (size 1.27 1.27)) hide)) (property "Datasheet" "" (at 149.86 90.17 0) (effects (font (size 1.27 1.27)) hide)) (pin "1") (instances (project "cartridge_32k" (path "/7406a4ab-9e40-5a47-bfe2-c7a63f89be7c" (reference "#PWR0107") (unit 1)))))
-  (symbol (lib_id "placard_std:C") (at 149.86 86.36 0) (unit 1) (in_bom yes) (on_board yes) (dnp no) (property "Reference" "C1" (at 151.86 85.86 0) (effects (font (size 2.54 2.54) bold) (justify left bottom))) (property "Value" "100n" (at 151.86 88.96 0) (effects (font (size 2 2)) (justify left top))) (property "Footprint" "Capacitor_THT:C_Disc_D5.0mm_W2.5mm_P5.00mm" (at 149.86 86.36 0) (effects (font (size 1.27 1.27)) hide)) (property "Datasheet" "~" (at 149.86 86.36 0) (effects (font (size 1.27 1.27)) hide)) (property "Manufacturer" "KEMET" (at 149.86 86.36 0) (effects (font (size 1.27 1.27)) hide)) (property "MPN" "C320C104K5R5TA" (at 149.86 86.36 0) (effects (font (size 1.27 1.27)) hide)) (pin "1") (pin "2") (instances (project "cartridge_32k" (path "/7406a4ab-9e40-5a47-bfe2-c7a63f89be7c" (reference "C1") (unit 1)))))
+  (symbol (lib_id "placard_std:C") (at 149.86 86.36 0) (unit 1) (in_bom yes) (on_board yes) (dnp no) (property "Reference" "C1" (at 151.86 85.86 0) (effects (font (size 2.54 2.54) bold) (justify left bottom))) (property "Value" "100n" (at 151.86 88.96 0) (effects (font (size 2 2)) (justify left top))) (property "Footprint" "Capacitor_THT:C_Disc_D5.0mm_W2.5mm_P5.00mm" (at 149.86 86.36 0) (effects (font (size 1.27 1.27)) hide)) (property "Datasheet" "~" (at 149.86 86.36 0) (effects (font (size 1.27 1.27)) hide)) (property "Manufacturer" "TDK" (at 149.86 86.36 0) (effects (font (size 1.27 1.27)) hide)) (property "MPN" "FG28X7R1H104KNT00" (at 149.86 86.36 0) (effects (font (size 1.27 1.27)) hide)) (pin "1") (pin "2") (instances (project "cartridge_32k" (path "/7406a4ab-9e40-5a47-bfe2-c7a63f89be7c" (reference "C1") (unit 1)))))
   (symbol (lib_id "power:+5V") (at 160.02 205.74 0) (unit 1) (in_bom yes) (on_board yes) (dnp no) (property "Reference" "#PWR0108" (at 160.02 205.74 0) (effects (font (size 1.27 1.27)) hide)) (property "Value" "+5V" (at 160.02 199.39 0) (effects (font (size 2 2)))) (property "Footprint" "" (at 160.02 205.74 0) (effects (font (size 1.27 1.27)) hide)) (property "Datasheet" "" (at 160.02 205.74 0) (effects (font (size 1.27 1.27)) hide)) (pin "1") (instances (project "cartridge_32k" (path "/7406a4ab-9e40-5a47-bfe2-c7a63f89be7c" (reference "#PWR0108") (unit 1)))))
   (wire (pts (xy 160.02 205.74) (xy 167.64 205.74)) (stroke (width 0) (type default)))
@@
   (symbol (lib_id "power:+5V") (at 250.19 53.34 0) (unit 1) (in_bom yes) (on_board yes) (dnp no) (property "Reference" "#PWR0116" (at 250.19 53.34 0) (effects (font (size 1.27 1.27)) hide)) (property "Value" "+5V" (at 250.19 46.99 0) (effects (font (size 2 2)))) (property "Footprint" "" (at 250.19 53.34 0) (effects (font (size 1.27 1.27)) hide)) (property "Datasheet" "" (at 250.19 53.34 0) (effects (font (size 1.27 1.27)) hide)) (pin "1") (instances (project "cartridge_32k" (path "/7406a4ab-9e40-5a47-bfe2-c7a63f89be7c" (reference "#PWR0116") (unit 1)))))
   (symbol (lib_id "power:GND") (at 250.19 60.96 0) (unit 1) (in_bom yes) (on_board yes) (dnp no) (property "Reference" "#PWR0117" (at 250.19 60.96 0) (effects (font (size 1.27 1.27)) hide)) (property "Value" "GND" (at 250.19 67.31 0) (effects (font (size 2 2)) hide)) (property "Footprint" "" (at 250.19 60.96 0) (effects (font (size 1.27 1.27)) hide)) (property "Datasheet" "" (at 250.19 60.96 0) (effects (font (size 1.27 1.27)) hide)) (pin "1") (instances (project "cartridge_32k" (path "/7406a4ab-9e40-5a47-bfe2-c7a63f89be7c" (reference "#PWR0117") (unit 1)))))
-  (symbol (lib_id "placard_std:C") (at 250.19 57.15 0) (unit 1) (in_bom yes) (on_board yes) (dnp no) (property "Reference" "C2" (at 252.19 56.65 0) (effects (font (size 2.54 2.54) bold) (justify left bottom))) (property "Value" "100n" (at 252.19 59.75 0) (effects (font (size 2 2)) (justify left top))) (property "Footprint" "Capacitor_THT:C_Disc_D5.0mm_W2.5mm_P5.00mm" (at 250.19 57.15 0) (effects (font (size 1.27 1.27)) hide)) (property "Datasheet" "~" (at 250.19 57.15 0) (effects (font (size 1.27 1.27)) hide)) (property "Manufacturer" "KEMET" (at 250.19 57.15 0) (effects (font (size 1.27 1.27)) hide)) (property "MPN" "C320C104K5R5TA" (at 250.19 57.15 0) (effects (font (size 1.27 1.27)) hide)) (pin "1") (pin "2") (instances (project "cartridge_32k" (path "/7406a4ab-9e40-5a47-bfe2-c7a63f89be7c" (reference "C2") (unit 1)))))
+  (symbol (lib_id "placard_std:C") (at 250.19 57.15 0) (unit 1) (in_bom yes) (on_board yes) (dnp no) (property "Reference" "C2" (at 252.19 56.65 0) (effects (font (size 2.54 2.54) bold) (justify left bottom))) (property "Value" "100n" (at 252.19 59.75 0) (effects (font (size 2 2)) (justify left top))) (property "Footprint" "Capacitor_THT:C_Disc_D5.0mm_W2.5mm_P5.00mm" (at 250.19 57.15 0) (effects (font (size 1.27 1.27)) hide)) (property "Datasheet" "~" (at 250.19 57.15 0) (effects (font (size 1.27 1.27)) hide)) (property "Manufacturer" "TDK" (at 250.19 57.15 0) (effects (font (size 1.27 1.27)) hide)) (property "MPN" "FG28X7R1H104KNT00" (at 250.19 57.15 0) (effects (font (size 1.27 1.27)) hide)) (pin "1") (pin "2") (instances (project "cartridge_32k" (path "/7406a4ab-9e40-5a47-bfe2-c7a63f89be7c" (reference "C2") (unit 1)))))
   (wire (pts (xy 267.97 167.64) (xy 267.97 165.1)) (stroke (width 0) (type default)))
   (symbol (lib_id "power:+5V") (at 267.97 165.1 0) (unit 1) (in_bom yes) (on_board yes) (dnp no) (property "Reference" "#PWR0118" (at 267.97 165.1 0) (effects (font (size 1.27 1.27)) hide)) (property "Value" "+5V" (at 267.97 158.75 0) (effects (font (size 2 2)))) (property "Footprint" "" (at 267.97 165.1 0) (effects (font (size 1.27 1.27)) hide)) (property "Datasheet" "" (at 267.97 165.1 0) (effects (font (size 1.27 1.27)) hide)) (pin "1") (instances (project "cartridge_32k" (path "/7406a4ab-9e40-5a47-bfe2-c7a63f89be7c" (reference "#PWR0118") (unit 1)))))
@@
   (symbol (lib_id "power:+5V") (at 247.65 153.67 0) (unit 1) (in_bom yes) (on_board yes) (dnp no) (property "Reference" "#PWR0121" (at 247.65 153.67 0) (effects (font (size 1.27 1.27)) hide)) (property "Value" "+5V" (at 247.65 147.32 0) (effects (font (size 2 2)))) (property "Footprint" "" (at 247.65 153.67 0) (effects (font (size 1.27 1.27)) hide)) (property "Datasheet" "" (at 247.65 153.67 0) (effects (font (size 1.27 1.27)) hide)) (pin "1") (instances (project "cartridge_32k" (path "/7406a4ab-9e40-5a47-bfe2-c7a63f89be7c" (reference "#PWR0121") (unit 1)))))
   (symbol (lib_id "power:GND") (at 247.65 161.29 0) (unit 1) (in_bom yes) (on_board yes) (dnp no) (property "Reference" "#PWR0122" (at 247.65 161.29 0) (effects (font (size 1.27 1.27)) hide)) (property "Value" "GND" (at 247.65 167.64 0) (effects (font (size 2 2)) hide)) (property "Footprint" "" (at 247.65 161.29 0) (effects (font (size 1.27 1.27)) hide)) (property "Datasheet" "" (at 247.65 161.29 0) (effects (font (size 1.27 1.27)) hide)) (pin "1") (instances (project "cartridge_32k" (path "/7406a4ab-9e40-5a47-bfe2-c7a63f89be7c" (reference "#PWR0122") (unit 1)))))
-  (symbol (lib_id "placard_std:C") (at 247.65 157.48 0) (unit 1) (in_bom yes) (on_board yes) (dnp no) (property "Reference" "C3" (at 249.65 156.98 0) (effects (font (size 2.54 2.54) bold) (justify left bottom))) (property "Value" "100n" (at 249.65 160.08 0) (effects (font (size 2 2)) (justify left top))) (property "Footprint" "Capacitor_THT:C_Disc_D5.0mm_W2.5mm_P5.00mm" (at 247.65 157.48 0) (effects (font (size 1.27 1.27)) hide)) (property "Datasheet" "~" (at 247.65 157.48 0) (effects (font (size 1.27 1.27)) hide)) (property "Manufacturer" "KEMET" (at 247.65 157.48 0) (effects (font (size 1.27 1.27)) hide)) (property "MPN" "C320C104K5R5TA" (at 247.65 157.48 0) (effects (font (size 1.27 1.27)) hide)) (pin "1") (pin "2") (instances (project "cartridge_32k" (path "/7406a4ab-9e40-5a47-bfe2-c7a63f89be7c" (reference "C3") (unit 1)))))
+  (symbol (lib_id "placard_std:C") (at 247.65 157.48 0) (unit 1) (in_bom yes) (on_board yes) (dnp no) (property "Reference" "C3" (at 249.65 156.98 0) (effects (font (size 2.54 2.54) bold) (justify left bottom))) (property "Value" "100n" (at 249.65 160.08 0) (effects (font (size 2 2)) (justify left top))) (property "Footprint" "Capacitor_THT:C_Disc_D5.0mm_W2.5mm_P5.00mm" (at 247.65 157.48 0) (effects (font (size 1.27 1.27)) hide)) (property "Datasheet" "~" (at 247.65 157.48 0) (effects (font (size 1.27 1.27)) hide)) (property "Manufacturer" "TDK" (at 247.65 157.48 0) (effects (font (size 1.27 1.27)) hide)) (property "MPN" "FG28X7R1H104KNT00" (at 247.65 157.48 0) (effects (font (size 1.27 1.27)) hide)) (pin "1") (pin "2") (instances (project "cartridge_32k" (path "/7406a4ab-9e40-5a47-bfe2-c7a63f89be7c" (reference "C3") (unit 1)))))
   (text "U2 holds the 32K image, programmed off the board;" (at 22 192 0) (effects (font (size 2.5 2.5)) (justify left bottom)))
   (text "its /WE is tied high.  U3 is the ROM the CPU" (at 22 196 0) (effects (font (size 2.5 2.5)) (justify left bottom)))

Commit message: Cartridge slot: contacts in cartridge chip-pin order for autorouting
The cartridge boards would not route with the address lines in bus
order on the connector (the loader PLD sits right behind the fingers).
Each side's signals now leave the fingers in the order of the chip pins
they reach, which lets both cartridge boards route on four layers.
One pinout table (CART_PINOUT) feeds J8 on the main board and J1 on the
cartridges; the slot symbol, every sheet, the PDFs, EXPANSION.md and
SCHEMATIC_PLAN.md follow.  The main board's J8 traces need rerouting.

Co-Authored-By: Claude Fable 5.1 <noreply@anthropic.com>
Claude-Session: https://claude.ai/code/session_017okF1JiLRNFTfH7Az85hff
Connections:
- net A0: now also J1.A22 (A0); no longer J1.A3 (A0)
- net A1: now also J1.A19 (A1); no longer J1.B3 (A1)
- net A10: now also J1.A18 (A10); no longer J1.A8 (A10)
- net A11: now also J1.A13 (A11); no longer J1.B8 (A11)
- net A12: now also J1.B3 (A12); no longer J1.A9 (A12)
- net A13: now also J1.A6 (A13); no longer J1.B9 (A13)
- net A14: now also J1.A3 (A14); no longer J1.A10 (A14)
- net A2: now also J1.A17 (A2); no longer J1.A4 (A2)
- net A3: now also J1.A15 (A3); no longer J1.B4 (A3)
- net A4: now also J1.A14 (A4); no longer J1.A5 (A4)
- net A5: now also J1.B9 (A5); no longer J1.B5 (A5)
- net A6: now also J1.B7 (A6); no longer J1.A6
- net A7: now also J1.A4 (A7); no longer J1.B6 (A7)
- net A8: now also J1.A8; no longer J1.A7 (A8)
- net A9: now also J1.A9; no longer J1.B7 (A9)
- net D0: now also J1.A24 (D0); no longer J1.A12 (D0)
- net D1: now also J1.A27 (D1); no longer J1.B12 (D1)
- net D2: now also J1.A29 (D2); no longer J1.A13 (D2)
- net D3: now also J1.A32 (D3); no longer J1.B13 (D3)
- net D4: now also J1.A30 (D4); no longer J1.A14 (D4)
- net D5: now also J1.B27 (D5); no longer J1.B14 (D5)
- net D6: now also J1.A25 (D6); no longer J1.A15 (D6)
- net D7: now also J1.B22 (D7); no longer J1.B15 (D7)
- net ~{CE_LO}: now also J1.A5 (/CE_LO); no longer J1.A16 (/CE_LO)
- net ~{ROM_OE}: now also J1.A16 (/ROM_OE); no longer J1.A17 (/ROM_OE)
- net at U1.1 (CLK): now also J1.B4 (CLK); no longer J1.A20 (CLK)
- net at U1.22 (RUN): now also J1.B6 (RUN); no longer J1.A19 (RUN)
- net at U1.23 (STALL_OUT): now also J1.B5 (STALL_OUT); no longer J1.B18 (STALL_OUT)
- net at U1.3 (PIXEL_ENABLE): now also J1.A7 (PIXEL_ENABLE); no longer J1.A18 (PIXEL_ENABLE)
- net at U1.4 (PC_ENABLE): now also J1.B8 (PC_ENABLE); no longer J1.B19 (PC_ENABLE)
- net at U1.5 (STALL_IN): now also J1.B12 (STALL_IN); no longer J1.B17 (STALL_IN)
Changed lines of the file:
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@@
 (kicad_sch (version 20230121) (generator eeschema)
   (paper "A3")
-  (title_block (title "Placard: ROM cartridge, 32K") (date "2026-10-25") (rev "1") (company "Placard computer") (comment 1 "Generated by src/scripts/gen_kicad_schematic.py; plan in docs/SCHEMATIC_PLAN.md") (comment 2 "Cartridge chips U1-U3 (docs/CHIPS.md, ROM cartridge); decoupling Cn goes with Un"))
+  (title_block (title "Placard: ROM cartridge, 32K") (date "2026-10-26") (rev "1") (company "Placard computer") (comment 1 "Generated by src/scripts/gen_kicad_schematic.py; plan in docs/SCHEMATIC_PLAN.md") (comment 2 "Cartridge chips U1-U3 (docs/CHIPS.md, ROM cartridge); decoupling Cn goes with Un"))
   (text "ROM cartridge, 32K" (at 15 22 0) (effects (font (size 6 6) bold) (justify left bottom)))
   (text "One EEPROM copied into one SRAM at power-up by the loader PLD (ROM.md, \"Loading the cartridge\")" (at 15 30 0) (effects (font (size 3 3)) (justify left bottom)))
@@
   (wire (pts (xy 82.55 167.64) (xy 82.55 170.18)) (stroke (width 0) (type default)))
   (symbol (lib_id "power:GND") (at 82.55 170.18 0) (unit 1) (in_bom yes) (on_board yes) (dnp no) (property "Reference" "#PWR0103" (at 82.55 170.18 0) (effects (font (size 1.27 1.27)) hide)) (property "Value" "GND" (at 82.55 176.53 0) (effects (font (size 2 2)) hide)) (property "Footprint" "" (at 82.55 170.18 0) (effects (font (size 1.27 1.27)) hide)) (property "Datasheet" "" (at 82.55 170.18 0) (effects (font (size 1.27 1.27)) hide)) (pin "1") (instances (project "cartridge_32k" (path "/7406a4ab-9e40-5a47-bfe2-c7a63f89be7c" (reference "#PWR0103") (unit 1)))))
-  (symbol (lib_id "placard_parts:Cartridge_Slot") (at 82.55 119.38 0) (unit 1) (in_bom no) (on_board yes) (dnp no) (property "Reference" "J1" (at 67 69 0) (effects (font (size 2.54 2.54) bold) (justify left bottom))) (property "Value" "Card edge (87715-9106 mate)" (at 88 176 0) (effects (font (size 2 2)) (justify left top))) (property "Footprint" "placard:Card_Edge_87715-9106" (at 82.55 119.38 0) (effects (font (size 1.27 1.27)) hide)) (property "Datasheet" "~" (at 82.55 119.38 0) (effects (font (size 1.27 1.27)) hide)) (pin "A3") (pin "B3") (pin "A4") (pin "B4") (pin "A5") (pin "B5") (pin "A6") (pin "B6") (pin "A7") (pin "B7") (pin "A8") (pin "B8") (pin "A9") (pin "B9") (pin "A10") (pin "A16") (pin "B16") (pin "A17") (pin "B10") (pin "A22") (pin "A23") (pin "A24") (pin "A25") (pin "A26") (pin "A27") (pin "A28") (pin "A29") (pin "A30") (pin "A32") (pin "B20") (pin "A12") (pin "B12") (pin "A13") (pin "B13") (pin "A14") (pin "B14") (pin "A15") (pin "B15") (pin "A20") (pin "A18") (pin "B19") (pin "B17") (pin "B18") (pin "A19") (pin "B22") (pin "B23") (pin "B24") (pin "B25") (pin "B26") (pin "B27") (pin "B28") (pin "B29") (pin "B30") (pin "B32") (pin "A2") (pin "B2") (pin "A1") (pin "B1") (pin "A11") (pin "B11") (pin "A21") (pin "B21") (pin "A31") (pin "B31") (instances (project "cartridge_32k" (path "/7406a4ab-9e40-5a47-bfe2-c7a63f89be7c" (reference "J1") (unit 1)))))
+  (symbol (lib_id "placard_parts:Cartridge_Slot") (at 82.55 119.38 0) (unit 1) (in_bom no) (on_board yes) (dnp no) (property "Reference" "J1" (at 67 69 0) (effects (font (size 2.54 2.54) bold) (justify left bottom))) (property "Value" "Card edge (87715-9106 mate)" (at 88 176 0) (effects (font (size 2 2)) (justify left top))) (property "Footprint" "placard:Card_Edge_87715-9106" (at 82.55 119.38 0) (effects (font (size 1.27 1.27)) hide)) (property "Datasheet" "~" (at 82.55 119.38 0) (effects (font (size 1.27 1.27)) hide)) (pin "A22") (pin "A19") (pin "A17") (pin "A15") (pin "A14") (pin "B9") (pin "B7") (pin "A4") (pin "A8") (pin "A9") (pin "A18") (pin "A13") (pin "B3") (pin "A6") (pin "A3") (pin "A5") (pin "B16") (pin "A16") (pin "B10") (pin "A10") (pin "A12") (pin "B13") (pin "B14") (pin "B15") (pin "B17") (pin "B18") (pin "B19") (pin "A20") (pin "B20") (pin "A23") (pin "A24") (pin "A27") (pin "A29") (pin "A32") (pin "A30") (pin "B27") (pin "A25") (pin "B22") (pin "B4") (pin "A7") (pin "B8") (pin "B12") (pin "B5") (pin "B6") (pin "B23") (pin "B24") (pin "B25") (pin "A26") (pin "B26") (pin "A28") (pin "B28") (pin "B29") (pin "B30") (pin "B32") (pin "A2") (pin "B2") (pin "A1") (pin "B1") (pin "A11") (pin "B11") (pin "A21") (pin "B21") (pin "A31") (pin "B31") (instances (project "cartridge_32k" (path "/7406a4ab-9e40-5a47-bfe2-c7a63f89be7c" (reference "J1") (unit 1)))))
   (wire (pts (xy 57.15 119.38) (xy 52.07 119.38)) (stroke (width 0) (type default)))
   (wire (pts (xy 57.15 124.46) (xy 52.07 124.46)) (stroke (width 0) (type default)))

Commit message: Put every symbol, footprint and 3D model in the project library
- gen_kicad_stock_footprints.py: copies of the KiCad 9.0.6 footprints the
  boards use (C_Disc, CP_Radial, DO-15/DO-35, LED, pin header, oscillator,
  TO-92, SIP9, mounting holes, net tie) into placard.pretty, and KiCad's
  STEP models for them and for the DIP socket / resistor kit footprints
  into placard.3dshapes
- model paths use the PLACARD_LIB text variable (main board
  ${KIPRJMOD}/lib, cartridges ${KIPRJMOD}/../lib) so the shared footprints
  find their models in all three projects
- placard_std gains the 28C256 EEPROM and the power symbols; symbol
  Footprint defaults name placard footprints (relay, SIP9, oscillator,
  TO-92, EEPROM socket)
- schematics regenerated with placard_std power/EEPROM symbols and
  placard: footprints; BOM CSVs and PDFs regenerated
- cartridge .kicad_pro files take in Justin's local KiCad 9 settings

Co-Authored-By: Claude Opus 5.5 <noreply@anthropic.com>
Claude-Session: https://claude.ai/code/session_017okF1JiLRNFTfH7Az85hff
Parts:
- C1, C2, C3: footprint Capacitor_THT:C_Disc_D5.0mm_W2.5mm_P5.00mm -> placard:C_Disc_D5.0mm_W2.5mm_P5.00mm
- U2: symbol Memory_EEPROM:28C256 -> placard_std:28C256
